File: schematic/power_eth.kicad_sch (KiCad schematic)
At the start: 45 parts, among them J1 ARJP11A-MASA-B-A-EMU2, U2 TLV62569DBV, U3 LAN8742A, Y2 25MHz ABM8G

Commit message: Reverse diode orientation
Signed-off-by: Lee Smet <lee.smet@hotmail.com>
Connections:
- net VPOE_N: now also D1.2 (A); no longer D1.1 (K)
- net VPOE_P: now also D1.1 (K); no longer D1.2 (A)
Other:
- moved on the sheet: D1

Commit message: More schematic works
Signed-off-by: Lee Smet <lee.smet@hotmail.com>
Other:
- note added: "Magjack CT regulators"

Commit message: Fix photoMOS package and part, ethernet crystal
Signed-off-by: Lee Smet <lee.smet@hotmail.com>
Parts:
- added R29: 499, Resistor_SMD:R_0402_1005Metric, symbol Device:R
- PS1: footprint (none) -> granite:Silvertel_Ag9905MT
- Y2: value 25MHz ABM8G -> 25MHz 12pF YXC
Connections:
- net at C27.1, Y2.3: now also R29.1; no longer U3.4 (XTAL2)
- new net: R29.2, U3.4 (XTAL2)
Changed lines of the file:
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@@
 	(wire
 		(pts
+			(xy 85.09 236.22) (xy 82.55 236.22)
+		)
+		(stroke
+			(width 0)
+			(type default)
+		)
+	)
+	(wire
+		(pts
 			(xy 123.19 208.28) (xy 156.21 208.28)
 		)
@@
 	(wire
 		(pts
+			(xy 74.93 236.22) (xy 72.39 236.22)
+		)
+		(stroke
+			(width 0)
+			(type default)
+		)
+	)
+	(wire
+		(pts
 			(xy 179.07 104.14) (xy 184.15 104.14)
 		)
@@
 	(wire
 		(pts
-			(xy 85.09 236.22) (xy 72.39 236.22)
-		)
-		(stroke
-			(width 0)
-			(type default)
-		)
-	)
-	(wire
-		(pts
 			(xy 142.24 181.61) (xy 142.24 182.88)
 		)
@@
 			)
 		)
-		(property "Footprint" ""
+		(property "Footprint" "granite:Silvertel_Ag9905MT"
 			(at 163.83 104.14 0)
 			(hide yes)
@@
 			)
 		)
-		(property "Value" "25MHz ABM8G"
+		(property "Value" "25MHz 12pF YXC"
 			(at 63.5 241.3 0)
 			(show_name no)
@@
 					(unit 1)
 				)
+			)
+		)
+	)
+	(symbol
+		(lib_id "Device:R")
+		(at 78.74 236.22 90)
+		(unit 1)
+		(body_style 1)
+		(exclude_from_sim no)
+		(in_bom yes)
+		(on_board yes)
+		(in_pos_files yes)
+		(dnp no)
+		(property "Reference" "R29"
+			(at 79.756 239.014 90)
+			(show_name no)
+			(do_not_autoplace no)
+			(effects
+				(font
+					(size 1.27 1.27)
+				)
+				(justify left)
+			)
+		)
+		(property "Value" "499"
+			(at 79.502 240.792 90)
+			(show_name no)
+			(do_not_autoplace no)
+			(effects
+				(font
+					(size 1.27 1.27)
+				)
+				(justify left)
+			)
+		)
+		(property "Footprint" "Resistor_SMD:R_0402_1005Metric"
+			(at 78.74 236.22 0)
+			(hide yes)
+			(show_name no)
+			(do_not_autoplace no)
+			(effects
+				(font
+					(size 1.27 1.27)
+				)
+			)
+		)
+		(property "Datasheet" ""
+			(at 78.74 236.22 0)
+			(hide yes)
+			(show_name no)
+			(do_not_autoplace no)
+			(effects
+				(font
+					(size 1.27 1.27)
+				)
+			)
+		)
+		(property "Description" ""
+			(at 78.74 236.22 0)
+			(hide yes)
+			(show_name no)
+			(do_not_autoplace no)
+			(effects
+				(font
+					(size 1.27 1.27)
+				)
+			)
+		)
+		(pin "1"
+		)
+		(pin "2"
+		)
+		(instances
+			(project "granite_controller"
+				(path "/bd3d1081-8fd5-561e-93ea-9d28b3145149/8063e2cb-b212-5b7f-a3a7-22937e0bc76b"
+					(reference "R29")
+					(unit 1)
+				)

Commit message: Add manufacturer and MPN to schematic parts
Signed-off-by: Lee Smet <lee.smet@hotmail.com>
Parts:
- C1, C2: MANUFACTURER (none) -> Panasonic; MPN (none) -> 6SVPC220MV
- C26, C27: MANUFACTURER (none) -> Murata; MPN (none) -> GRM1555C1H220JA01D
- C28: MANUFACTURER (none) -> Samsung Electro-Mechanics; MPN (none) -> CL10A105KO8NNNC
- C29, C30, C31, C32, C34, C35: MANUFACTURER (none) -> YAGEO; MPN (none) -> CC0402KRX7R7BB104
- C3, C4: MANUFACTURER (none) -> Samsung Electro-Mechanics; MPN (none) -> CL21A226MAYNNNE
- C36: MANUFACTURER (none) -> KEMET; MPN (none) -> C1812C102KGRACTU
- D1: MANUFACTURER (none) -> Diodes Incorporated; MPN (none) -> SMAJ58A-13-F
- D2, D3: MANUFACTURER (none) -> MDD (Microdiode); MPN (none) -> SS34
- J1: MANUFACTURER (none) -> Abracon; MPN (none) -> ARJP11A-MASA-B-A-EMU2
- L1: MANUFACTURER (none) -> Sunlord; MPN (none) -> SWPA3015S2R2MT
- PS1: MANUFACTURER (none) -> Silvertel; MPN (none) -> AG9905MT
- R1: MANUFACTURER (none) -> YAGEO; MPN (none) -> RC0402FR-07100KL
- R10, R11, R12, R13, R14, R9: MANUFACTURER (none) -> YAGEO; MPN (none) -> RC0402FR-0733RL
- R15: MANUFACTURER (none) -> YAGEO; MPN (none) -> RC0402FR-0712K1L
- R16: MANUFACTURER (none) -> YAGEO; MPN (none) -> RC0402FR-071K5L
- R17, R18, R19: MANUFACTURER (none) -> UNI-ROYAL; MPN (none) -> 0402WGF1002TCE
- R2: MANUFACTURER (none) -> YAGEO; MPN (none) -> RC0402FR-0722K1L
- R20, R21, R22, R23: MANUFACTURER (none) -> YAGEO; MPN (none) -> RC0402FR-0749R9L
- R26, R27: MANUFACTURER (none) -> UNI-ROYAL; MPN (none) -> 0603WAF0000T5E
- R28: MANUFACTURER (none) -> YAGEO; MPN (none) -> RC0603FR-071ML
- R29: MANUFACTURER (none) -> YAGEO; MPN (none) -> RC0402FR-07499RL
- R3, R4: MANUFACTURER (none) -> YAGEO; MPN (none) -> RC0402FR-07470RL
- U2: MANUFACTURER (none) -> Texas Instruments; MPN (none) -> TLV62569DBVR
- U3: MANUFACTURER (none) -> Microchip; MPN (none) -> LAN8742A-CZ-TR
- Y2: MANUFACTURER (none) -> YXC; MPN (none) -> X322525MOB4SI

Commit message: Proper footprint for photoMOS
Signed-off-by: Lee Smet <lee.smet@hotmail.com>
Parts:
- C1, C2: footprint Capacitor_SMD:CP_Elec_6.3x5.8 -> granite:CP_Elec_6.3x5.9_Panasonic_SVPC_C6
Changed lines of the file:
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@@
 			)
 		)
-		(property "Footprint" "Capacitor_SMD:CP_Elec_6.3x5.8"
+		(property "Footprint" "granite:CP_Elec_6.3x5.9_Panasonic_SVPC_C6"
 			(at 219.71 91.44 0)
 			(hide yes)
@@
 			)
 		)
-		(property "Footprint" "Capacitor_SMD:CP_Elec_6.3x5.8"
+		(property "Footprint" "granite:CP_Elec_6.3x5.9_Panasonic_SVPC_C6"
 			(at 190.5 99.06 0)
 			(hide yes)
