File: schematic/relays_a.kicad_sch (KiCad schematic)
At the start: 49 parts, among them J11 MB01_FP, J12 MB02_FP, J13 MB03_FP, J14 MB04_FP, J15 MB05_FP, J16 MB06_FP, J17 MB07_FP, K1 TLP176A, K10 TLP176A, K11 TLP176A, K12 TLP176A, K13 TLP176A, K14 TLP176A, K2 TLP176A, K3 TLP176A, K4 TLP176A, K5 TLP176A, K6 TLP176A, K7 TLP176A, K8 TLP176A, K9 TLP176A

Commit message: More schematic works
Signed-off-by: Lee Smet <lee.smet@hotmail.com>
Changed lines of the file:
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@@
 	)
 	(bus_entry
-		(at 15.24 119.38)
+		(at 15.24 125.73)
 		(size 2.54 -2.54)
 		(stroke
@@
 	)
 	(bus_entry
-		(at 15.24 68.58)
+		(at 15.24 74.93)
 		(size 2.54 -2.54)
 		(stroke
@@
 	)
 	(bus_entry
-		(at 15.24 144.78)
+		(at 15.24 151.13)
 		(size 2.54 -2.54)
 		(stroke
@@
 	)
 	(bus_entry
-		(at 15.24 43.18)
+		(at 15.24 49.53)
 		(size 2.54 -2.54)
 		(stroke
@@
 	)
 	(bus_entry
-		(at 15.24 124.46)
+		(at 15.24 130.81)
 		(size 2.54 -2.54)
 		(stroke
@@
 	)
 	(bus_entry
-		(at 15.24 129.54)
+		(at 15.24 135.89)
 		(size 2.54 -2.54)
 		(stroke
@@
 	)
 	(bus_entry
-		(at 15.24 53.34)
+		(at 15.24 59.69)
 		(size 2.54 -2.54)
 		(stroke
@@
 	)
 	(bus_entry
-		(at 15.24 48.26)
+		(at 15.24 54.61)
 		(size 2.54 -2.54)
 		(stroke
@@
 	)
 	(bus_entry
-		(at 15.24 149.86)
+		(at 15.24 156.21)
 		(size 2.54 -2.54)
 		(stroke
@@
 	)
 	(bus_entry
-		(at 15.24 134.62)
+		(at 15.24 140.97)
 		(size 2.54 -2.54)
 		(stroke
@@
 	)
 	(bus_entry
-		(at 15.24 58.42)
+		(at 15.24 64.77)
 		(size 2.54 -2.54)
 		(stroke
@@
 	)
 	(bus_entry
-		(at 15.24 139.7)
+		(at 15.24 146.05)
 		(size 2.54 -2.54)
 		(stroke
@@
 	)
 	(bus_entry
-		(at 15.24 38.1)
+		(at 15.24 44.45)
 		(size 2.54 -2.54)
 		(stroke
@@
 	)
 	(bus_entry
-		(at 15.24 63.5)
+		(at 15.24 69.85)
 		(size 2.54 -2.54)
 		(stroke
@@
 	(wire
 		(pts
-			(xy 17.78 116.84) (xy 27.94 116.84)
+			(xy 17.78 123.19) (xy 27.94 123.19)
 		)
 		(stroke
@@
 	(wire
 		(pts
-			(xy 17.78 66.04) (xy 27.94 66.04)
+			(xy 17.78 72.39) (xy 27.94 72.39)
 		)
 		(stroke
@@
 	(bus
 		(pts
-			(xy 15.24 30.48) (xy 15.24 68.58)
+			(xy 15.24 36.83) (xy 15.24 74.93)
 		)
 		(stroke
@@
 	(wire
 		(pts
-			(xy 17.78 147.32) (xy 27.94 147.32)
+			(xy 17.78 153.67) (xy 27.94 153.67)
 		)
 		(stroke
@@
 	(wire
 		(pts
-			(xy 17.78 50.8) (xy 27.94 50.8)
+			(xy 17.78 57.15) (xy 27.94 57.15)
 		)
 		(stroke
@@
 	(wire
 		(pts
-			(xy 17.78 55.88) (xy 27.94 55.88)
+			(xy 17.78 62.23) (xy 27.94 62.23)
 		)
 		(stroke
@@
 	(wire
 		(pts
-			(xy 17.78 137.16) (xy 27.94 137.16)
+			(xy 17.78 143.51) (xy 27.94 143.51)
 		)
 		(stroke
@@
 	(wire
 		(pts
-			(xy 17.78 35.56) (xy 27.94 35.56)
+			(xy 17.78 41.91) (xy 27.94 41.91)
 		)
 		(stroke
@@
 	(bus
 		(pts
-			(xy 15.24 111.76) (xy 15.24 149.86)
+			(xy 15.24 118.11) (xy 15.24 156.21)
 		)
 		(stroke
@@
 	(wire
 		(pts
-			(xy 17.78 142.24) (xy 27.94 142.24)
-		)
-		(stroke
-			(width 0)
-			(type default)
-		)
-	)
-	(wire
-		(pts
-			(xy 17.78 121.92) (xy 27.94 121.92)
+			(xy 17.78 148.59) (xy 27.94 148.59)
+		)
+		(stroke
+			(width 0)
+			(type default)
+		)
+	)
+	(wire
+		(pts
+			(xy 17.78 128.27) (xy 27.94 128.27)
 		)
 		(stroke
@@
 	(wire
 		(pts
-			(xy 17.78 60.96) (xy 27.94 60.96)
+			(xy 17.78 67.31) (xy 27.94 67.31)
 		)
 		(stroke
@@
 	(wire
 		(pts
-			(xy 17.78 40.64) (xy 27.94 40.64)
+			(xy 17.78 46.99) (xy 27.94 46.99)
 		)
 		(stroke
@@
 	(wire
 		(pts
-			(xy 17.78 132.08) (xy 27.94 132.08)
+			(xy 17.78 138.43) (xy 27.94 138.43)
 		)
 		(stroke
@@
 	(wire
 		(pts
-			(xy 17.78 127) (xy 27.94 127)
+			(xy 17.78 133.35) (xy 27.94 133.35)
 		)
 		(stroke
@@
 	(wire
 		(pts
-			(xy 17.78 45.72) (xy 27.94 45.72)
+			(xy 17.78 52.07) (xy 27.94 52.07)
 		)
 		(stroke
@@
 	)
 	(label "RST_DRV2"
-		(at 27.94 40.64 0)
+		(at 27.94 46.99 0)
 		(effects
 			(font
@@
 	)
 	(label "PWR_DRV4"
-		(at 27.94 132.08 0)
+		(at 27.94 138.43 0)
 		(effects
 			(font
@@
 	)
 	(label "PWR_DRV1"
-		(at 27.94 116.84 0)
+		(at 27.94 123.19 0)
 		(effects
 			(font
@@
 	)
 	(label "RST_DRV1"
-		(at 27.94 35.56 0)
+		(at 27.94 41.91 0)
 		(effects
 			(font
@@
 	)
 	(label "PWR_DRV3"
-		(at 27.94 127 0)
+		(at 27.94 133.35 0)
 		(effects
 			(font
@@
 	)
 	(label "RST_DRV7"
-		(at 27.94 66.04 0)
+		(at 27.94 72.39 0)
 		(effects
 			(font
@@
 	)
 	(label "RST_DRV6"
-		(at 27.94 60.96 0)
+		(at 27.94 67.31 0)
 		(effects
 			(font
@@
 	)
 	(label "PWR_DRV2"
-		(at 27.94 121.92 0)
+		(at 27.94 128.27 0)
 		(effects
 			(font
@@
 	)
 	(label "PWR_DRV7"
-		(at 27.94 147.32 0)
+		(at 27.94 153.67 0)
 		(effects
 			(font
@@
 	)
 	(label "RST_DRV5"
-		(at 27.94 55.88 0)
+		(at 27.94 62.23 0)
 		(effects
 			(font
@@
 	)
 	(label "RST_DRV4"
-		(at 27.94 50.8 0)
+		(at 27.94 57.15 0)
 		(effects
 			(font
@@
 	)
 	(label "RST_DRV3"
-		(at 27.94 45.72 0)
+		(at 27.94 52.07 0)
 		(effects
 			(font
@@
 	)
 	(label "PWR_DRV6"
-		(at 27.94 142.24 0)
+		(at 27.94 148.59 0)
 		(effects
 			(font
@@
 	)
 	(label "PWR_DRV5"
-		(at 27.94 137.16 0)
+		(at 27.94 143.51 0)
 		(effects
 			(font
@@
 	(hierarchical_label "PWR_DRV[1..14]"
 		(shape input)
-		(at 15.24 111.76 90)
+		(at 15.24 118.11 90)
 		(effects
 			(font
@@
 	(hierarchical_label "RST_DRV[1..14]"
 		(shape input)
-		(at 15.24 30.48 90)
-		(effects
-			(font
+		(at 15.24 36.83 90)
+		(effects
+			(font

Commit message: Fix photoMOS package and part, ethernet crystal
Signed-off-by: Lee Smet <lee.smet@hotmail.com>
Parts:
- K1, K10, K11, K12, K13, K14, K2, K3, K4, K5, K6, K7, K8, K9: value TLP176A -> TLP176AM; footprint Package_SO:SOP-4_3.8x4.1mm_P2.54mm -> Package_SO:SOIC-4_4.55x3.7mm_P2.54mm; symbol Relay_SolidState:CPC1017N -> granite:TLP176AM
Connections:
- net GND: now also K1.3, K10.3, K11.3, K12.3, K13.3, K14.3, K2.3, K3.3, K4.3, K5.3, K6.3, K7.3, K8.3, K9.3; no longer K1.2, K10.2, K11.2, K12.2, K13.2, K14.2, K2.2, K3.2, K4.2, K5.2, K6.2, K7.2, K8.2, K9.2
- net at J12.1 (Pin_1): now also K3.6; no longer K3.4
- net at J12.3 (Pin_3): now also K4.6; no longer K4.4
- net at R205.2: now also K5.4; no longer K5.3
- net at J13.1 (Pin_1): now also K5.6; no longer K5.4
- net at J15.1 (Pin_1): now also K9.6; no longer K9.4
- net at J15.3 (Pin_3): now also K10.6; no longer K10.4
- net at R209.2: now also K9.4; no longer K9.3
- net at J11.1 (Pin_1): now also K1.6; no longer K1.4
- net at J11.3 (Pin_3): now also K2.6; no longer K2.4
- net at R213.2: now also K13.4; no longer K13.3
- net at J13.3 (Pin_3): now also K6.6; no longer K6.4
- net at R204.2: now also K4.4; no longer K4.3
- net at J17.1 (Pin_1): now also K13.6; no longer K13.4
- net at J17.3 (Pin_3): now also K14.6; no longer K14.4
- net at R207.2: now also K7.4; no longer K7.3
- net at R203.2: now also K3.4; no longer K3.3
- net at R201.2: now also K1.4; no longer K1.3
- net at R212.2: now also K12.4; no longer K12.3
- net at R210.2: now also K10.4; no longer K10.3
- net at R214.2: now also K14.4; no longer K14.3
- net at R208.2: now also K8.4; no longer K8.3
- net at J14.3 (Pin_3): now also K8.6; no longer K8.4
- net at R202.2: now also K2.4; no longer K2.3
- net at R211.2: now also K11.4; no longer K11.3
- net at R206.2: now also K6.4; no longer K6.3
- net at J16.1 (Pin_1): now also K11.6; no longer K11.4
- net at J16.3 (Pin_3): now also K12.6; no longer K12.4
- net at J14.1 (Pin_1): now also K7.6; no longer K7.4
Other:
- note added: "Channels 1-7: 2x photoMOS contact closure (RESET, PWR BTN) per motherboard front-panel header. Floating outputs. TLP176AM: 3mA max trigger, ~6.2mA drive."
- note removed: "Channels 1-7: 2x photoMOS contact closure (RESET, PWR BTN) per motherboard front-panel header. Floating outputs. TLP176A: 3mA max trigger, ~6.5mA drive."

Commit message: Add manufacturer and MPN to schematic parts
Signed-off-by: Lee Smet <lee.smet@hotmail.com>
Parts:
- J11, J12, J13, J14, J15, J16, J17: MANUFACTURER (none) -> JST; MPN (none) -> B4B-PH-K-S(LF)(SN)
- K1, K10, K11, K12, K13, K14, K2, K3, K4, K5, K6, K7, K8, K9: MANUFACTURER (none) -> Toshiba; MPN (none) -> TLP176AM(TPL,E)
- R101, R102, R103, R104, R105, R106, R107, R108, R109, R110, R111, R112, R113, R114: MANUFACTURER (none) -> YAGEO; MPN (none) -> RC0402FR-07330RL
- R201, R202, R203, R204, R205, R206, R207, R208, R209, R210, R211, R212, R213, R214: MANUFACTURER (none) -> YAGEO; MPN (none) -> RC0603FR-07100RL
