File: schematic/relays_b.kicad_sch (KiCad schematic)
At the start: 49 parts, among them J18 MB08_FP, J19 MB09_FP, J20 MB10_FP, J21 MB11_FP, J22 MB12_FP, J23 MB13_FP, J24 MB14_FP, K15 TLP176A, K16 TLP176A, K17 TLP176A, K18 TLP176A, K19 TLP176A, K20 TLP176A, K21 TLP176A, K22 TLP176A, K23 TLP176A, K24 TLP176A, K25 TLP176A, K26 TLP176A, K27 TLP176A, K28 TLP176A

Commit message: More schematic works
Signed-off-by: Lee Smet <lee.smet@hotmail.com>
Changed lines of the file:
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@@
 	)
 	(bus_entry
-		(at 15.24 43.18)
+		(at 15.24 49.53)
 		(size 2.54 -2.54)
 		(stroke
@@
 	)
 	(bus_entry
-		(at 15.24 129.54)
+		(at 15.24 135.89)
 		(size 2.54 -2.54)
 		(stroke
@@
 	)
 	(bus_entry
-		(at 15.24 144.78)
+		(at 15.24 151.13)
 		(size 2.54 -2.54)
 		(stroke
@@
 	)
 	(bus_entry
-		(at 15.24 48.26)
+		(at 15.24 54.61)
 		(size 2.54 -2.54)
 		(stroke
@@
 	)
 	(bus_entry
-		(at 15.24 38.1)
+		(at 15.24 44.45)
 		(size 2.54 -2.54)
 		(stroke
@@
 	)
 	(bus_entry
-		(at 15.24 53.34)
+		(at 15.24 59.69)
 		(size 2.54 -2.54)
 		(stroke
@@
 	)
 	(bus_entry
-		(at 15.24 124.46)
+		(at 15.24 130.81)
 		(size 2.54 -2.54)
 		(stroke
@@
 	)
 	(bus_entry
-		(at 15.24 68.58)
+		(at 15.24 74.93)
 		(size 2.54 -2.54)
 		(stroke
@@
 	)
 	(bus_entry
-		(at 15.24 58.42)
+		(at 15.24 64.77)
 		(size 2.54 -2.54)
 		(stroke
@@
 	)
 	(bus_entry
-		(at 15.24 149.86)
+		(at 15.24 156.21)
 		(size 2.54 -2.54)
 		(stroke
@@
 	)
 	(bus_entry
-		(at 15.24 134.62)
+		(at 15.24 140.97)
 		(size 2.54 -2.54)
 		(stroke
@@
 	)
 	(bus_entry
-		(at 15.24 139.7)
+		(at 15.24 146.05)
 		(size 2.54 -2.54)
 		(stroke
@@
 	)
 	(bus_entry
-		(at 15.24 119.38)
+		(at 15.24 125.73)
 		(size 2.54 -2.54)
 		(stroke
@@
 	)
 	(bus_entry
-		(at 15.24 63.5)
+		(at 15.24 69.85)
 		(size 2.54 -2.54)
 		(stroke
@@
 	(wire
 		(pts
-			(xy 17.78 66.04) (xy 27.94 66.04)
+			(xy 17.78 72.39) (xy 27.94 72.39)
 		)
 		(stroke
@@
 	(wire
 		(pts
-			(xy 17.78 50.8) (xy 27.94 50.8)
+			(xy 17.78 57.15) (xy 27.94 57.15)
 		)
 		(stroke
@@
 	(wire
 		(pts
-			(xy 17.78 35.56) (xy 27.94 35.56)
+			(xy 17.78 41.91) (xy 27.94 41.91)
 		)
 		(stroke
@@
 	(bus
 		(pts
-			(xy 15.24 111.76) (xy 15.24 149.86)
+			(xy 15.24 118.11) (xy 15.24 156.21)
 		)
 		(stroke
@@
 	(wire
 		(pts
-			(xy 17.78 132.08) (xy 27.94 132.08)
+			(xy 17.78 138.43) (xy 27.94 138.43)
 		)
 		(stroke
@@
 	(wire
 		(pts
-			(xy 17.78 147.32) (xy 27.94 147.32)
+			(xy 17.78 153.67) (xy 27.94 153.67)
 		)
 		(stroke
@@
 	(wire
 		(pts
-			(xy 17.78 142.24) (xy 27.94 142.24)
+			(xy 17.78 148.59) (xy 27.94 148.59)
 		)
 		(stroke
@@
 	(wire
 		(pts
-			(xy 17.78 116.84) (xy 27.94 116.84)
+			(xy 17.78 123.19) (xy 27.94 123.19)
 		)
 		(stroke
@@
 	(bus
 		(pts
-			(xy 15.24 30.48) (xy 15.24 68.58)
+			(xy 15.24 36.83) (xy 15.24 74.93)
 		)
 		(stroke
@@
 	(wire
 		(pts
-			(xy 17.78 55.88) (xy 27.94 55.88)
+			(xy 17.78 62.23) (xy 27.94 62.23)
 		)
 		(stroke
@@
 	(wire
 		(pts
-			(xy 17.78 60.96) (xy 27.94 60.96)
+			(xy 17.78 67.31) (xy 27.94 67.31)
 		)
 		(stroke
@@
 	(wire
 		(pts
-			(xy 17.78 45.72) (xy 27.94 45.72)
-		)
-		(stroke
-			(width 0)
-			(type default)
-		)
-	)
-	(wire
-		(pts
-			(xy 17.78 127) (xy 27.94 127)
+			(xy 17.78 52.07) (xy 27.94 52.07)
+		)
+		(stroke
+			(width 0)
+			(type default)
+		)
+	)
+	(wire
+		(pts
+			(xy 17.78 133.35) (xy 27.94 133.35)
 		)
 		(stroke
@@
 	(wire
 		(pts
-			(xy 17.78 40.64) (xy 27.94 40.64)
+			(xy 17.78 46.99) (xy 27.94 46.99)
 		)
 		(stroke
@@
 	(wire
 		(pts
-			(xy 17.78 137.16) (xy 27.94 137.16)
+			(xy 17.78 143.51) (xy 27.94 143.51)
 		)
 		(stroke
@@
 	(wire
 		(pts
-			(xy 17.78 121.92) (xy 27.94 121.92)
+			(xy 17.78 128.27) (xy 27.94 128.27)
 		)
 		(stroke
@@
 	)
 	(label "RST_DRV11"
-		(at 27.94 50.8 0)
+		(at 27.94 57.15 0)
 		(effects
 			(font
@@
 	)
 	(label "PWR_DRV11"
-		(at 27.94 132.08 0)
+		(at 27.94 138.43 0)
 		(effects
 			(font
@@
 	)
 	(label "PWR_DRV10"
-		(at 27.94 127 0)
+		(at 27.94 133.35 0)
 		(effects
 			(font
@@
 	)
 	(label "PWR_DRV13"
-		(at 27.94 142.24 0)
+		(at 27.94 148.59 0)
 		(effects
 			(font
@@
 	)
 	(label "RST_DRV8"
-		(at 27.94 35.56 0)
+		(at 27.94 41.91 0)
 		(effects
 			(font
@@
 	)
 	(label "RST_DRV10"
-		(at 27.94 45.72 0)
+		(at 27.94 52.07 0)
 		(effects
 			(font
@@
 	)
 	(label "PWR_DRV9"
-		(at 27.94 121.92 0)
+		(at 27.94 128.27 0)
 		(effects
 			(font
@@
 	)
 	(label "RST_DRV9"
-		(at 27.94 40.64 0)
+		(at 27.94 46.99 0)
 		(effects
 			(font
@@
 	)
 	(label "RST_DRV13"
-		(at 27.94 60.96 0)
+		(at 27.94 67.31 0)
 		(effects
 			(font
@@
 	)
 	(label "PWR_DRV12"
-		(at 27.94 137.16 0)
+		(at 27.94 143.51 0)
 		(effects
 			(font
@@
 	)
 	(label "PWR_DRV8"
-		(at 27.94 116.84 0)
+		(at 27.94 123.19 0)
 		(effects
 			(font
@@
 	)
 	(label "RST_DRV12"
-		(at 27.94 55.88 0)
+		(at 27.94 62.23 0)
 		(effects
 			(font
@@
 	)
 	(label "PWR_DRV14"
-		(at 27.94 147.32 0)
+		(at 27.94 153.67 0)
 		(effects
 			(font
@@
 	)
 	(label "RST_DRV14"
-		(at 27.94 66.04 0)
+		(at 27.94 72.39 0)
 		(effects
 			(font
@@
 	(hierarchical_label "PWR_DRV[1..14]"
 		(shape input)
-		(at 15.24 111.76 90)
+		(at 15.24 118.11 90)
 		(effects
 			(font
@@
 	(hierarchical_label "RST_DRV[1..14]"
 		(shape input)
-		(at 15.24 30.48 90)
-		(effects
-			(font
+		(at 15.24 36.83 90)
+		(effects
+			(font

Commit message: Fix photoMOS package and part, ethernet crystal
Signed-off-by: Lee Smet <lee.smet@hotmail.com>
Parts:
- K15, K16, K17, K18, K19, K20, K21, K22, K23, K24, K25, K26, K27, K28: value TLP176A -> TLP176AM; footprint Package_SO:SOP-4_3.8x4.1mm_P2.54mm -> Package_SO:SOIC-4_4.55x3.7mm_P2.54mm; symbol Relay_SolidState:CPC1017N -> granite:TLP176AM
Connections:
- net GND: now also K15.3, K16.3, K17.3, K18.3, K19.3, K20.3, K21.3, K22.3, K23.3, K24.3, K25.3, K26.3, K27.3, K28.3; no longer K15.2, K16.2, K17.2, K18.2, K19.2, K20.2, K21.2, K22.2, K23.2, K24.2, K25.2, K26.2, K27.2, K28.2
- net at R219.2: now also K19.4; no longer K19.3
- net at R224.2: now also K24.4; no longer K24.3
- net at J22.3 (Pin_3): now also K24.6; no longer K24.4
- net at J24.1 (Pin_1): now also K27.6; no longer K27.4
- net at J24.3 (Pin_3): now also K28.6; no longer K28.4
- net at J18.1 (Pin_1): now also K15.6; no longer K15.4
- net at J18.3 (Pin_3): now also K16.6; no longer K16.4
- net at R215.2: now also K15.4; no longer K15.3
- net at R223.2: now also K23.4; no longer K23.3
- net at R217.2: now also K17.4; no longer K17.3
- net at J19.1 (Pin_1): now also K17.6; no longer K17.4
- net at R221.2: now also K21.4; no longer K21.3
- net at J21.1 (Pin_1): now also K21.6; no longer K21.4
- net at R222.2: now also K22.4; no longer K22.3
- net at J23.1 (Pin_1): now also K25.6; no longer K25.4
- net at J23.3 (Pin_3): now also K26.6; no longer K26.4
- net at R227.2: now also K27.4; no longer K27.3
- net at R225.2: now also K25.4; no longer K25.3
- net at R228.2: now also K28.4; no longer K28.3
- net at J20.1 (Pin_1): now also K19.6; no longer K19.4
- net at J20.3 (Pin_3): now also K20.6; no longer K20.4
- net at J19.3 (Pin_3): now also K18.6; no longer K18.4
- net at R216.2: now also K16.4; no longer K16.3
- net at R226.2: now also K26.4; no longer K26.3
- net at R218.2: now also K18.4; no longer K18.3
- net at J21.3 (Pin_3): now also K22.6; no longer K22.4
- net at R220.2: now also K20.4; no longer K20.3
- net at J22.1 (Pin_1): now also K23.6; no longer K23.4
Other:
- note added: "Channels 8-14: 2x photoMOS contact closure (RESET, PWR BTN) per motherboard front-panel header. Floating outputs. TLP176AM: 3mA max trigger, ~6.2mA drive."
- note removed: "Channels 8-14: 2x photoMOS contact closure (RESET, PWR BTN) per motherboard front-panel header. Floating outputs. TLP176A: 3mA max trigger, ~6.5mA drive."

Commit message: Add manufacturer and MPN to schematic parts
Signed-off-by: Lee Smet <lee.smet@hotmail.com>
Parts:
- J18, J19, J20, J21, J22, J23, J24: MANUFACTURER (none) -> JST; MPN (none) -> B4B-PH-K-S(LF)(SN)
- K15, K16, K17, K18, K19, K20, K21, K22, K23, K24, K25, K26, K27, K28: MANUFACTURER (none) -> Toshiba; MPN (none) -> TLP176AM(TPL,E)
- R115, R116, R117, R118, R119, R120, R121, R122, R123, R124, R125, R126, R127, R128: MANUFACTURER (none) -> YAGEO; MPN (none) -> RC0402FR-07330RL
- R215, R216, R217, R218, R219, R220, R221, R222, R223, R224, R225, R226, R227, R228: MANUFACTURER (none) -> YAGEO; MPN (none) -> RC0603FR-07100RL
