File: schematic/relays.kicad_sch (KiCad schematic)
At the start: 60 parts, among them J11 MB01_FP, J12 MB02_FP, J13 MB03_FP, J14 MB04_FP, J15 MB05_FP, J16 MB06_FP, J17 MB07_FP, J18 MB08_FP, K1 TLP176AM, K10 TLP176AM, K11 TLP176AM, K12 TLP176AM, K13 TLP176AM, K14 TLP176AM, K15 TLP176AM, K16 TLP176AM, K2 TLP176AM, K3 TLP176AM, K4 TLP176AM, K5 TLP176AM, K6 TLP176AM, K7 TLP176AM, K8 TLP176AM, K9 TLP176AM, U14 MCP23017-E/SO

Commit message: Rev C: ESP32-C6 + W5500 controller for immersion
Schematic rework per docs/controller.md.

- MCU: ESP32-C6-MINI-1-N4 replaces STM32H563VIT6 (KiCad-stock
  module). EN/BOOT test pads, USB-C via the C6 USB Serial/JTAG with
  22R series resistors behind the existing USBLC6.
- Ethernet: W5500 over SPI replaces LAN8742A/RMII. PHY network,
  center taps, AVDD ferrite and LED wiring per WIZnet's W5500
  Ethernet Shield reference; ARJP11A magjack and PoE path unchanged.
- I2C split: internal bus (relay MCP23017, TMP1075) on HP I2C with
  its own expander reset (EXP_nRESET_INT, GPIO14); external bus to
  the header (software I2C on GPIO6/7) with EXP_nRESET (GPIO4,
  pulled low) and the shared EXP_INT.
- Expansion header J8 now 2x6: external I2C, reset, interrupt,
  GPIO5/8/15, fused 3V3/5V, all protected as before.
- C1/C2: KEMET T520 molded tantalum-polymer instead of rubber-sealed
  aluminium-polymer cans (immersion).
- Sheets regenerated: Power, Ethernet, MCU replace power_eth and
  mcu_usb; root and project net classes updated (RMII/SWD/RST
  classes removed). Board regenerated, nothing placed yet.
- Spec updated to the captured design.
Connections:
- net EXP_nRESET renamed EXP_nRESET_INT
- net I2C1_SCL renamed I2C_INT_SCL
- net I2C1_SDA renamed I2C_INT_SDA
Other:
- note added: "Channels 1-8: 2x photoMOS contact closure (RESET, PWR BTN) per motherboard front-panel header. Floating outputs. TLP176AM: 3mA max trigger, ~6mA drive. U14 MCP23017 @0x20 sources the LED current: GPA0-7 = PWR_DRV1-8, GPB0-7 = RST_DRV1-8 (GPA7/GPB7 are output-only). R32 holds U14 in reset unless the MCU drives EXP_nRESET_INT high: MCU reset/hang -> all GPIO Hi-Z -> all buttons released. U14 is on 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"
- note removed: "Channels 1-8: 2x photoMOS contact closure (RESET, PWR BTN) per motherboard front-panel header. Floating outputs. TLP176AM: 3mA max trigger, ~6mA drive. U14 MCP23017 @0x20 sources the LED current: GPA0-7 = PWR_DRV1-8, GPB0-7 = RST_DRV1-8 (GPA7/GPB7 are output-only). R32 holds U14 in reset unless the MCU drives EXP_nRESET high: MCU reset/hang -> all GPIO Hi-Z -> all buttons released. EXP_nRESET / E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"
Changed lines of the file:
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@@
 		(title "Granite Controller - Relay channels")
 		(date "2026-10-07")
-		(rev "B")
+		(rev "C")
 	)
 	(symbol
@@
 		)
 	)
-	(global_label "I2C1_SCL"
+	(global_label "I2C_INT_SCL"
 		(shape bidirectional)
 		(at 45.72 111.76 180)
@@
 		)
 	)
-	(global_label "I2C1_SDA"
+	(global_label "I2C_INT_SDA"
 		(shape bidirectional)
 		(at 45.72 114.3 180)
@@
 		)
 	)
-	(global_label "EXP_nRESET"
+	(global_label "EXP_nRESET_INT"
 		(shape bidirectional)
 		(at 45.72 134.62 180)
@@
 		)
 	)
-	(global_label "EXP_nRESET"
+	(global_label "EXP_nRESET_INT"
 		(shape bidirectional)
 		(at 25.4 158.75 90)
@@
 		)
 	)
-	(text "Channels 1-8: 2x photoMOS contact closure (RESET, PWR BTN) per motherboard front-panel header. Floating outputs.\nTLP176AM: 3mA max trigger, ~6mA drive. U14 MCP23017 @0x20 sources the LED current: GPA0-7 = PWR_DRV1-8, GPB0-7 = RST_DRV1-8 (GPA7/GPB7 are output-only).\nR32 holds U14 in reset unless the MCU drives EXP_nRESET high: MCU reset/hang -> all GPIO Hi-Z -> all buttons released.\nEXP_nRESET / EXP_INT are shared with extra MCP23017 modules on the expansion header (INT open-drain, mirrored)."
+	(text "Channels 1-8: 2x photoMOS contact closure (RESET, PWR BTN) per motherboard front-panel header. Floating outputs.\nTLP176AM: 3mA max trigger, ~6mA drive. U14 MCP23017 @0x20 sources the LED current: GPA0-7 = PWR_DRV1-8, GPB0-7 = RST_DRV1-8 (GPA7/GPB7 are output-only).\nR32 holds U14 in reset unless the MCU drives EXP_nRESET_INT high: MCU reset/hang -> all GPIO Hi-Z -> all buttons released.\nU14 is on the internal I2C bus with its own reset line; EXP_INT is shared with add-on modules on the expansion header (INT open-drain, mirrored)."
 		(exclude_from_sim no)
 		(at 228.6 50.8 0)
