File: schematic/relays.kicad_sch (KiCad schematic)
At the start: 60 parts, among them J11 MB01_FP, J12 MB02_FP, J13 MB03_FP, J14 MB04_FP, J15 MB05_FP, J16 MB06_FP, J17 MB07_FP, J18 MB08_FP, K1 TLP176AM, K10 TLP176AM, K11 TLP176AM, K12 TLP176AM, K13 TLP176AM, K14 TLP176AM, K15 TLP176AM, K16 TLP176AM, K2 TLP176AM, K3 TLP176AM, K4 TLP176AM, K5 TLP176AM, K6 TLP176AM, K7 TLP176AM, K8 TLP176AM, K9 TLP176AM, U14 MCP23017-E/SO

Commit message: Assign LCSC part numbers, mark PS1 DNP for JLC assembly
Every BOM line except PS1 now carries an LCSC field. Generic passives
move to JLC basic parts with equal or better ratings. Parts not stocked
at LCSC are swapped: C1/C2 to T520D227M010ATE018 (10 V), F1 to
0805L035/24XR, J8 to a generic gold 2x6 header, D6 to SMF3.3A.
PS1 (Ag9905MT) is DNP: bought separately and hand-soldered.
Parts:
- C38: LCSC (none) -> C1525; MANUFACTURER YAGEO -> Samsung Electro-Mechanics; MPN CC0402KRX7R7BB104 -> CL05B104KO5NNNC
- J11, J12, J13, J14, J15, J16, J17, J18: LCSC (none) -> C131334
- K1, K10, K11, K12, K13, K14, K15, K16, K2, K3, K4, K5, K6, K7, K8, K9: LCSC (none) -> C5370540
- R101, R102, R103, R104, R105, R106, R107, R108, R109, R110, R111, R112, R113, R114, R115, R116: LCSC (none) -> C25104; MANUFACTURER YAGEO -> UNI-ROYAL; MPN RC0402FR-07330RL -> 0402WGF3300TCE
- R201, R202, R203, R204, R205, R206, R207, R208, R209, R210, R211, R212, R213, R214, R215, R216: LCSC (none) -> C22775; MANUFACTURER YAGEO -> UNI-ROYAL; MPN RC0603FR-07100RL -> 0603WAF1000T5E
- R32, R33: LCSC (none) -> C25744
- U14: LCSC (none) -> C47023

Commit message: WROOM-1-N8, node power sensing, dry contacts, I2C port, VIN sense
- U1 ESP32-C6-MINI-1-N4 -> ESP32-C6-WROOM-1-N8 (8 MB for two OTA
  slots; N16 is a drop-in). Project-local symbol and footprint from the
  datasheet. GPIO14 is not on the WROOM: EXP_nRESET_INT moves to
  GPIO10; GPIO11 spare.
- Node connectors J11-J18 go to JST PH 5p: PWR_SW, RST_SW, node GND,
  PLED+, PLED-. PLED drives 2x TLP290-4 AC-input optos; 10k pull-ups
  -> U15 MCP23017 @0x21 GPA0-7 (NODE_ON1-8).
- U15 GPB0-3: 4 dry-contact inputs (J10, RC + TPD4E05U06 ESD).
- J9 I2C sensor port (JST PH 4p, Qwiic order) on the protected header bus.
- VIN_SENSE 100k/10k divider to GPIO5 (ADC); J8 pin 9 now unused.
Parts:
- removed J11: MB01_FP, Connector_JST:JST_PH_B4B-PH-K_1x04_P2.00mm_Vertical, symbol Connector_Generic:Conn_01x04
- removed J12: MB02_FP, Connector_JST:JST_PH_B4B-PH-K_1x04_P2.00mm_Vertical, symbol Connector_Generic:Conn_01x04
- removed J13: MB03_FP, Connector_JST:JST_PH_B4B-PH-K_1x04_P2.00mm_Vertical, symbol Connector_Generic:Conn_01x04
- removed J14: MB04_FP, Connector_JST:JST_PH_B4B-PH-K_1x04_P2.00mm_Vertical, symbol Connector_Generic:Conn_01x04
- removed J15: MB05_FP, Connector_JST:JST_PH_B4B-PH-K_1x04_P2.00mm_Vertical, symbol Connector_Generic:Conn_01x04
- removed J16: MB06_FP, Connector_JST:JST_PH_B4B-PH-K_1x04_P2.00mm_Vertical, symbol Connector_Generic:Conn_01x04
- removed J17: MB07_FP, Connector_JST:JST_PH_B4B-PH-K_1x04_P2.00mm_Vertical, symbol Connector_Generic:Conn_01x04
- removed J18: MB08_FP, Connector_JST:JST_PH_B4B-PH-K_1x04_P2.00mm_Vertical, symbol Connector_Generic:Conn_01x04
- added C46: 100n, Capacitor_SMD:C_0402_1005Metric, symbol Device:C
- added J11: MB01_FP, Connector_JST:JST_PH_B5B-PH-K_1x05_P2.00mm_Vertical, symbol Connector_Generic:Conn_01x05
- added J12: MB02_FP, Connector_JST:JST_PH_B5B-PH-K_1x05_P2.00mm_Vertical, symbol Connector_Generic:Conn_01x05
- added J13: MB03_FP, Connector_JST:JST_PH_B5B-PH-K_1x05_P2.00mm_Vertical, symbol Connector_Generic:Conn_01x05
- added J14: MB04_FP, Connector_JST:JST_PH_B5B-PH-K_1x05_P2.00mm_Vertical, symbol Connector_Generic:Conn_01x05
- added J15: MB05_FP, Connector_JST:JST_PH_B5B-PH-K_1x05_P2.00mm_Vertical, symbol Connector_Generic:Conn_01x05
- added J16: MB06_FP, Connector_JST:JST_PH_B5B-PH-K_1x05_P2.00mm_Vertical, symbol Connector_Generic:Conn_01x05
- added J17: MB07_FP, Connector_JST:JST_PH_B5B-PH-K_1x05_P2.00mm_Vertical, symbol Connector_Generic:Conn_01x05
- added J18: MB08_FP, Connector_JST:JST_PH_B5B-PH-K_1x05_P2.00mm_Vertical, symbol Connector_Generic:Conn_01x05
- added R39, R40, R41, R42, R43, R44, R45, R46: 10k, Resistor_SMD:R_0402_1005Metric, symbol Device:R
- added R47, R48, R49, R50, R51, R52, R53, R54: 220, Resistor_SMD:R_0402_1005Metric, symbol Device:R
- added U15: MCP23017-E/SO, Package_SO:SOIC-28W_7.5x17.9mm_P1.27mm, symbol Interface_Expansion:MCP23017x-x-SO
- added U16, U17: TLP290-4, Package_SO:SOP-16_4.55x10.3mm_P1.27mm, symbol Isolator:TLP290-4
Connections:
- net MB1_RST_A is gone; now on net MB1_COM: K1.6
- net MB2_RST_A is gone; now on net MB2_COM: K3.6
- net MB3_RST_A is gone; now on net MB3_COM: K5.6
- net MB4_RST_A is gone; now on net MB4_COM: K7.6
- net MB5_RST_A is gone; now on net MB5_COM: K9.6
- net MB6_RST_A is gone; now on net MB6_COM: K11.6
- net MB7_RST_A is gone; now on net MB7_COM: K13.6
- net MB8_RST_A is gone; now on net MB8_COM: K15.6
- net +3V3: now also C46.1, R39.1, R40.1, R41.1, R42.1, R43.1, R44.1, R45.1, R46.1, U15.15 (A0), U15.9 (V_{DD})
- net EXP_INT: now also U15.20 (INTA)
- net EXP_nRESET_INT: now also U15.18 (~{RESET})
- net GND: now also C46.2, U15.10 (V_{SS}), U15.16 (A1), U15.17 (A2), U16.11, U16.13, U16.15, U16.9, U17.11, U17.13, U17.15, U17.9
- net I2C_INT_SCL: now also U15.12 (SCK)
- net I2C_INT_SDA: now also U15.13 (SDA)
- net MB1_PWR_B: now also J11.1 (Pin_1)
- net MB1_RST_B: now also J11.2 (Pin_2)
- net MB2_PWR_B: now also J12.1 (Pin_1)
- net MB2_RST_B: now also J12.2 (Pin_2)
- net MB3_PWR_B: now also J13.1 (Pin_1)
- net MB3_RST_B: now also J13.2 (Pin_2)
- net MB4_PWR_B: now also J14.1 (Pin_1)
- net MB4_RST_B: now also J14.2 (Pin_2)
- net MB5_PWR_B: now also J15.1 (Pin_1)
- net MB5_RST_B: now also J15.2 (Pin_2)
- net MB6_PWR_B: now also J16.1 (Pin_1)
- net MB6_RST_B: now also J16.2 (Pin_2)
- net MB7_PWR_B: now also J17.1 (Pin_1)
- net MB7_RST_B: now also J17.2 (Pin_2)
- net MB8_PWR_B: now also J18.1 (Pin_1)
- net MB8_RST_B: now also J18.2 (Pin_2)
- net MB1_PWR_A renamed MB1_COM
- net MB1_COM: now also J11.3 (Pin_3)
- net MB2_PWR_A renamed MB2_COM
- net MB2_COM: now also J12.3 (Pin_3)
- net MB3_PWR_A renamed MB3_COM
- net MB3_COM: now also J13.3 (Pin_3)
- net MB4_PWR_A renamed MB4_COM
- net MB4_COM: now also J14.3 (Pin_3)
- net MB5_PWR_A renamed MB5_COM
- net MB5_COM: now also J15.3 (Pin_3)
- net MB6_PWR_A renamed MB6_COM
- net MB6_COM: now also J16.3 (Pin_3)
- net MB7_PWR_A renamed MB7_COM
- net MB7_COM: now also J17.3 (Pin_3)
- net MB8_PWR_A renamed MB8_COM
- net MB8_COM: now also J18.3 (Pin_3)
- new net: R51.2, U17.1
- new net: R47.2, U16.1
- new net: R54.2, U17.7
- new net: R50.2, U16.7
- new net: R52.2, U17.3
- new net: R49.2, U16.5
- new net: R48.2, U16.3
- new net: R53.2, U17.5
- new net DRY_IN1: U15.1 (GPB0)
- new net DRY_IN2: U15.2 (GPB1)
- new net DRY_IN3: U15.3 (GPB2)
- new net DRY_IN4: U15.4 (GPB3)
- new net MB1_PLED_N: J11.5 (Pin_5), U16.2
- new net MB1_PLED_P: J11.4 (Pin_4), R47.1
- new net MB2_PLED_N: J12.5 (Pin_5), U16.4
- new net MB2_PLED_P: J12.4 (Pin_4), R48.1
- new net MB3_PLED_N: J13.5 (Pin_5), U16.6
- new net MB3_PLED_P: J13.4 (Pin_4), R49.1
- new net MB4_PLED_N: J14.5 (Pin_5), U16.8
- new net MB4_PLED_P: J14.4 (Pin_4), R50.1
- new net MB5_PLED_N: J15.5 (Pin_5), U17.2
- new net MB5_PLED_P: J15.4 (Pin_4), R51.1
- new net MB6_PLED_N: J16.5 (Pin_5), U17.4
- new net MB6_PLED_P: J16.4 (Pin_4), R52.1
- new net MB7_PLED_N: J17.5 (Pin_5), U17.6
- new net MB7_PLED_P: J17.4 (Pin_4), R53.1
- new net MB8_PLED_N: J18.5 (Pin_5), U17.8
- new net MB8_PLED_P: J18.4 (Pin_4), R54.1
- new net NODE_ON1: R39.2, U15.21 (GPA0), U16.16
- new net NODE_ON2: R40.2, U15.22 (GPA1), U16.14
- new net NODE_ON3: R41.2, U15.23 (GPA2), U16.12
- new net NODE_ON4: R42.2, U15.24 (GPA3), U16.10
- new net NODE_ON5: R43.2, U15.25 (GPA4), U17.16
- new net NODE_ON6: R44.2, U15.26 (GPA5), U17.14
- new net NODE_ON7: R45.2, U15.27 (GPA6), U17.12
- new net NODE_ON8: R46.2, U15.28 (GPA7), U17.10
- no-connect marks 1 -> 8
Other:
- note added: "Channels 1-8: 2x photoMOS contact closure (RESET, PWR BTN) per motherboard front-panel header. Floating outputs. TLP176AM: 3mA max trigger, ~6mA drive. U14 MCP23017 @0x20 sources the LED current: GPA0-7 = PWR_DRV1-8, GPB0-7 = RST_DRV1-8 (GPA7/GPB7 are output-only). R32 holds U14 and U15 in reset unless the MCU drives EXP_nRESET_INT high: MCU reset/hang -> all GPIO Hi-Z -> all buttons released. U1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"
- note added: "Node connector J11-J18 (JST PH 5p): 1 PWR_SW, 2 RST_SW, 3 node GND (common return of both buttons), 4 PLED+, 5 PLED-. PLED sense: TLP290-4 (AC input, either polarity), 220R in series with the node's own LED resistor, 10k pull-up -> NODE_ONn low = node power LED lit. U15 MCP23017 @0x21: GPA0-7 = NODE_ON1-8, GPB0-3 = DRY_IN1-4 (expansion sheet), GPB4-7 spare."
- note removed: "Channels 1-8: 2x photoMOS contact closure (RESET, PWR BTN) per motherboard front-panel header. Floating outputs. TLP176AM: 3mA max trigger, ~6mA drive. U14 MCP23017 @0x20 sources the LED current: GPA0-7 = PWR_DRV1-8, GPB0-7 = RST_DRV1-8 (GPA7/GPB7 are output-only). R32 holds U14 in reset unless the MCU drives EXP_nRESET_INT high: MCU reset/hang -> all GPIO Hi-Z -> all buttons released. U14 is on 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"

Commit message: Fix the 2026-10 review findings
Schematic: NODE_ON8 to U15 GPB4 (GPA7 is output-only), F3 1206L075/33NR,
VBUS bleeder R65/C52, R38 12.4k (BUCK_5V 5.44 V), D9 SMAJ6.0A crowbar on
BUCK_5V, R101-R116 270R, C26/C27 15 pF, R39-R46 47k, D6 value.

Layout: hole-clearance rule with units (0.3 mm) and 6.5 mm keep-outs at
H1-H4, EN RC / decoupling / VIN_SENSE filter at U1, no F.Cu under the
module body, vias kept off the U1 EPAD, zones 1 mm from the short edges
for mouse-bite rails, silk 1.0/0.15 mm, autorouter vias moved out of
SMD pads (only the U1 pad 29 thermal vias remain).

tools/jlcfab.py: per-footprint rotation/centroid corrections checked
against EasyEDA footprints (K*, U2, U8, JST fixed; U1, J2 offsets), no
drill maps in the zip. Docs: controller.md, handoff, review status.

ERC 0; DRC 0 unconnected, 0 parity, 3 known violations.
Parts:
- R101, R102, R103, R104, R105, R106, R107, R108, R109, R110, R111, R112, R113, R114, R115, R116: value 330 -> 270; LCSC C25104 -> C2909342; MANUFACTURER UNI-ROYAL -> FOJAN; MPN 0402WGF3300TCE -> FRC0402F2700TS
- R39, R40, R41, R42, R43, R44, R45, R46: value 10k -> 47k; LCSC C25744 -> C25792; MPN 0402WGF1002TCE -> 0402WGF4702TCE
Connections:
- net NODE_ON8: now also U15.5 (GPB4); no longer U15.28 (GPA7)
Other:
- note added: "Channels 1-8: 2x photoMOS contact closure (RESET, PWR BTN) per motherboard front-panel header. Floating outputs. TLP176AM: 3mA max trigger, ~6.5mA drive (270R). U14 MCP23017 @0x20 sources the LED current: GPA0-7 = PWR_DRV1-8, GPB0-7 = RST_DRV1-8 (GPA7/GPB7 are output-only). R32 holds U14 and U15 in reset unless the MCU drives EXP_nRESET_INT high: MCU reset/hang -> all GPIO Hi-Z -> all buttons rel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"
- note added: "Node connector J11-J18 (JST PH 5p): 1 PWR_SW, 2 RST_SW, 3 node GND (common return of both buttons), 4 PLED+, 5 PLED-. PLED sense: TLP290-4 (AC input, either polarity), 220R in series with the node's own LED resistor, 47k pull-up -> NODE_ONn low = node power LED lit. U15 MCP23017 @0x21: GPA0-6 = NODE_ON1-7, GPB4 = NODE_ON8 (GPA7 is output-only), GPB0-3 = DRY_IN1-4 (expansion sheet), GPB5-7 spare."
- note removed: "Channels 1-8: 2x photoMOS contact closure (RESET, PWR BTN) per motherboard front-panel header. Floating outputs. TLP176AM: 3mA max trigger, ~6mA drive. U14 MCP23017 @0x20 sources the LED current: GPA0-7 = PWR_DRV1-8, GPB0-7 = RST_DRV1-8 (GPA7/GPB7 are output-only). R32 holds U14 and U15 in reset unless the MCU drives EXP_nRESET_INT high: MCU reset/hang -> all GPIO Hi-Z -> all buttons released. U1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"
- note removed: "Node connector J11-J18 (JST PH 5p): 1 PWR_SW, 2 RST_SW, 3 node GND (common return of both buttons), 4 PLED+, 5 PLED-. PLED sense: TLP290-4 (AC input, either polarity), 220R in series with the node's own LED resistor, 10k pull-up -> NODE_ONn low = node power LED lit. U15 MCP23017 @0x21: GPA0-7 = NODE_ON1-8, GPB0-3 = DRY_IN1-4 (expansion sheet), GPB4-7 spare."
