File: schematic/expansion.kicad_sch (KiCad schematic)
At the start: 9 parts, among them J8 EXPANSION, U6 TPD4E05U06DQA, U7 TPD4E05U06DQA

Commit message: Assign LCSC part numbers, mark PS1 DNP for JLC assembly
Every BOM line except PS1 now carries an LCSC field. Generic passives
move to JLC basic parts with equal or better ratings. Parts not stocked
at LCSC are swapped: C1/C2 to T520D227M010ATE018 (10 V), F1 to
0805L035/24XR, J8 to a generic gold 2x6 header, D6 to SMF3.3A.
PS1 (Ag9905MT) is DNP: bought separately and hand-soldered.
Parts:
- D6: LCSC (none) -> C37331473; MANUFACTURER Littelfuse -> GOODWORK; MPN SMF3.3 -> SMF3.3A
- D7: LCSC (none) -> C151296
- F1: LCSC (none) -> C7472565; MANUFACTURER Bourns -> LUTE; MPN MF-PSMF035X-2 -> 0805L035/24XR
- F2: LCSC (none) -> C151162; MPN 1206L050/15YR-A -> 1206L050/15YR
- J8: LCSC (none) -> C7501277; MANUFACTURER Samtec -> Megastar; MPN TSW-106-07-G-D -> ZX-PZ2.54-2-6PZZ
- RN1, RN2: LCSC (none) -> C43557; MANUFACTURER YAGEO -> UNI-ROYAL; MPN YC124-JR-07330RL -> 4D02WGJ0331TCE
- U6, U7: LCSC (none) -> C138714
Changed lines of the file:
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@@
 			)
 		)
-		(property "MANUFACTURER" "YAGEO"
+		(property "MANUFACTURER" "UNI-ROYAL"
 			(at 55.88 50.8 0)
 			(hide yes)
@@
 			)
 		)
-		(property "MPN" "YC124-JR-07330RL"
+		(property "MPN" "4D02WGJ0331TCE"
+			(at 55.88 50.8 0)
+			(hide yes)
+			(show_name no)
+			(do_not_autoplace no)
+			(effects
+				(font
+					(size 1.27 1.27)
+				)
+			)
+		)
+		(property "LCSC" "C43557"
 			(at 55.88 50.8 0)
 			(hide yes)
@@
 			)
 		)
+		(property "LCSC" "C138714"
+			(at 127 55.88 0)
+			(hide yes)
+			(show_name no)
+			(do_not_autoplace no)
+			(effects
+				(font
+					(size 1.27 1.27)
+				)
+			)
+		)
 		(pin "1"
 		)
@@
 			)
 		)
-		(property "MANUFACTURER" "YAGEO"
+		(property "MANUFACTURER" "UNI-ROYAL"
 			(at 55.88 83.82 0)
 			(hide yes)
@@
 			)
 		)
-		(property "MPN" "YC124-JR-07330RL"
+		(property "MPN" "4D02WGJ0331TCE"
+			(at 55.88 83.82 0)
+			(hide yes)
+			(show_name no)
+			(do_not_autoplace no)
+			(effects
+				(font
+					(size 1.27 1.27)
+				)
+			)
+		)
+		(property "LCSC" "C43557"
 			(at 55.88 83.82 0)
 			(hide yes)
@@
 			)
 		)
+		(property "LCSC" "C138714"
+			(at 127 88.9 0)
+			(hide yes)
+			(show_name no)
+			(do_not_autoplace no)
+			(effects
+				(font
+					(size 1.27 1.27)
+				)
+			)
+		)
 		(pin "1"
 		)
@@
 			)
 		)
-		(property "MANUFACTURER" "Samtec"
+		(property "MANUFACTURER" "Megastar"
 			(at 187.96 66.04 0)
 			(hide yes)
@@
 			)
 		)
-		(property "MPN" "TSW-106-07-G-D"
+		(property "MPN" "ZX-PZ2.54-2-6PZZ"
+			(at 187.96 66.04 0)
+			(hide yes)
+			(show_name no)
+			(do_not_autoplace no)
+			(effects
+				(font
+					(size 1.27 1.27)
+				)
+			)
+		)
+		(property "LCSC" "C7501277"
 			(at 187.96 66.04 0)
 			(hide yes)
@@
 			)
 		)
-		(property "MANUFACTURER" "Bourns"
+		(property "MANUFACTURER" "LUTE"
 			(at 35.56 121.92 0)
 			(hide yes)
@@
 			)
 		)
-		(property "MPN" "MF-PSMF035X-2"
+		(property "MPN" "0805L035/24XR"
+			(at 35.56 121.92 0)
+			(hide yes)
+			(show_name no)
+			(do_not_autoplace no)
+			(effects
+				(font
+					(size 1.27 1.27)
+				)
+			)
+		)
+		(property "LCSC" "C7472565"
 			(at 35.56 121.92 0)
 			(hide yes)
@@
 			)
 		)
-		(property "MANUFACTURER" "Littelfuse"
+		(property "MANUFACTURER" "GOODWORK"
 			(at 45.72 125.73 0)
 			(hide yes)
@@
 			)
 		)
-		(property "MPN" "SMF3.3"
+		(property "MPN" "SMF3.3A"
+			(at 45.72 125.73 0)
+			(hide yes)
+			(show_name no)
+			(do_not_autoplace no)
+			(effects
+				(font
+					(size 1.27 1.27)
+				)
+			)
+		)
+		(property "LCSC" "C37331473"
 			(at 45.72 125.73 0)
 			(hide yes)
@@
 			)
 		)
-		(property "MPN" "1206L050/15YR-A"
+		(property "MPN" "1206L050/15YR"
+			(at 35.56 142.24 0)
+			(hide yes)
+			(show_name no)
+			(do_not_autoplace no)
+			(effects
+				(font
+					(size 1.27 1.27)
+				)
+			)
+		)
+		(property "LCSC" "C151162"
 			(at 35.56 142.24 0)
 			(hide yes)
@@
 			(at 45.72 146.05 0)
 			(hide yes)
+			(show_name no)
+			(do_not_autoplace no)
+			(effects
+				(font
+					(size 1.27 1.27)
+				)
+			)
+		)
+		(property "LCSC" "C151296"
+			(at 45.72 146.05 0)
+			(hide yes)

Commit message: WROOM-1-N8, node power sensing, dry contacts, I2C port, VIN sense
- U1 ESP32-C6-MINI-1-N4 -> ESP32-C6-WROOM-1-N8 (8 MB for two OTA
  slots; N16 is a drop-in). Project-local symbol and footprint from the
  datasheet. GPIO14 is not on the WROOM: EXP_nRESET_INT moves to
  GPIO10; GPIO11 spare.
- Node connectors J11-J18 go to JST PH 5p: PWR_SW, RST_SW, node GND,
  PLED+, PLED-. PLED drives 2x TLP290-4 AC-input optos; 10k pull-ups
  -> U15 MCP23017 @0x21 GPA0-7 (NODE_ON1-8).
- U15 GPB0-3: 4 dry-contact inputs (J10, RC + TPD4E05U06 ESD).
- J9 I2C sensor port (JST PH 4p, Qwiic order) on the protected header bus.
- VIN_SENSE 100k/10k divider to GPIO5 (ADC); J8 pin 9 now unused.
Parts:
- added C47, C48, C49, C50: 100n, Capacitor_SMD:C_0402_1005Metric, symbol Device:C
- added J10: DRY_IN, Connector_JST:JST_PH_B5B-PH-K_1x05_P2.00mm_Vertical, symbol Connector_Generic:Conn_01x05
- added J9: I2C_SENSOR, Connector_JST:JST_PH_B4B-PH-K_1x04_P2.00mm_Vertical, symbol Connector_Generic:Conn_01x04
- added R55, R56, R57, R58: 1k, Resistor_SMD:R_0402_1005Metric, symbol Device:R
- added R59, R60, R61, R62: 10k, Resistor_SMD:R_0402_1005Metric, symbol Device:R
- added U18: TPD4E05U06DQA, Package_SON:USON-10_2.5x1.0mm_P0.5mm, symbol Power_Protection:TPD4E05U06DQA
Connections:
- net +3V3: now also R59.1, R60.1, R61.1, R62.1
- net GND: now also C47.2, C48.2, C49.2, C50.2, J10.5 (Pin_5), J9.1 (Pin_1), U18.3 (GND), U18.8 (GND)
- net HDR_3V3: now also J9.2 (Pin_2)
- net HDR_SCL: now also J9.4 (Pin_4)
- net HDR_SDA: now also J9.3 (Pin_3)
- net GPIO_IO5: no longer names the net of RN2.8 (R1.2)
- new net DRYC1: J10.1 (Pin_1), R55.2, R59.2, U18.1 (D1+)
- new net DRYC2: J10.2 (Pin_2), R56.2, R60.2, U18.2 (D1-)
- new net DRYC3: J10.3 (Pin_3), R57.2, R61.2, U18.4 (D2+)
- new net DRYC4: J10.4 (Pin_4), R58.2, R62.2, U18.5 (D2-)
- new net DRY_IN1: C47.1, R55.1
- new net DRY_IN2: C48.1, R56.1
- new net DRY_IN3: C49.1, R57.1
- new net DRY_IN4: C50.1, R58.1
- no-connect marks 11 -> 16
Other:
- note added: "Dry-contact inputs (leak / level float / lid switch): contact to GND. 10k pull-up, 1k + 100n RC, TPD4E05U06 ESD, J10 JST PH 5p (1-4 IN, 5 GND) -> U15 GPB0-3."
- note added: "J9 I2C sensor port (JST PH 4p, Qwiic pin order): GND, 3V3, SDA, SCL on the protected header bus (same 330R + ESD + PTC as J8)."

Commit message: Fix the 2026-10 review findings
Schematic: NODE_ON8 to U15 GPB4 (GPA7 is output-only), F3 1206L075/33NR,
VBUS bleeder R65/C52, R38 12.4k (BUCK_5V 5.44 V), D9 SMAJ6.0A crowbar on
BUCK_5V, R101-R116 270R, C26/C27 15 pF, R39-R46 47k, D6 value.

Layout: hole-clearance rule with units (0.3 mm) and 6.5 mm keep-outs at
H1-H4, EN RC / decoupling / VIN_SENSE filter at U1, no F.Cu under the
module body, vias kept off the U1 EPAD, zones 1 mm from the short edges
for mouse-bite rails, silk 1.0/0.15 mm, autorouter vias moved out of
SMD pads (only the U1 pad 29 thermal vias remain).

tools/jlcfab.py: per-footprint rotation/centroid corrections checked
against EasyEDA footprints (K*, U2, U8, JST fixed; U1, J2 offsets), no
drill maps in the zip. Docs: controller.md, handoff, review status.

ERC 0; DRC 0 unconnected, 0 parity, 3 known violations.
Parts:
- D6: value SMF3.3 -> SMF3.3A
Changed lines of the file:
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@@
 			)
 		)
-		(property "Value" "SMF3.3"
+		(property "Value" "SMF3.3A"
 			(at 48.26 127 90)
 			(show_name no)
