File: granite_controller.kicad_pcb (KiCad board)
At the start: 4 copper layers, 183 parts, among them J1 ARJP11A-MASA-B-A-EMU2, J11 MB01_FP, J12 MB02_FP, J13 MB03_FP, J14 MB04_FP, J15 MB05_FP, J16 MB06_FP, J17 MB07_FP, J18 MB08_FP, J19 MB09_FP, J2 USB4105-xx-A, J20 MB10_FP, J21 MB11_FP, J22 MB12_FP, J23 MB13_FP, J24 MB14_FP, J3 TC2030-IDC-NL, J4 1WIRE, J5 1WIRE, J6 1WIRE, J7 1WIRE, K1 TLP176AM, K10 TLP176AM, K11 TLP176AM, K12 TLP176AM, K13 TLP176AM, K14 TLP176AM, K15 TLP176AM, K16 TLP176AM, K17 TLP176AM, K18 TLP176AM, K19 TLP176AM, K2 TLP176AM, K20 TLP176AM, K21 TLP176AM, K22 TLP176AM, K23 TLP176AM, K24 TLP176AM, K25 TLP176AM, K26 TLP176AM, K27 TLP176AM, K28 TLP176AM, K3 TLP176AM, K4 TLP176AM, K5 TLP176AM, K6 TLP176AM, K7 TLP176AM, K8 TLP176AM, K9 TLP176AM, U1 STM32H563VIT6, U2 TLV62569DBV, U3 LAN8742A, U4 USBLC6-2SC6, U5 TMP1075D, Y1 25MHz ABM8G, Y2 25MHz 12pF YXC

Commit message: Add protected GPIO expansion header
New sheet 'Expansion header' with J8, a 2x18 2.54 mm header (DNP),
bringing out the 28 spare U1 GPIOs plus I2C1, 3V3 and 5V.

- Each signal: 330R series resistor (4x0402 array, MCU side) and a
  TPD4E05U06 ESD clamp at the header pin.
- 3V3 and 5V header pins: PTC fuse plus a TVS to GND.
- PC13-PC15 stay unconnected (backup domain, LSE).
- U1 spare pins labelled GPIO_<pin>; the I2C1 labels on U1 became
  global so the header can reach the bus. Net class patterns added
  for I2C1_*, HDR_3V3 and HDR_5V.
- Board regenerated from the netlist (nothing was placed yet).
Parts:
- added D6: SMF3.3, Diode_SMD:D_SOD-123F, F.Cu at (-40.0, 0.00)
- added D7: SMF5.0A, Diode_SMD:D_SOD-123F, F.Cu at (-26.0, 0.00)
- added F1: PTC 350mA, Fuse:Fuse_0805_2012Metric, F.Cu at (-12.0, 0.00)
- added F2: PTC 500mA, Fuse:Fuse_1206_3216Metric, F.Cu at (2.00, 0.00)
- added J8: EXPANSION, Connector_PinHeader_2.54mm:PinHeader_2x18_P2.54mm_Vertical, F.Cu at (16.0, 0.00)
- added RN1: 4x330, Resistor_SMD:R_Array_Convex_4x0402, F.Cu at (30.0, 0.00)
- added RN2: 4x330, Resistor_SMD:R_Array_Convex_4x0402, F.Cu at (-40.0, 14.0)
- added RN3: 4x330, Resistor_SMD:R_Array_Convex_4x0402, F.Cu at (-26.0, 14.0)
- added RN4: 4x330, Resistor_SMD:R_Array_Convex_4x0402, F.Cu at (-12.0, 14.0)
- added RN5: 4x330, Resistor_SMD:R_Array_Convex_4x0402, F.Cu at (2.00, 14.0)
- added RN6: 4x330, Resistor_SMD:R_Array_Convex_4x0402, F.Cu at (16.0, 14.0)
- added RN7: 4x330, Resistor_SMD:R_Array_Convex_4x0402, F.Cu at (30.0, 14.0)
- added RN8: 4x330, Resistor_SMD:R_Array_Convex_4x0402, F.Cu at (-40.0, 28.0)
- added U10: TPD4E05U06DQA, Package_SON:USON-10_2.5x1.0mm_P0.5mm, F.Cu at (30.0, 28.0)
- added U11: TPD4E05U06DQA, Package_SON:USON-10_2.5x1.0mm_P0.5mm, F.Cu at (-40.0, 42.0)
- added U12: TPD4E05U06DQA, Package_SON:USON-10_2.5x1.0mm_P0.5mm, F.Cu at (-26.0, 42.0)
- added U13: TPD4E05U06DQA, Package_SON:USON-10_2.5x1.0mm_P0.5mm, F.Cu at (-12.0, 42.0)
- added U6: TPD4E05U06DQA, Package_SON:USON-10_2.5x1.0mm_P0.5mm, F.Cu at (-26.0, 28.0)
- added U7: TPD4E05U06DQA, Package_SON:USON-10_2.5x1.0mm_P0.5mm, F.Cu at (-12.0, 28.0)
- added U8: TPD4E05U06DQA, Package_SON:USON-10_2.5x1.0mm_P0.5mm, F.Cu at (2.00, 28.0)
- added U9: TPD4E05U06DQA, Package_SON:USON-10_2.5x1.0mm_P0.5mm, F.Cu at (16.0, 28.0)
Connections:
- net /MCU and USB/I2C1_SCL renamed I2C1_SCL
- net /MCU and USB/I2C1_SDA renamed I2C1_SDA
- U1 pad 15: unconnected-(U1-PC0-Pad15) -> GPIO_PC0
- U1 pad 17: unconnected-(U1-PC2-Pad17) -> GPIO_PC2
- U1 pad 18: unconnected-(U1-PC3-Pad18) -> GPIO_PC3
- U1 pad 23: unconnected-(U1-PA0-Pad23) -> GPIO_PA0
- U1 pad 26: unconnected-(U1-PA3-Pad26) -> GPIO_PA3
- U1 pad 29: unconnected-(U1-PA4-Pad29) -> GPIO_PA4
- U1 pad 31: unconnected-(U1-PA6-Pad31) -> GPIO_PA6
- U1 pad 36: unconnected-(U1-PB1-Pad36) -> GPIO_PB1
- U1 pad 37: unconnected-(U1-PB2-Pad37) -> GPIO_PB2
- U1 pad 47: unconnected-(U1-PB10-Pad47) -> GPIO_PB10
- U1 pad 52: unconnected-(U1-PB13-Pad52) -> GPIO_PB13
- U1 pad 53: unconnected-(U1-PB14-Pad53) -> GPIO_PB14
- U1 pad 61: unconnected-(U1-PD14-Pad61) -> GPIO_PD14
- U1 pad 62: unconnected-(U1-PD15-Pad62) -> GPIO_PD15
- U1 pad 63: unconnected-(U1-PC6-Pad63) -> GPIO_PC6
- U1 pad 64: unconnected-(U1-PC7-Pad64) -> GPIO_PC7
- U1 pad 65: unconnected-(U1-PC8-Pad65) -> GPIO_PC8
- U1 pad 66: unconnected-(U1-PC9-Pad66) -> GPIO_PC9
- U1 pad 67: unconnected-(U1-PA8-Pad67) -> GPIO_PA8
- U1 pad 69: unconnected-(U1-PA10-Pad69) -> GPIO_PA10
- U1 pad 77: unconnected-(U1-PA15(JTDI)-Pad77) -> GPIO_PA15
- U1 pad 78: unconnected-(U1-PC10-Pad78) -> GPIO_PC10
- U1 pad 79: unconnected-(U1-PC11-Pad79) -> GPIO_PC11
- U1 pad 80: unconnected-(U1-PC12-Pad80) -> GPIO_PC12
- U1 pad 90: unconnected-(U1-PB4(NJTRST)-Pad90) -> GPIO_PB4
- U1 pad 95: unconnected-(U1-PB8-Pad95) -> GPIO_PB8
- U1 pad 96: unconnected-(U1-PB9-Pad96) -> GPIO_PB9
- U1 pad 97: unconnected-(U1-PE0-Pad97) -> GPIO_PE0

Commit message: Rework for 8 nodes with MCP23017 relay drive
Target is now 8 motherboards per frame (was 14 in the schematic).

- relays_a/relays_b (14 channels, 28 photoMOS) replaced by one
  'Relay channels' sheet: 8 channels, 16 TLP176AM, J11-J18, same
  per-channel circuit and parts.
- U14 MCP23017 @0x20 drives the LEDs: GPA0-7 = PWR_DRV1-8,
  GPB0-7 = RST_DRV1-8. R32 pulls EXP_nRESET low so U14 stays in
  reset (all buttons released) unless the MCU drives it; R33 pulls
  up the shared open-drain EXP_INT.
- MCU: the two 14-bit drive buses are gone; PE2 = EXP_nRESET,
  PE3 = EXP_INT, the other 26 freed pins are no-connect.
- Expansion header J8 grows to 2x20 and carries I2C1, EXP_nRESET
  and EXP_INT (pins 5-8) for extra expander modules or a later
  power board, plus 3V3/5V on both ends.
- Net classes for the second relay bank removed; drive patterns
  point at the new sheet. Board regenerated (nothing placed).
Parts:
- removed J19: MB09_FP, Connector_JST:JST_PH_B4B-PH-K_1x04_P2.00mm_Vertical
- removed J20: MB10_FP, Connector_JST:JST_PH_B4B-PH-K_1x04_P2.00mm_Vertical
- removed J21: MB11_FP, Connector_JST:JST_PH_B4B-PH-K_1x04_P2.00mm_Vertical
- removed J22: MB12_FP, Connector_JST:JST_PH_B4B-PH-K_1x04_P2.00mm_Vertical
- removed J23: MB13_FP, Connector_JST:JST_PH_B4B-PH-K_1x04_P2.00mm_Vertical
- removed J24: MB14_FP, Connector_JST:JST_PH_B4B-PH-K_1x04_P2.00mm_Vertical
- removed K17, K18, K19, K20, K21, K22, K23, K24, K25, K26, K27, K28: TLP176AM, Package_SO:SOIC-4_4.55x3.7mm_P2.54mm
- removed R117, R118, R119, R120, R121, R122, R123, R124, R125, R126, R127, R128: 330, Resistor_SMD:R_0402_1005Metric
- removed R217, R218, R219, R220, R221, R222, R223, R224, R225, R226, R227, R228: 100, Resistor_SMD:R_0603_1608Metric
- added C38: 100n, Capacitor_SMD:C_0402_1005Metric, F.Cu at (-220.0, 0.00)
- added R32: 10k, Resistor_SMD:R_0402_1005Metric, F.Cu at (-206.0, 56.0)
- added R33: 10k, Resistor_SMD:R_0402_1005Metric, F.Cu at (-192.0, 56.0)
- added U14: MCP23017-E/SO, Package_SO:SOIC-28W_7.5x17.9mm_P1.27mm, F.Cu at (-150.0, 126.0)
- J8: footprint Connector_PinHeader_2.54mm:PinHeader_2x18_P2.54mm_Vertical -> Connector_PinHeader_2.54mm:PinHeader_2x20_P2.54mm_Vertical
- moved R116 156.4 mm to (-220.0, 98.0)
- moved R215 130.6 mm to (-178.0, 126.0)
- moved K16 125.3 mm to (-220.0, 56.0)
- moved D6 90.0 mm to (-130.0, 0.00)
- moved D7 90.0 mm to (-116.0, 0.00)
- moved F1 90.0 mm to (-102.0, 0.00)
- moved F2 90.0 mm to (-88.0, 0.00)
- moved J8 90.0 mm to (-74.0, 0.00)
- moved RN1 90.0 mm to (-60.0, 0.00)
- moved RN2 90.0 mm to (-130.0, 14.0)
- moved RN3 90.0 mm to (-116.0, 14.0)
- moved RN4 90.0 mm to (-102.0, 14.0)
- moved RN5 90.0 mm to (-88.0, 14.0)
- moved RN6 90.0 mm to (-74.0, 14.0)
- moved RN7 90.0 mm to (-60.0, 14.0)
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Connections:
- net Net-(J11-Pin_1) renamed /Relay channels/MB1_RST_A
- net Net-(J11-Pin_3) renamed /Relay channels/MB1_PWR_A
- net Net-(J12-Pin_1) renamed /Relay channels/MB2_RST_A
- net Net-(J12-Pin_3) renamed /Relay channels/MB2_PWR_A
- net Net-(J13-Pin_1) renamed /Relay channels/MB3_RST_A
- net Net-(J13-Pin_3) renamed /Relay channels/MB3_PWR_A
- net Net-(J14-Pin_1) renamed /Relay channels/MB4_RST_A
- net Net-(J14-Pin_3) renamed /Relay channels/MB4_PWR_A
- net Net-(J15-Pin_1) renamed /Relay channels/MB5_RST_A
- net Net-(J15-Pin_3) renamed /Relay channels/MB5_PWR_A
- net Net-(J16-Pin_1) renamed /Relay channels/MB6_RST_A
- net Net-(J16-Pin_3) renamed /Relay channels/MB6_PWR_A
- net Net-(J17-Pin_1) renamed /Relay channels/MB7_RST_A
- net Net-(J17-Pin_3) renamed /Relay channels/MB7_PWR_A
- net Net-(J18-Pin_1) renamed /Relay channels/MB8_RST_A
- net Net-(J18-Pin_3) renamed /Relay channels/MB8_PWR_A
- J11 pad 2: Net-(J11-Pin_2) -> /Relay channels/MB1_RST_B
- J11 pad 4: Net-(J11-Pin_4) -> /Relay channels/MB1_PWR_B
- J12 pad 2: Net-(J12-Pin_2) -> /Relay channels/MB2_RST_B
- J12 pad 4: Net-(J12-Pin_4) -> /Relay channels/MB2_PWR_B
- J13 pad 2: Net-(J13-Pin_2) -> /Relay channels/MB3_RST_B
- J13 pad 4: Net-(J13-Pin_4) -> /Relay channels/MB3_PWR_B
- J14 pad 2: Net-(J14-Pin_2) -> /Relay channels/MB4_RST_B
- J14 pad 4: Net-(J14-Pin_4) -> /Relay channels/MB4_PWR_B
- J15 pad 2: Net-(J15-Pin_2) -> /Relay channels/MB5_RST_B
- J15 pad 4: Net-(J15-Pin_4) -> /Relay channels/MB5_PWR_B
- J16 pad 2: Net-(J16-Pin_2) -> /Relay channels/MB6_RST_B
- J16 pad 4: Net-(J16-Pin_4) -> /Relay channels/MB6_PWR_B
- J17 pad 2: Net-(J17-Pin_2) -> /Relay channels/MB7_RST_B
- J17 pad 4: Net-(J17-Pin_4) -> /Relay channels/MB7_PWR_B
- J18 pad 2: Net-(J18-Pin_2) -> /Relay channels/MB8_RST_B
- J18 pad 4: Net-(J18-Pin_4) -> /Relay channels/MB8_PWR_B
- J8 pad 10: /Expansion header/HDR_PC0 -> /Expansion header/HDR_PA3
- J8 pad 11: /Expansion header/HDR_PC2 -> /Expansion header/HDR_PA4
- J8 pad 12: /Expansion header/HDR_PC3 -> /Expansion header/HDR_PA6
- J8 pad 13: /Expansion header/HDR_PC6 -> /Expansion header/HDR_PB1
- J8 pad 14: /Expansion header/HDR_PC7 -> /Expansion header/HDR_PC0
- J8 pad 15: /Expansion header/HDR_PC8 -> /Expansion header/HDR_PC2
- J8 pad 16: /Expansion header/HDR_PC9 -> /Expansion header/HDR_PC3
- J8 pad 17: /Expansion header/HDR_PC10 -> /Expansion header/HDR_PC6
- J8 pad 18: /Expansion header/HDR_PC11 -> /Expansion header/HDR_PC7
- J8 pad 19: /Expansion header/HDR_PC12 -> /Expansion header/HDR_PC8
- J8 pad 20: /Expansion header/HDR_PA15 -> /Expansion header/HDR_PC9
- J8 pad 21: /Expansion header/HDR_SCL -> /Expansion header/HDR_PC10
- J8 pad 22: /Expansion header/HDR_SDA -> /Expansion header/HDR_PC11
- J8 pad 23: /Expansion header/HDR_PB8 -> /Expansion header/HDR_PC12
- J8 pad 24: /Expansion header/HDR_PB9 -> /Expansion header/HDR_PA15
- J8 pad 25: /Expansion header/HDR_PA8 -> /Expansion header/HDR_PB8
- J8 pad 26: /Expansion header/HDR_PA10 -> /Expansion header/HDR_PB9
- J8 pad 27: /Expansion header/HDR_PB4 -> /Expansion header/HDR_PA8
- J8 pad 28: /Expansion header/HDR_PB2 -> /Expansion header/HDR_PA10
- J8 pad 29: /Expansion header/HDR_PB10 -> /Expansion header/HDR_PB4
- J8 pad 30: /Expansion header/HDR_PB13 -> /Expansion header/HDR_PB2
- J8 pad 31: /Expansion header/HDR_PB14 -> /Expansion header/HDR_PB10
- J8 pad 32: /Expansion header/HDR_PD14 -> /Expansion header/HDR_PB13
- J8 pad 33: /Expansion header/HDR_PD15 -> /Expansion header/HDR_PB14
- J8 pad 34: /Expansion header/HDR_PE0 -> /Expansion header/HDR_PD14
- J8 pad 35: GND -> /Expansion header/HDR_PD15
- J8 pad 36: GND -> /Expansion header/HDR_PE0
- J8 pad 5: /Expansion header/HDR_PA0 -> /Expansion header/HDR_SCL
- J8 pad 6: /Expansion header/HDR_PA3 -> /Expansion header/HDR_SDA
- J8 pad 7: /Expansion header/HDR_PA4 -> /Expansion header/HDR_EXP_nRESET
- J8 pad 8: /Expansion header/HDR_PA6 -> /Expansion header/HDR_EXP_INT
- J8 pad 9: /Expansion header/HDR_PB1 -> /Expansion header/HDR_PA0
- R101 pad 1: Net-(K1-Pad1) -> /Relay channels/RST_DRV1
- R101 pad 2: /MCU and USB/RST_DRV1 -> Net-(K1-Pad1)
- R102 pad 1: Net-(K2-Pad1) -> /Relay channels/PWR_DRV1
- R102 pad 2: /MCU and USB/PWR_DRV1 -> Net-(K2-Pad1)
- R103 pad 1: Net-(K3-Pad1) -> /Relay channels/RST_DRV2
- R103 pad 2: /MCU and USB/RST_DRV2 -> Net-(K3-Pad1)
- R104 pad 1: Net-(K4-Pad1) -> /Relay channels/PWR_DRV2
- R104 pad 2: /MCU and USB/PWR_DRV2 -> Net-(K4-Pad1)
- R105 pad 1: Net-(K5-Pad1) -> /Relay channels/RST_DRV3
- R105 pad 2: /MCU and USB/RST_DRV3 -> Net-(K5-Pad1)
- R106 pad 1: Net-(K6-Pad1) -> /Relay channels/PWR_DRV3
- R106 pad 2: /MCU and USB/PWR_DRV3 -> Net-(K6-Pad1)
- R107 pad 1: Net-(K7-Pad1) -> /Relay channels/RST_DRV4
- R107 pad 2: /MCU and USB/RST_DRV4 -> Net-(K7-Pad1)
- R108 pad 1: Net-(K8-Pad1) -> /Relay channels/PWR_DRV4
- R108 pad 2: /MCU and USB/PWR_DRV4 -> Net-(K8-Pad1)
- R109 pad 1: Net-(K9-Pad1) -> /Relay channels/RST_DRV5
- R109 pad 2: /MCU and USB/RST_DRV5 -> Net-(K9-Pad1)
- R110 pad 1: Net-(K10-Pad1) -> /Relay channels/PWR_DRV5
- R110 pad 2: /MCU and USB/PWR_DRV5 -> Net-(K10-Pad1)
- R111 pad 1: Net-(K11-Pad1) -> /Relay channels/RST_DRV6
- R111 pad 2: /MCU and USB/RST_DRV6 -> Net-(K11-Pad1)
- R112 pad 1: Net-(K12-Pad1) -> /Relay channels/PWR_DRV6
- R112 pad 2: /MCU and USB/PWR_DRV6 -> Net-(K12-Pad1)
- R113 pad 1: Net-(K13-Pad1) -> /Relay channels/RST_DRV7
- R113 pad 2: /MCU and USB/RST_DRV7 -> Net-(K13-Pad1)
- R114 pad 1: Net-(K14-Pad1) -> /Relay channels/PWR_DRV7
- R114 pad 2: /MCU and USB/PWR_DRV7 -> Net-(K14-Pad1)
- R115 pad 1: Net-(K15-Pad1) -> /Relay channels/RST_DRV8
- R115 pad 2: /MCU and USB/RST_DRV8 -> Net-(K15-Pad1)
- R116 pad 1: Net-(K16-Pad1) -> /Relay channels/PWR_DRV8
- R116 pad 2: /MCU and USB/PWR_DRV8 -> Net-(K16-Pad1)
- R201 pad 1: Net-(J11-Pin_2) -> Net-(K1-Pad4)
- R201 pad 2: Net-(K1-Pad4) -> /Relay channels/MB1_RST_B
- R202 pad 1: Net-(J11-Pin_4) -> Net-(K2-Pad4)
- R202 pad 2: Net-(K2-Pad4) -> /Relay channels/MB1_PWR_B
- R203 pad 1: Net-(J12-Pin_2) -> Net-(K3-Pad4)
- R203 pad 2: Net-(K3-Pad4) -> /Relay channels/MB2_RST_B
- R204 pad 1: Net-(J12-Pin_4) -> Net-(K4-Pad4)
- R204 pad 2: Net-(K4-Pad4) -> /Relay channels/MB2_PWR_B
- R205 pad 1: Net-(J13-Pin_2) -> Net-(K5-Pad4)
- R205 pad 2: Net-(K5-Pad4) -> /Relay channels/MB3_RST_B
- R206 pad 1: Net-(J13-Pin_4) -> Net-(K6-Pad4)
- R206 pad 2: Net-(K6-Pad4) -> /Relay channels/MB3_PWR_B
- R207 pad 1: Net-(J14-Pin_2) -> Net-(K7-Pad4)
- R207 pad 2: Net-(K7-Pad4) -> /Relay channels/MB4_RST_B
- R208 pad 1: Net-(J14-Pin_4) -> Net-(K8-Pad4)
- R208 pad 2: Net-(K8-Pad4) -> /Relay channels/MB4_PWR_B
- R209 pad 1: Net-(J15-Pin_2) -> Net-(K9-Pad4)
- R209 pad 2: Net-(K9-Pad4) -> /Relay channels/MB5_RST_B
- R210 pad 1: Net-(J15-Pin_4) -> Net-(K10-Pad4)
- R210 pad 2: Net-(K10-Pad4) -> /Relay channels/MB5_PWR_B
- R211 pad 1: Net-(J16-Pin_2) -> Net-(K11-Pad4)
- R211 pad 2: Net-(K11-Pad4) -> /Relay channels/MB6_RST_B
- R212 pad 1: Net-(J16-Pin_4) -> Net-(K12-Pad4)
- R212 pad 2: Net-(K12-Pad4) -> /Relay channels/MB6_PWR_B
- R213 pad 1: Net-(J17-Pin_2) -> Net-(K13-Pad4)
- R213 pad 2: Net-(K13-Pad4) -> /Relay channels/MB7_RST_B
- R214 pad 1: Net-(J17-Pin_4) -> Net-(K14-Pad4)
- R214 pad 2: Net-(K14-Pad4) -> /Relay channels/MB7_PWR_B
- R215 pad 1: Net-(J18-Pin_2) -> Net-(K15-Pad4)
- R215 pad 2: Net-(K15-Pad4) -> /Relay channels/MB8_RST_B
- R216 pad 1: Net-(J18-Pin_4) -> Net-(K16-Pad4)
- R216 pad 2: Net-(K16-Pad4) -> /Relay channels/MB8_PWR_B
- RN1 pad 1: /Expansion header/HDR_PA0 -> /Expansion header/HDR_SCL
- RN1 pad 2: /Expansion header/HDR_PA3 -> /Expansion header/HDR_SDA
- RN1 pad 3: /Expansion header/HDR_PA4 -> /Expansion header/HDR_EXP_nRESET
- RN1 pad 4: /Expansion header/HDR_PA6 -> /Expansion header/HDR_EXP_INT
- RN1 pad 5: GPIO_PA6 -> EXP_INT
- RN1 pad 6: GPIO_PA4 -> EXP_nRESET
- RN1 pad 7: GPIO_PA3 -> I2C1_SDA
- RN1 pad 8: GPIO_PA0 -> I2C1_SCL
- RN2 pad 1: /Expansion header/HDR_PB1 -> /Expansion header/HDR_PA0
- RN2 pad 2: /Expansion header/HDR_PC0 -> /Expansion header/HDR_PA3
- RN2 pad 3: /Expansion header/HDR_PC2 -> /Expansion header/HDR_PA4
- RN2 pad 4: /Expansion header/HDR_PC3 -> /Expansion header/HDR_PA6
- RN2 pad 5: GPIO_PC3 -> GPIO_PA6
- RN2 pad 6: GPIO_PC2 -> GPIO_PA4
- RN2 pad 7: GPIO_PC0 -> GPIO_PA3
- RN2 pad 8: GPIO_PB1 -> GPIO_PA0
- RN3 pad 1: /Expansion header/HDR_PC6 -> /Expansion header/HDR_PB1
- RN3 pad 2: /Expansion header/HDR_PC7 -> /Expansion header/HDR_PC0
- RN3 pad 3: /Expansion header/HDR_PC8 -> /Expansion header/HDR_PC2
- RN3 pad 4: /Expansion header/HDR_PC9 -> /Expansion header/HDR_PC3
- RN3 pad 5: GPIO_PC9 -> GPIO_PC3
- RN3 pad 6: GPIO_PC8 -> GPIO_PC2
- RN3 pad 7: GPIO_PC7 -> GPIO_PC0
- RN3 pad 8: GPIO_PC6 -> GPIO_PB1
- RN4 pad 1: /Expansion header/HDR_PC10 -> /Expansion header/HDR_PC6
- RN4 pad 2: /Expansion header/HDR_PC11 -> /Expansion header/HDR_PC7
- RN4 pad 3: /Expansion header/HDR_PC12 -> /Expansion header/HDR_PC8
- RN4 pad 4: /Expansion header/HDR_PA15 -> /Expansion header/HDR_PC9
- RN4 pad 5: GPIO_PA15 -> GPIO_PC9
- RN4 pad 6: GPIO_PC12 -> GPIO_PC8
- RN4 pad 7: GPIO_PC11 -> GPIO_PC7
- RN4 pad 8: GPIO_PC10 -> GPIO_PC6
- RN5 pad 1: /Expansion header/HDR_SCL -> /Expansion header/HDR_PC10
- RN5 pad 2: /Expansion header/HDR_SDA -> /Expansion header/HDR_PC11
- RN5 pad 3: /Expansion header/HDR_PB8 -> /Expansion header/HDR_PC12
- RN5 pad 4: /Expansion header/HDR_PB9 -> /Expansion header/HDR_PA15
- RN5 pad 5: GPIO_PB9 -> GPIO_PA15
- RN5 pad 6: GPIO_PB8 -> GPIO_PC12
- RN5 pad 7: I2C1_SDA -> GPIO_PC11
- RN5 pad 8: I2C1_SCL -> GPIO_PC10
- RN6 pad 1: /Expansion header/HDR_PA8 -> /Expansion header/HDR_PB8
- RN6 pad 2: /Expansion header/HDR_PA10 -> /Expansion header/HDR_PB9
- RN6 pad 3: /Expansion header/HDR_PB4 -> /Expansion header/HDR_PA8
- RN6 pad 4: /Expansion header/HDR_PB2 -> /Expansion header/HDR_PA10
- RN6 pad 5: GPIO_PB2 -> GPIO_PA10
- RN6 pad 6: GPIO_PB4 -> GPIO_PA8
- RN6 pad 7: GPIO_PA10 -> GPIO_PB9
- RN6 pad 8: GPIO_PA8 -> GPIO_PB8
- RN7 pad 1: /Expansion header/HDR_PB10 -> /Expansion header/HDR_PB4
- RN7 pad 2: /Expansion header/HDR_PB13 -> /Expansion header/HDR_PB2
- RN7 pad 3: /Expansion header/HDR_PB14 -> /Expansion header/HDR_PB10
- RN7 pad 4: /Expansion header/HDR_PD14 -> /Expansion header/HDR_PB13
- RN7 pad 5: GPIO_PD14 -> GPIO_PB13
- RN7 pad 6: GPIO_PB14 -> GPIO_PB10
- RN7 pad 7: GPIO_PB13 -> GPIO_PB2
- RN7 pad 8: GPIO_PB10 -> GPIO_PB4
- RN8 pad 1: /Expansion header/HDR_PD15 -> /Expansion header/HDR_PB14
- RN8 pad 2: /Expansion header/HDR_PE0 -> /Expansion header/HDR_PD14
- RN8 pad 3: unconnected-(RN8-R3.1-Pad3) -> /Expansion header/HDR_PD15
- RN8 pad 4: unconnected-(RN8-R4.1-Pad4) -> /Expansion header/HDR_PE0
- RN8 pad 5: unconnected-(RN8-R4.2-Pad5) -> GPIO_PE0
- RN8 pad 6: unconnected-(RN8-R3.2-Pad6) -> GPIO_PD15
- RN8 pad 7: GPIO_PE0 -> GPIO_PD14
- RN8 pad 8: GPIO_PD15 -> GPIO_PB14
- U1 pad 1: /MCU and USB/PWR_DRV1 -> EXP_nRESET
- U1 pad 2: /MCU and USB/PWR_DRV2 -> EXP_INT
- U1 pad 3: /MCU and USB/PWR_DRV3 -> unconnected-(U1-PE4-Pad3)
- U1 pad 38: /MCU and USB/PWR_DRV6 -> unconnected-(U1-PE7-Pad38)
- U1 pad 39: /MCU and USB/PWR_DRV7 -> unconnected-(U1-PE8-Pad39)
- U1 pad 4: /MCU and USB/PWR_DRV4 -> unconnected-(U1-PE5-Pad4)
- U1 pad 40: /MCU and USB/PWR_DRV8 -> unconnected-(U1-PE9-Pad40)
- U1 pad 41: /MCU and USB/PWR_DRV9 -> unconnected-(U1-PE10-Pad41)
- U1 pad 42: /MCU and USB/PWR_DRV10 -> unconnected-(U1-PE11-Pad42)
- U1 pad 43: /MCU and USB/PWR_DRV11 -> unconnected-(U1-PE12-Pad43)
- U1 pad 44: /MCU and USB/PWR_DRV12 -> unconnected-(U1-PE13-Pad44)
- U1 pad 45: /MCU and USB/PWR_DRV13 -> unconnected-(U1-PE14-Pad45)
- U1 pad 46: /MCU and USB/PWR_DRV14 -> unconnected-(U1-PE15-Pad46)
- U1 pad 5: /MCU and USB/PWR_DRV5 -> unconnected-(U1-PE6-Pad5)
- U1 pad 55: /MCU and USB/RST_DRV9 -> unconnected-(U1-PD8-Pad55)
- U1 pad 56: /MCU and USB/RST_DRV10 -> unconnected-(U1-PD9-Pad56)
- U1 pad 57: /MCU and USB/RST_DRV11 -> unconnected-(U1-PD10-Pad57)
- U1 pad 58: /MCU and USB/RST_DRV12 -> unconnected-(U1-PD11-Pad58)
- U1 pad 59: /MCU and USB/RST_DRV13 -> unconnected-(U1-PD12-Pad59)
- U1 pad 60: /MCU and USB/RST_DRV14 -> unconnected-(U1-PD13-Pad60)
- U1 pad 81: /MCU and USB/RST_DRV1 -> unconnected-(U1-PD0-Pad81)
- U1 pad 82: /MCU and USB/RST_DRV2 -> unconnected-(U1-PD1-Pad82)
- U1 pad 83: /MCU and USB/RST_DRV3 -> unconnected-(U1-PD2-Pad83)
- U1 pad 84: /MCU and USB/RST_DRV4 -> unconnected-(U1-PD3-Pad84)
- U1 pad 85: /MCU and USB/RST_DRV5 -> unconnected-(U1-PD4-Pad85)
- U1 pad 86: /MCU and USB/RST_DRV6 -> unconnected-(U1-PD5-Pad86)
- U1 pad 87: /MCU and USB/RST_DRV7 -> unconnected-(U1-PD6-Pad87)
- U1 pad 88: /MCU and USB/RST_DRV8 -> unconnected-(U1-PD7-Pad88)
- U10 pad 1: /Expansion header/HDR_SCL -> /Expansion header/HDR_PC10
- U10 pad 2: /Expansion header/HDR_SDA -> /Expansion header/HDR_PC11
- U10 pad 4: /Expansion header/HDR_PB8 -> /Expansion header/HDR_PC12
- U10 pad 5: /Expansion header/HDR_PB9 -> /Expansion header/HDR_PA15
- U11 pad 1: /Expansion header/HDR_PA8 -> /Expansion header/HDR_PB8
- U11 pad 2: /Expansion header/HDR_PA10 -> /Expansion header/HDR_PB9
- U11 pad 4: /Expansion header/HDR_PB4 -> /Expansion header/HDR_PA8
- U11 pad 5: /Expansion header/HDR_PB2 -> /Expansion header/HDR_PA10
- U12 pad 1: /Expansion header/HDR_PB10 -> /Expansion header/HDR_PB4
- U12 pad 2: /Expansion header/HDR_PB13 -> /Expansion header/HDR_PB2
- U12 pad 4: /Expansion header/HDR_PB14 -> /Expansion header/HDR_PB10
- U12 pad 5: /Expansion header/HDR_PD14 -> /Expansion header/HDR_PB13
- U13 pad 1: /Expansion header/HDR_PD15 -> /Expansion header/HDR_PB14
- U13 pad 2: /Expansion header/HDR_PE0 -> /Expansion header/HDR_PD14
- U13 pad 4: unconnected-(U13-D2+-Pad4) -> /Expansion header/HDR_PD15
- U13 pad 5: unconnected-(U13-D2--Pad5) -> /Expansion header/HDR_PE0
- U6 pad 1: /Expansion header/HDR_PA0 -> /Expansion header/HDR_SCL
- U6 pad 2: /Expansion header/HDR_PA3 -> /Expansion header/HDR_SDA
- U6 pad 4: /Expansion header/HDR_PA4 -> /Expansion header/HDR_EXP_nRESET
- U6 pad 5: /Expansion header/HDR_PA6 -> /Expansion header/HDR_EXP_INT
- U7 pad 1: /Expansion header/HDR_PB1 -> /Expansion header/HDR_PA0
- U7 pad 2: /Expansion header/HDR_PC0 -> /Expansion header/HDR_PA3
- U7 pad 4: /Expansion header/HDR_PC2 -> /Expansion header/HDR_PA4
- U7 pad 5: /Expansion header/HDR_PC3 -> /Expansion header/HDR_PA6
- U8 pad 1: /Expansion header/HDR_PC6 -> /Expansion header/HDR_PB1
- U8 pad 2: /Expansion header/HDR_PC7 -> /Expansion header/HDR_PC0
- U8 pad 4: /Expansion header/HDR_PC8 -> /Expansion header/HDR_PC2
- U8 pad 5: /Expansion header/HDR_PC9 -> /Expansion header/HDR_PC3
- U9 pad 1: /Expansion header/HDR_PC10 -> /Expansion header/HDR_PC6
- U9 pad 2: /Expansion header/HDR_PC11 -> /Expansion header/HDR_PC7
- U9 pad 4: /Expansion header/HDR_PC12 -> /Expansion header/HDR_PC8
- U9 pad 5: /Expansion header/HDR_PA15 -> /Expansion header/HDR_PC9

Commit message: Rev C: ESP32-C6 + W5500 controller for immersion
Schematic rework per docs/controller.md.

- MCU: ESP32-C6-MINI-1-N4 replaces STM32H563VIT6 (KiCad-stock
  module). EN/BOOT test pads, USB-C via the C6 USB Serial/JTAG with
  22R series resistors behind the existing USBLC6.
- Ethernet: W5500 over SPI replaces LAN8742A/RMII. PHY network,
  center taps, AVDD ferrite and LED wiring per WIZnet's W5500
  Ethernet Shield reference; ARJP11A magjack and PoE path unchanged.
- I2C split: internal bus (relay MCP23017, TMP1075) on HP I2C with
  its own expander reset (EXP_nRESET_INT, GPIO14); external bus to
  the header (software I2C on GPIO6/7) with EXP_nRESET (GPIO4,
  pulled low) and the shared EXP_INT.
- Expansion header J8 now 2x6: external I2C, reset, interrupt,
  GPIO5/8/15, fused 3V3/5V, all protected as before.
- C1/C2: KEMET T520 molded tantalum-polymer instead of rubber-sealed
  aluminium-polymer cans (immersion).
- Sheets regenerated: Power, Ethernet, MCU replace power_eth and
  mcu_usb; root and project net classes updated (RMII/SWD/RST
  classes removed). Board regenerated, nothing placed yet.
- Spec updated to the captured design.
Parts:
- removed C20, C21: 4.7u, Capacitor_SMD:C_0603_1608Metric
- removed C24, C25: 2.2u, Capacitor_SMD:C_0603_1608Metric
- removed C33, C37: 100n, Capacitor_SMD:C_0402_1005Metric
- removed J3: TC2030-IDC-NL, Connector:Tag-Connect_TC2030-IDC-NL_2x03_P1.27mm_Vertical
- removed R31: 100, Resistor_SMD:R_0603_1608Metric
- removed RN3, RN4, RN5, RN6, RN7, RN8: 4x330, Resistor_SMD:R_Array_Convex_4x0402
- removed U10, U11, U12, U13, U8, U9: TPD4E05U06DQA, Package_SON:USON-10_2.5x1.0mm_P0.5mm
- removed Y1: 25MHz ABM8G, Crystal:Crystal_SMD_Abracon_ABM8G-4Pin_3.2x2.5mm
- added C14: 1u, Capacitor_SMD:C_0603_1608Metric, F.Cu at (-192.0, 0.00)
- added C15: 100n, Capacitor_SMD:C_0402_1005Metric, F.Cu at (-178.0, 0.00)
- added L2: 120R@100MHz, Inductor_SMD:L_0603_1608Metric, F.Cu at (-310.0, 42.0)
- added R34: 22, Resistor_SMD:R_0402_1005Metric, F.Cu at (-164.0, 42.0)
- added R35: 22, Resistor_SMD:R_0402_1005Metric, F.Cu at (-150.0, 42.0)
- added R36: 100, Resistor_SMD:R_0603_1608Metric, F.Cu at (-220.0, 56.0)
- C1, C2: value 220u/6V3 poly -> 220u/6V3 Ta-poly; footprint granite:CP_Elec_6.3x5.9_Panasonic_SVPC_C6 -> Capacitor_Tantalum_SMD:CP_EIA-7343-31_Kemet-D
- C12, C32: value 100n -> 10u; footprint Capacitor_SMD:C_0402_1005Metric -> Capacitor_SMD:C_0805_2012Metric
- C26, C27: value 22p -> 18p
- C28: value 1u -> 6.8n; footprint Capacitor_SMD:C_0603_1608Metric -> Capacitor_SMD:C_0402_1005Metric
- C29: value 100n -> 6.8n
- C30: value 100n -> 4.7u; footprint Capacitor_SMD:C_0402_1005Metric -> Capacitor_SMD:C_0603_1608Metric
- C31, C35: value 100n -> 10n
- C34: value 100n -> 22n
- C5, C6: value 15p -> 100n
- J8: footprint Connector_PinHeader_2.54mm:PinHeader_2x20_P2.54mm_Vertical -> Connector_PinHeader_2.54mm:PinHeader_2x06_P2.54mm_Vertical
- R13, R14: value 33 -> 4.7k
- R15: value 12.1k -> 12.4k 1%
- R16: value 1.5k -> 10k
- R26: value 0 -> 10; footprint Resistor_SMD:R_0603_1608Metric -> Resistor_SMD:R_0402_1005Metric
- R27: value 0 -> 10k; footprint Resistor_SMD:R_0603_1608Metric -> Resistor_SMD:R_0402_1005Metric
- R29: value 499 -> 1M
- R3, R4: value 470 -> 330
- TP1: value NRST -> EN
- TP2: value BOOT0 -> BOOT
- U1: value STM32H563VIT6 -> ESP32-C6-MINI-1-N4; footprint Package_QFP:LQFP-100_14x14mm_P0.5mm -> RF_Module:ESP32-C6-MINI-1
- U3: value LAN8742A -> W5500; footprint Package_DFN_QFN:VQFN-24-1EP_4x4mm_P0.5mm_EP2.5x2.5mm_ThermalVias -> Package_QFP:LQFP-48_7x7mm_P0.5mm
- moved R19 198.5 mm to (-150.0, 28.0)
- moved R13 168.3 mm to (-178.0, 28.0)
- moved R14 168.3 mm to (-164.0, 28.0)
- moved R29 162.4 mm to (-240.0, 70.0)
- moved R27 157.7 mm to (-192.0, 42.0)
- moved R10 132.7 mm to (-254.0, 42.0)
- moved R11 132.7 mm to (-240.0, 42.0)
- moved R9 132.7 mm to (-268.0, 42.0)
- moved C28 132.0 mm to (-268.0, 14.0)
- moved C29 132.0 mm to (-254.0, 14.0)
- moved C30 132.0 mm to (-240.0, 14.0)
- moved C35 132.0 mm to (-268.0, 28.0)
- moved C36 132.0 mm to (-254.0, 28.0)
- moved D4 107.7 mm to (-164.0, 0.00)
- moved D5 107.7 mm to (-150.0, 0.00)
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Connections:
- net /Expansion header/HDR_EXP_INT renamed /Expansion header/HDR_INT
- net /Expansion header/HDR_EXP_nRESET renamed /Expansion header/HDR_nRESET
- net /Expansion header/HDR_PA0 renamed /Expansion header/HDR_IO5
- net /Expansion header/HDR_PA3 renamed /Expansion header/HDR_IO8
- net /Expansion header/HDR_PA4 renamed /Expansion header/HDR_IO15
- net /MCU and USB/OW_DATA renamed /MCU/OW_DATA
- net /Power and Ethernet/FB_3V3 renamed /Power/FB_3V3
- net /Power and Ethernet/POE_5V renamed /Power/POE_5V
- net /Power and Ethernet/VPOE_N renamed VPOE_N
- net /Power and Ethernet/VPOE_P renamed VPOE_P
- net Net-(D4-A) renamed /MCU/LED_A
- net Net-(J2-CC1) renamed /MCU/USB_CC1
- net Net-(J2-CC2) renamed /MCU/USB_CC2
- net Net-(J2-D+-PadA6) renamed /MCU/USB_CONN_D+
- net Net-(J2-D--PadA7) renamed /MCU/USB_CONN_D-
- net Net-(U2-SW) renamed /Power/SW_3V3
- C10 pad 1: GND -> /Ethernet/+3V3A
- C10 pad 2: +3V3 -> GND
- C11 pad 1: GND -> +3V3
- C11 pad 2: +3V3 -> GND
- C12 pad 1: GND -> +3V3
- C12 pad 2: +3V3 -> GND
- C13 pad 1: GND -> +3V3
- C13 pad 2: +3V3 -> GND
- C26 pad 1: Net-(U3-XTAL1/CLKIN) -> /Ethernet/ETH_XI
- C27 pad 1: Net-(C27-Pad1) -> /Ethernet/ETH_XO
- C28 pad 1: GND -> /Ethernet/ETH_RXP_T
- C28 pad 2: /Power and Ethernet/VDDCR -> /Ethernet/ETH_RX+
- C29 pad 1: GND -> /Ethernet/ETH_RXN_T
- C29 pad 2: +3V3 -> /Ethernet/ETH_RX-
- C3 pad 1: GND -> +5V
- C3 pad 2: +5V -> GND
- C30 pad 1: GND -> /Ethernet/ETH_TOCAP
- C30 pad 2: +3V3 -> GND
- C31 pad 1: GND -> /Ethernet/ETH_1V2O
- C31 pad 2: +3V3 -> GND
- C32 pad 1: GND -> /Ethernet/+3V3A
- C32 pad 2: +3V3 -> GND
- C34 pad 1: GND -> /Ethernet/ETH_TCT
- C34 pad 2: /Power and Ethernet/ETH_TCT -> GND
- C35 pad 1: GND -> /Ethernet/ETH_RCT
- C35 pad 2: /Power and Ethernet/ETH_RCT -> GND
- C36 pad 1: Net-(C36-Pad1) -> /Ethernet/ETH_SHLD
- C4 pad 1: GND -> +3V3
- C4 pad 2: +3V3 -> GND
- C5 pad 1: Net-(U1-PH0) -> /Ethernet/+3V3A
- C6 pad 1: Net-(U1-PH1) -> /Ethernet/+3V3A
- C7 pad 1: GND -> /Ethernet/+3V3A
- C7 pad 2: /MCU and USB/NRST -> GND
- C8 pad 1: GND -> /Ethernet/+3V3A
- C8 pad 2: +3V3 -> GND
- C9 pad 1: GND -> /Ethernet/+3V3A
- C9 pad 2: +3V3 -> GND
- J1 pad 1: /Power and Ethernet/ETH_TX+ -> /Ethernet/ETH_TX+
- J1 pad 11: /Power and Ethernet/PHY_LED2 -> +3V3
- J1 pad 12: Net-(J1-Pad12) -> /Ethernet/ETH_LEDK_LINK
- J1 pad 13: /Power and Ethernet/PHY_LED1 -> +3V3
- J1 pad 14: Net-(J1-Pad14) -> /Ethernet/ETH_LEDK_ACT
- J1 pad 2: /Power and Ethernet/ETH_TX- -> /Ethernet/ETH_TX-
- J1 pad 3: /Power and Ethernet/ETH_RX+ -> /Ethernet/ETH_RX+
- J1 pad 4: /Power and Ethernet/ETH_TCT -> /Ethernet/ETH_TCT
- J1 pad 5: /Power and Ethernet/ETH_RCT -> /Ethernet/ETH_RCT
- J1 pad 6: /Power and Ethernet/ETH_RX- -> /Ethernet/ETH_RX-
- J1 pad 7: Net-(C36-Pad1) -> /Ethernet/ETH_SHLD
- J8 pad 12: /Expansion header/HDR_PA6 -> GND
- R10 pad 1: /MCU and USB/ETH_TXD1 -> /Ethernet/ETH_TXN
- R10 pad 2: Net-(U3-TXD1) -> /Ethernet/ETH_TX-
- R11 pad 1: /MCU and USB/ETH_TX_EN -> /Ethernet/ETH_RXP
- R11 pad 2: Net-(U3-TXEN) -> /Ethernet/ETH_RXP_T
- R12 pad 1: /MCU and USB/ETH_REF_CLK -> /Ethernet/ETH_RXN
- R12 pad 2: Net-(U3-~{INT}/REFCLKO) -> /Ethernet/ETH_RXN_T
- R13 pad 1: /MCU and USB/ETH_RXD0 -> +3V3
- R13 pad 2: Net-(U3-RXD0/MODE0) -> I2C_EXT_SCL
- R14 pad 1: /MCU and USB/ETH_RXD1 -> +3V3
- R14 pad 2: Net-(U3-RXD1/MODE1) -> I2C_EXT_SDA
- R15 pad 1: GND -> /Ethernet/ETH_EXRES
- R15 pad 2: /Power and Ethernet/RBIAS -> GND
- R16 pad 2: /MCU and USB/ETH_MDIO -> ETH_CS
- R17 pad 1: GND -> +3V3
- R17 pad 2: /Power and Ethernet/PHY_LED1 -> ETH_INT
- R18 pad 1: GND -> +3V3
- R18 pad 2: /Power and Ethernet/PHY_LED2 -> ETH_RST
- R19 pad 1: +3V3 -> EXP_nRESET
- R19 pad 2: /MCU and USB/ETH_nRST -> GND
- R20 pad 1: +3V3 -> /Ethernet/ETH_TX+
- R20 pad 2: /Power and Ethernet/ETH_TX+ -> /Ethernet/+3V3A
- R21 pad 1: /Power and Ethernet/ETH_TX- -> /Ethernet/ETH_TX-
- R21 pad 2: +3V3 -> /Ethernet/+3V3A
- R22 pad 1: /Power and Ethernet/ETH_RX+ -> /Ethernet/ETH_RXP_T
- R22 pad 2: +3V3 -> /Ethernet/ETH_RCT
- R23 pad 1: /Power and Ethernet/ETH_RX- -> /Ethernet/ETH_RXN_T
- R23 pad 2: +3V3 -> /Ethernet/ETH_RCT
- R26 pad 1: /Power and Ethernet/ETH_TCT -> /Ethernet/ETH_TCT
- R26 pad 2: +3V3 -> /Ethernet/+3V3A
- R27 pad 1: /Power and Ethernet/ETH_RCT -> +3V3
- R27 pad 2: +3V3 -> GPIO_IO8
- R28 pad 1: GND -> /Ethernet/ETH_SHLD
- R28 pad 2: Net-(C36-Pad1) -> GND
- R29 pad 1: Net-(C27-Pad1) -> /Ethernet/ETH_XI
- R29 pad 2: Net-(U3-XTAL2) -> /Ethernet/ETH_XO
- R3 pad 1: GND -> /Ethernet/ETH_LEDK_LINK
- R3 pad 2: Net-(J1-Pad14) -> /Ethernet/ETH_LED_LINK
- R32 pad 1: EXP_nRESET -> EXP_nRESET_INT
- R4 pad 1: Net-(J1-Pad12) -> /Ethernet/ETH_LEDK_ACT
- R4 pad 2: GND -> /Ethernet/ETH_LED_ACT
- R5 pad 2: I2C1_SCL -> I2C_INT_SCL
- R6 pad 2: I2C1_SDA -> I2C_INT_SDA
- R7 pad 1: GND -> +3V3
- R7 pad 2: /MCU and USB/BOOT0 -> /MCU/C6_EN
- R8 pad 1: /MCU and USB/LED_HB -> /MCU/LED_HB
- R9 pad 1: /MCU and USB/ETH_TXD0 -> /Ethernet/ETH_TXP
- R9 pad 2: Net-(U3-TXD0) -> /Ethernet/ETH_TX+
- RN1 pad 7: I2C1_SDA -> I2C_EXT_SDA
- RN1 pad 8: I2C1_SCL -> I2C_EXT_SCL
- RN2 pad 4: /Expansion header/HDR_PA6 -> unconnected-(RN2-R4.1-Pad4)
- RN2 pad 5: GPIO_PA6 -> unconnected-(RN2-R4.2-Pad5)
- RN2 pad 6: GPIO_PA4 -> GPIO_IO15
- RN2 pad 7: GPIO_PA3 -> GPIO_IO8
- RN2 pad 8: GPIO_PA0 -> GPIO_IO5
- TP1 pad 1: /MCU and USB/NRST -> /MCU/C6_EN
- TP2 pad 1: /MCU and USB/BOOT0 -> /MCU/C6_BOOT
- U1 pad 1: EXP_nRESET -> GND
- U1 pad 10: GND -> GPIO_IO5
- U1 pad 11: +3V3 -> GND
- U1 pad 12: Net-(U1-PH0) -> EXP_INT
- U1 pad 13: Net-(U1-PH1) -> /MCU/LED_HB
- U1 pad 14: /MCU and USB/NRST -> GND
- U1 pad 15: GPIO_PC0 -> I2C_EXT_SDA
- U1 pad 16: /MCU and USB/ETH_MDC -> I2C_EXT_SCL
- U1 pad 17: GPIO_PC2 -> /MCU/C6_USB_D-
- U1 pad 18: GPIO_PC3 -> /MCU/C6_USB_D+
- U1 pad 19: GND -> EXP_nRESET_INT
- U1 pad 2: EXP_INT -> GND
- U1 pad 20: GND -> GPIO_IO15
- U1 pad 21: +3V3 -> unconnected-(U1-NC-Pad21)
- U1 pad 22: +3V3 -> GPIO_IO8
- U1 pad 23: GPIO_PA0 -> /MCU/C6_BOOT
- U1 pad 24: /MCU and USB/ETH_REF_CLK -> ETH_CS
- U1 pad 25: /MCU and USB/ETH_MDIO -> ETH_SCLK
- U1 pad 26: GPIO_PA3 -> ETH_MOSI
- U1 pad 27: GND -> ETH_MISO
- U1 pad 28: +3V3 -> ETH_INT
- U1 pad 29: GPIO_PA4 -> ETH_RST
- U1 pad 3: unconnected-(U1-PE4-Pad3) -> +3V3
- U1 pad 30: /MCU and USB/ETH_TX_EN -> /MCU/OW_MCU
- U1 pad 31: GPIO_PA6 -> /MCU/OW_MCU
- U1 pad 32: /MCU and USB/ETH_CRS_DV -> unconnected-(U1-NC-Pad32)
- U1 pad 33: /MCU and USB/ETH_RXD0 -> unconnected-(U1-NC-Pad33)
- U1 pad 34: /MCU and USB/ETH_RXD1 -> unconnected-(U1-NC-Pad34)
- U1 pad 35: /MCU and USB/LED_HB -> unconnected-(U1-NC-Pad35)
- U1 pad 36: GPIO_PB1 -> GND
- U1 pad 37: GPIO_PB2 -> GND
- U1 pad 38: unconnected-(U1-PE7-Pad38) -> GND
- U1 pad 39: unconnected-(U1-PE8-Pad39) -> GND
- U1 pad 40: unconnected-(U1-PE9-Pad40) -> GND
- U1 pad 41: unconnected-(U1-PE10-Pad41) -> GND
- U1 pad 42: unconnected-(U1-PE11-Pad42) -> GND
- U1 pad 43: unconnected-(U1-PE12-Pad43) -> GND
- U1 pad 44: unconnected-(U1-PE13-Pad44) -> GND
- U1 pad 45: unconnected-(U1-PE14-Pad45) -> GND
- U1 pad 46: unconnected-(U1-PE15-Pad46) -> GND
- U1 pad 47: GPIO_PB10 -> GND
- U1 pad 48: Net-(C24-Pad1) -> GND
- U1 pad 5: unconnected-(U1-PE6-Pad5) -> I2C_INT_SDA
- U1 pad 50: +3V3 -> GND
- U1 pad 51: /MCU and USB/ETH_TXD0 -> GND
- U1 pad 52: GPIO_PB13 -> GND
- U1 pad 53: GPIO_PB14 -> GND
- U1 pad 6: +3V3 -> I2C_INT_SCL
- U1 pad 8: unconnected-(U1-PC14-Pad8) -> /MCU/C6_EN
- U1 pad 9: unconnected-(U1-PC15-Pad9) -> EXP_nRESET
- U14 pad 12: I2C1_SCL -> I2C_INT_SCL
- U14 pad 13: I2C1_SDA -> I2C_INT_SDA
- U14 pad 18: EXP_nRESET -> EXP_nRESET_INT
- U3 pad 1: +3V3 -> /Ethernet/ETH_TXN
- U3 pad 10: unconnected-(U3-RXER/PHYAD0-Pad10) -> /Ethernet/ETH_EXRES
- U3 pad 11: /MCU and USB/ETH_CRS_DV -> /Ethernet/+3V3A
- U3 pad 12: /MCU and USB/ETH_MDIO -> unconnected-(U3-NC-Pad12)
- U3 pad 13: /MCU and USB/ETH_MDC -> unconnected-(U3-NC-Pad13)
- U3 pad 14: Net-(U3-~{INT}/REFCLKO) -> GND
- U3 pad 15: /MCU and USB/ETH_nRST -> /Ethernet/+3V3A
- U3 pad 16: Net-(U3-TXEN) -> GND
- U3 pad 17: Net-(U3-TXD0) -> /Ethernet/+3V3A
- U3 pad 18: Net-(U3-TXD1) -> unconnected-(U3-VBG-Pad18)
- U3 pad 19: +3V3 -> GND
- U3 pad 2: /Power and Ethernet/PHY_LED2 -> /Ethernet/ETH_TXP
- U3 pad 20: /Power and Ethernet/ETH_TX- -> /Ethernet/ETH_TOCAP
- U3 pad 21: /Power and Ethernet/ETH_TX+ -> /Ethernet/+3V3A
- U3 pad 22: /Power and Ethernet/ETH_RX- -> /Ethernet/ETH_1V2O
- U3 pad 23: /Power and Ethernet/ETH_RX+ -> GND
- U3 pad 24: /Power and Ethernet/RBIAS -> unconnected-(U3-SPDLED-Pad24)
- U3 pad 25: GND -> /Ethernet/ETH_LED_LINK
- U3 pad 3: /Power and Ethernet/PHY_LED1 -> GND
- U3 pad 4: Net-(U3-XTAL2) -> /Ethernet/+3V3A
- U3 pad 5: Net-(U3-XTAL1/CLKIN) -> /Ethernet/ETH_RXN
- U3 pad 6: /Power and Ethernet/VDDCR -> /Ethernet/ETH_RXP
- U3 pad 7: Net-(U3-RXD1/MODE1) -> unconnected-(U3-DNC-Pad7)
- U3 pad 8: Net-(U3-RXD0/MODE0) -> /Ethernet/+3V3A
- U3 pad 9: +3V3 -> GND
- U4 pad 4: /MCU and USB/USB_D+ -> /MCU/USB_D+
- U4 pad 6: /MCU and USB/USB_D- -> /MCU/USB_D-
- U5 pad 1: I2C1_SDA -> I2C_INT_SDA
- U5 pad 2: I2C1_SCL -> I2C_INT_SCL
- U7 pad 5: /Expansion header/HDR_PA6 -> unconnected-(U7-D2--Pad5)
- Y2 pad 1: Net-(U3-XTAL1/CLKIN) -> /Ethernet/ETH_XI
- Y2 pad 3: Net-(C27-Pad1) -> /Ethernet/ETH_XO

Commit message: Regenerate PCB for JLCPCB
Fresh board from the current netlist (162 footprints, 0 parity issues),
all parked off-board, no outline yet. Stackup switched to JLC04161H-7628
(0.2104 mm 7628 prepreg, 0.5 oz inner). Diff pairs re-solved: ETH
0.16/0.15 = 101R with the fluid above, USB 0.25/0.15 = 89R in air
(service port). Docs updated for JLC as fab.
Parts:
- removed C1: 220u/6V3 Ta-poly, Capacitor_Tantalum_SMD:CP_EIA-7343-31_Kemet-D
- removed PS1: Ag9905-MT, granite:Silvertel_Ag9905MT
- added C40: 4.7u/50V, Capacitor_SMD:C_1206_3216Metric, F.Cu at (-358.0, 0.00)
- added C41: 4.7u/50V, Capacitor_SMD:C_1206_3216Metric, F.Cu at (-344.0, 0.00)
- added C42: 100n/50V, Capacitor_SMD:C_0402_1005Metric, F.Cu at (-330.0, 0.00)
- added C43: 100n/50V, Capacitor_SMD:C_0402_1005Metric, F.Cu at (-400.0, 14.0)
- added C44: 22u, Capacitor_SMD:C_0805_2012Metric, F.Cu at (-386.0, 14.0)
- added C45: 22u, Capacitor_SMD:C_0805_2012Metric, F.Cu at (-372.0, 14.0)
- added D8: SS34, Diode_SMD:D_SMA, F.Cu at (-400.0, 28.0)
- added F3: PTC 0.5A, Fuse:Fuse_1206_3216Metric, F.Cu at (-386.0, 28.0)
- added J3: 19V_IN, Connector_JST:JST_PH_B2B-PH-K_1x02_P2.00mm_Vertical, F.Cu at (-372.0, 28.0)
- added L3: 3u3, Inductor_SMD:L_Changjiang_FXL0630, F.Cu at (-344.0, 28.0)
- added R37: 100k, Resistor_SMD:R_0402_1005Metric, F.Cu at (-386.0, 42.0)
- added R38: 13k, Resistor_SMD:R_0402_1005Metric, F.Cu at (-372.0, 42.0)
- added U8: LMR51430YDDCR, Package_TO_SOT_SMD:SOT-23-6, F.Cu at (-344.0, 42.0)
- C2: value 220u/6V3 Ta-poly -> 220u/10V Ta-poly
- D1: value SMAJ58A -> SMAJ22A
- J1: value ARJP11A-MASA-B-A-EMU2 -> HR911105A; footprint Connector_RJ:RJ45_Abracon_ARJP11A-MA_Horizontal -> Connector_RJ:RJ45_Hanrun_HR911105A_Horizontal
- moved D3 70.0 mm to (-330.0, 14.0)
- moved R2 62.6 mm to (-400.0, 42.0)
- moved U2 39.6 mm to (-358.0, 42.0)
- moved L1 31.3 mm to (-358.0, 28.0)
- moved R1 31.3 mm to (-330.0, 28.0)
- moved D1 19.8 mm to (-358.0, 14.0)
- moved D2 19.8 mm to (-344.0, 14.0)
- moved C2 14.0 mm to (-400.0, 0.00)
- moved C3 14.0 mm to (-386.0, 0.00)
- moved C4 14.0 mm to (-372.0, 0.00)
Connections:
- D1 pad 1: VPOE_P -> Net-(D1-K)
- D1 pad 2: VPOE_N -> GND
- D2 pad 2: /Power/POE_5V -> /Power/BUCK_5V
- J1 pad 10: VPOE_N -> /Ethernet/ETH_LEDK_LINK
- J1 pad 11: +3V3 -> /Ethernet/ETH_LEDK_ACT
- J1 pad 12: /Ethernet/ETH_LEDK_LINK -> +3V3
- J1 pad 7: /Ethernet/ETH_SHLD -> unconnected-(J1-NC-Pad7)
- J1 pad 9: VPOE_P -> +3V3
- J1 pad SH: GND -> /Ethernet/ETH_SHLD
