File: granite_controller.kicad_pcb (KiCad board)
At the start: 4 copper layers, 162 parts, among them J1 HR911105A, J11 MB01_FP, J12 MB02_FP, J13 MB03_FP, J14 MB04_FP, J15 MB05_FP, J16 MB06_FP, J17 MB07_FP, J18 MB08_FP, J2 USB4105-xx-A, J3 19V_IN, J4 1WIRE, J5 1WIRE, J6 1WIRE, J7 1WIRE, J8 EXPANSION, K1 TLP176AM, K10 TLP176AM, K11 TLP176AM, K12 TLP176AM, K13 TLP176AM, K14 TLP176AM, K15 TLP176AM, K16 TLP176AM, K2 TLP176AM, K3 TLP176AM, K4 TLP176AM, K5 TLP176AM, K6 TLP176AM, K7 TLP176AM, K8 TLP176AM, K9 TLP176AM, U1 ESP32-C6-MINI-1-N4, U14 MCP23017-E/SO, U2 TLV62569DBV, U3 W5500, U4 USBLC6-2SC6, U5 TMP1075D, U6 TPD4E05U06DQA, U7 TPD4E05U06DQA, U8 LMR51430YDDCR, Y2 25MHz 12pF YXC

Commit message: Regenerate PCB for the WROOM-1, sensing and new connectors
200 footprints parked off-board, 0 parity issues.
Parts:
- added C46: 100n, Capacitor_SMD:C_0402_1005Metric, F.Cu at (-116.0, 0.00)
- added C47: 100n, Capacitor_SMD:C_0402_1005Metric, F.Cu at (-40.0, 0.00)
- added C48: 100n, Capacitor_SMD:C_0402_1005Metric, F.Cu at (-26.0, 0.00)
- added C49: 100n, Capacitor_SMD:C_0402_1005Metric, F.Cu at (-12.0, 0.00)
- added C50: 100n, Capacitor_SMD:C_0402_1005Metric, F.Cu at (2.00, 0.00)
- added C51: 100n, Capacitor_SMD:C_0402_1005Metric, F.Cu at (-358.0, 14.0)
- added J10: DRY_IN, Connector_JST:JST_PH_B5B-PH-K_1x05_P2.00mm_Vertical, F.Cu at (16.0, 14.0)
- added J9: I2C_SENSOR, Connector_JST:JST_PH_B4B-PH-K_1x04_P2.00mm_Vertical, F.Cu at (2.00, 14.0)
- added R39: 10k, Resistor_SMD:R_0402_1005Metric, F.Cu at (-74.0, 56.0)
- added R40: 10k, Resistor_SMD:R_0402_1005Metric, F.Cu at (-60.0, 56.0)
- added R41: 10k, Resistor_SMD:R_0402_1005Metric, F.Cu at (-130.0, 70.0)
- added R42: 10k, Resistor_SMD:R_0402_1005Metric, F.Cu at (-116.0, 70.0)
- added R43: 10k, Resistor_SMD:R_0402_1005Metric, F.Cu at (-102.0, 70.0)
- added R44: 10k, Resistor_SMD:R_0402_1005Metric, F.Cu at (-88.0, 70.0)
- added R45: 10k, Resistor_SMD:R_0402_1005Metric, F.Cu at (-74.0, 70.0)
- added R46: 10k, Resistor_SMD:R_0402_1005Metric, F.Cu at (-60.0, 70.0)
- added R47: 220, Resistor_SMD:R_0402_1005Metric, F.Cu at (-130.0, 84.0)
- added R48: 220, Resistor_SMD:R_0402_1005Metric, F.Cu at (-116.0, 84.0)
- added R49: 220, Resistor_SMD:R_0402_1005Metric, F.Cu at (-102.0, 84.0)
- added R50: 220, Resistor_SMD:R_0402_1005Metric, F.Cu at (-88.0, 84.0)
- added R51: 220, Resistor_SMD:R_0402_1005Metric, F.Cu at (-74.0, 84.0)
- added R52: 220, Resistor_SMD:R_0402_1005Metric, F.Cu at (-60.0, 84.0)
- added R53: 220, Resistor_SMD:R_0402_1005Metric, F.Cu at (-130.0, 98.0)
- added R54: 220, Resistor_SMD:R_0402_1005Metric, F.Cu at (-116.0, 98.0)
- added R55: 1k, Resistor_SMD:R_0402_1005Metric, F.Cu at (30.0, 14.0)
- added R56: 1k, Resistor_SMD:R_0402_1005Metric, F.Cu at (-40.0, 28.0)
- added R57: 1k, Resistor_SMD:R_0402_1005Metric, F.Cu at (-26.0, 28.0)
- added R58: 1k, Resistor_SMD:R_0402_1005Metric, F.Cu at (-12.0, 28.0)
- added R59: 10k, Resistor_SMD:R_0402_1005Metric, F.Cu at (2.00, 28.0)
- added R60: 10k, Resistor_SMD:R_0402_1005Metric, F.Cu at (16.0, 28.0)
- added R61: 10k, Resistor_SMD:R_0402_1005Metric, F.Cu at (30.0, 28.0)
- added R62: 10k, Resistor_SMD:R_0402_1005Metric, F.Cu at (-40.0, 42.0)
- added R63: 100k, Resistor_SMD:R_0402_1005Metric, F.Cu at (-344.0, 42.0)
- added R64: 10k, Resistor_SMD:R_0402_1005Metric, F.Cu at (-330.0, 42.0)
- added U15: MCP23017-E/SO, Package_SO:SOIC-28W_7.5x17.9mm_P1.27mm, F.Cu at (-60.0, 168.0)
- added U16: TLP290-4, Package_SO:SOP-16_4.55x10.3mm_P1.27mm, F.Cu at (-130.0, 182.0)
- added U17: TLP290-4, Package_SO:SOP-16_4.55x10.3mm_P1.27mm, F.Cu at (-116.0, 182.0)
- added U18: TPD4E05U06DQA, Package_SON:USON-10_2.5x1.0mm_P0.5mm, F.Cu at (30.0, 42.0)
- J11, J12, J13, J14, J15, J16, J17, J18: footprint Connector_JST:JST_PH_B4B-PH-K_1x04_P2.00mm_Vertical -> Connector_JST:JST_PH_B5B-PH-K_1x05_P2.00mm_Vertical
- U1: value ESP32-C6-MINI-1-N4 -> ESP32-C6-WROOM-1-N8; footprint RF_Module:ESP32-C6-MINI-1 -> granite:ESP32-C6-WROOM-1
- moved R104 75.4 mm to (-60.0, 98.0)
- moved R110 75.4 mm to (-60.0, 112.0)
- moved R116 75.4 mm to (-60.0, 126.0)
- moved R206 75.4 mm to (-60.0, 140.0)
- moved R212 75.4 mm to (-60.0, 154.0)
- moved D3 71.4 mm to (-400.0, 28.0)
- moved J15 71.4 mm to (-130.0, 14.0)
- moved K15 71.4 mm to (-130.0, 56.0)
- moved K3 71.4 mm to (-130.0, 28.0)
- moved K9 71.4 mm to (-130.0, 42.0)
- moved R1 71.4 mm to (-400.0, 42.0)
- moved RN1 70.0 mm to (-26.0, 42.0)
- moved D6 56.0 mm to (16.0, 0.00)
- moved D7 56.0 mm to (30.0, 0.00)
- moved R101 44.3 mm to (-102.0, 98.0)
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Connections:
- J11 pad 1: /Relay channels/MB1_RST_A -> /Relay channels/MB1_PWR_B
- J11 pad 3: /Relay channels/MB1_PWR_A -> /Relay channels/MB1_COM
- J11 pad 4: /Relay channels/MB1_PWR_B -> /Relay channels/MB1_PLED_P
- J12 pad 1: /Relay channels/MB2_RST_A -> /Relay channels/MB2_PWR_B
- J12 pad 3: /Relay channels/MB2_PWR_A -> /Relay channels/MB2_COM
- J12 pad 4: /Relay channels/MB2_PWR_B -> /Relay channels/MB2_PLED_P
- J13 pad 1: /Relay channels/MB3_RST_A -> /Relay channels/MB3_PWR_B
- J13 pad 3: /Relay channels/MB3_PWR_A -> /Relay channels/MB3_COM
- J13 pad 4: /Relay channels/MB3_PWR_B -> /Relay channels/MB3_PLED_P
- J14 pad 1: /Relay channels/MB4_RST_A -> /Relay channels/MB4_PWR_B
- J14 pad 3: /Relay channels/MB4_PWR_A -> /Relay channels/MB4_COM
- J14 pad 4: /Relay channels/MB4_PWR_B -> /Relay channels/MB4_PLED_P
- J15 pad 1: /Relay channels/MB5_RST_A -> /Relay channels/MB5_PWR_B
- J15 pad 3: /Relay channels/MB5_PWR_A -> /Relay channels/MB5_COM
- J15 pad 4: /Relay channels/MB5_PWR_B -> /Relay channels/MB5_PLED_P
- J16 pad 1: /Relay channels/MB6_RST_A -> /Relay channels/MB6_PWR_B
- J16 pad 3: /Relay channels/MB6_PWR_A -> /Relay channels/MB6_COM
- J16 pad 4: /Relay channels/MB6_PWR_B -> /Relay channels/MB6_PLED_P
- J17 pad 1: /Relay channels/MB7_RST_A -> /Relay channels/MB7_PWR_B
- J17 pad 3: /Relay channels/MB7_PWR_A -> /Relay channels/MB7_COM
- J17 pad 4: /Relay channels/MB7_PWR_B -> /Relay channels/MB7_PLED_P
- J18 pad 1: /Relay channels/MB8_RST_A -> /Relay channels/MB8_PWR_B
- J18 pad 3: /Relay channels/MB8_PWR_A -> /Relay channels/MB8_COM
- J18 pad 4: /Relay channels/MB8_PWR_B -> /Relay channels/MB8_PLED_P
- K1 pad 6: /Relay channels/MB1_RST_A -> /Relay channels/MB1_COM
- K10 pad 6: /Relay channels/MB5_PWR_A -> /Relay channels/MB5_COM
- K11 pad 6: /Relay channels/MB6_RST_A -> /Relay channels/MB6_COM
- K12 pad 6: /Relay channels/MB6_PWR_A -> /Relay channels/MB6_COM
- K13 pad 6: /Relay channels/MB7_RST_A -> /Relay channels/MB7_COM
- K14 pad 6: /Relay channels/MB7_PWR_A -> /Relay channels/MB7_COM
- K15 pad 6: /Relay channels/MB8_RST_A -> /Relay channels/MB8_COM
- K16 pad 6: /Relay channels/MB8_PWR_A -> /Relay channels/MB8_COM
- K2 pad 6: /Relay channels/MB1_PWR_A -> /Relay channels/MB1_COM
- K3 pad 6: /Relay channels/MB2_RST_A -> /Relay channels/MB2_COM
- K4 pad 6: /Relay channels/MB2_PWR_A -> /Relay channels/MB2_COM
- K5 pad 6: /Relay channels/MB3_RST_A -> /Relay channels/MB3_COM
- K6 pad 6: /Relay channels/MB3_PWR_A -> /Relay channels/MB3_COM
- K7 pad 6: /Relay channels/MB4_RST_A -> /Relay channels/MB4_COM
- K8 pad 6: /Relay channels/MB4_PWR_A -> /Relay channels/MB4_COM
- K9 pad 6: /Relay channels/MB5_RST_A -> /Relay channels/MB5_COM
- RN2 pad 8: GPIO_IO5 -> unconnected-(RN2-R1.2-Pad8)
- U1 pad 10: GPIO_IO5 -> GPIO_IO8
- U1 pad 11: GND -> EXP_nRESET_INT
- U1 pad 12: EXP_INT -> unconnected-(U1-IO11-Pad12)
- U1 pad 13: /MCU/LED_HB -> /MCU/C6_USB_D-
- U1 pad 14: GND -> /MCU/C6_USB_D+
- U1 pad 15: I2C_EXT_SDA -> /MCU/C6_BOOT
- U1 pad 16: I2C_EXT_SCL -> ETH_CS
- U1 pad 17: /MCU/C6_USB_D- -> ETH_SCLK
- U1 pad 18: /MCU/C6_USB_D+ -> ETH_MOSI
- U1 pad 19: EXP_nRESET_INT -> ETH_MISO
- U1 pad 2: GND -> +3V3
- U1 pad 20: GPIO_IO15 -> ETH_INT
- U1 pad 21: unconnected-(U1-NC-Pad21) -> ETH_RST
- U1 pad 22: GPIO_IO8 -> unconnected-(U1-NC-Pad22)
- U1 pad 23: /MCU/C6_BOOT -> GPIO_IO15
- U1 pad 24: ETH_CS -> /MCU/OW_MCU
- U1 pad 25: ETH_SCLK -> /MCU/OW_MCU
- U1 pad 26: ETH_MOSI -> I2C_INT_SCL
- U1 pad 27: ETH_MISO -> I2C_INT_SDA
- U1 pad 28: ETH_INT -> GND
- U1 pad 29: ETH_RST -> GND
- U1 pad 3: +3V3 -> /MCU/C6_EN
- U1 pad 4: unconnected-(U1-NC-Pad4) -> EXP_nRESET
- U1 pad 5: I2C_INT_SDA -> VIN_SENSE
- U1 pad 6: I2C_INT_SCL -> I2C_EXT_SDA
- U1 pad 7: unconnected-(U1-NC-Pad7) -> I2C_EXT_SCL
- U1 pad 8: /MCU/C6_EN -> EXP_INT
- U1 pad 9: EXP_nRESET -> /MCU/LED_HB

Commit message: Board outline 180 x 40 mm with corner M3 holes
tools/outline.py adds the Edge.Cuts rectangle (1 mm corners) and four
board-only M3 NPTH holes 4 mm in from each corner; it is idempotent so
it can be re-run after mkboard. mkboard now parks parts left of x = 0
so the parking grid stays off the outline.
Parts:
- added H1: MountingHole_3.2mm_M3, MountingHole:MountingHole_3.2mm_M3, F.Cu at (4.00, 4.00)
- added H2: MountingHole_3.2mm_M3, MountingHole:MountingHole_3.2mm_M3, F.Cu at (176.0, 4.00)
- added H3: MountingHole_3.2mm_M3, MountingHole:MountingHole_3.2mm_M3, F.Cu at (176.0, 36.0)
- added H4: MountingHole_3.2mm_M3, MountingHole:MountingHole_3.2mm_M3, F.Cu at (4.00, 36.0)
- moved C10 160.0 mm to (-400.0, 0.00)
- moved C11 160.0 mm to (-470.0, 14.0)
- moved C12 160.0 mm to (-380.0, 0.00)
- moved C13 160.0 mm to (-366.0, 0.00)
- moved C14 160.0 mm to (-352.0, 0.00)
- moved C15 160.0 mm to (-338.0, 0.00)
- moved C2 160.0 mm to (-560.0, 0.00)
- moved C26 160.0 mm to (-456.0, 14.0)
- moved C27 160.0 mm to (-442.0, 14.0)
- moved C28 160.0 mm to (-428.0, 14.0)
- moved C29 160.0 mm to (-414.0, 14.0)
- moved C3 160.0 mm to (-546.0, 0.00)
- moved C30 160.0 mm to (-400.0, 14.0)
- moved C31 160.0 mm to (-470.0, 28.0)
- moved C32 160.0 mm to (-456.0, 28.0)
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Other:
- board outline added: 180 x 40 mm

Commit message: Board 230 x 40 mm and first grouped placement
180 mm left the relay section ~90 % full; 230 mm gives ~70 %.
tools/place.py anchors the big parts (RJ45 and USB-C on the top edge,
WROOM antenna over the bottom edge, node connectors in two rows of
four) and packs the rest per sheet. DRC with project rules: no copper
or courtyard errors; silkscreen overlaps and routing remain.
Parts:
- moved R1 583.0 mm to (22.0, 7.01)
- moved U2 580.9 mm to (19.6, 17.7)
- moved D3 579.2 mm to (19.0, 13.8)
- moved C2 572.5 mm to (12.5, 3.44)
- moved U8 571.7 mm to (24.6, 20.7)
- moved R2 571.5 mm to (24.5, 7.01)
- moved C43 569.0 mm to (8.96, 7.00)
- moved C3 565.2 mm to (19.2, 2.02)
- moved R37 560.1 mm to (27.0, 7.01)
- moved C44 558.3 mm to (12.2, 7.53)
- moved D8 557.7 mm to (11.5, 14.8)
- moved F3 557.5 mm to (25.3, 13.2)
- moved C4 555.2 mm to (23.2, 2.02)
- moved C45 548.3 mm to (16.2, 7.53)
- moved R38 546.0 mm to (27.0, 8.52)
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Other:
- board size 180 x 40 mm -> 230 x 40 mm
