File: power/pm-19v-200w/pm-19v-200w.kicad_sch (KiCad schematic)
At the start: 58 parts, among them J1 Brick 1/8 (DOSA), J2 Aux, Q1 BSC070N10NS5, Q2 BSC070N10NS5, Q3 BSC070N10NS5, Q4 BSC070N10NS5, U1 LTC7810, U2 MCP65R46-1.21 (OV), U3 MCP65R46-1.21 (PG)

Commit message: pm-19v-200w: redraw the schematic with wires, power flow left to right, notes on sheet
Parts:
- C1, C2, C3, C4, C5, C6, C7, C8: value 2.2u 100V 1210 -> 2.2u
- C20, C21, C22, C23: value 22u 35V 1210 -> 22u
- C24, C25: value 100u 35V polymer -> 100u
- U2: value MCP65R46-1.21 (OV) -> MCP65R46-1.21
- U3: value MCP65R46-1.21 (PG) -> MCP65R46-1.21
Connections:
- net GND: now also U1.4 (PLLIN/SPREAD)
- net INTVCC: no longer U1.4 (PLLIN/SPREAD)
- net FB: no longer names the net of C12.2, R6.2, R7.1, U1.47 (VFB1)
- net ITH1: no longer names the net of C14.1, R8.1, U1.46 (ITH1)
- net ITH1_RC: no longer names the net of C13.1, R8.2
- net ITH2: no longer names the net of C16.1, U1.15 (ITH2)
- net OV_SNS: no longer names the net of R12.2, R13.1, U2.4 (-)
- net PG_SNS: no longer names the net of R14.2, R15.1, U3.3 (+)
- net SS1: no longer names the net of C15.1, U1.45 (TRACK/SS1)
- net SS2: no longer names the net of C17.1, U1.16 (TRACK/SS2)
Other:
- note added: "C1-C8: 2.2 uF 100 V X7R 1210 (~1 uF left at 54 V). C20-C23: 22 uF 35 V X7R 1210."
- note added: "C24, C25: 100 uF 35 V solid polymer. No wet electrolytics (immersion)."
- note added: "Current limit: 67 mV min / 8 mOhm = 8.4 A peak per phase, ~14 A DC total."
- note added: "DRVSET open: 10 V gate drive. NDRV = DRVCC (NDRV LDO unused). EXTVCC = VOUT once running."
- note added: "MOSFETs, inductors, compensation: first estimates, not verified."
- note added: "Notes"
- note added: "OV_KILL low above ~22.7 V, PGOOD high above ~17.3 V; comparators run from VAUX (VIN, 47k, 4.7 V zener)."
- note added: "PLLIN/SPREAD = GND: no sync, no spread spectrum. MODE = INTVCC: forced continuous."
- note added: "Two-phase: VFB2 = INTVCC, RUN2 = RUN1, ITH2 / TRACK/SS2 to 1 nF. FREQ = GND: 200 kHz per phase."
- note added: "UVLO 38.4 V / OVLO 62.7 V via R3-R5. RUN (J1.2) open = on, pulled low = off."

Commit message: pm-19v-200w: footprints, DOSA eighth-brick pin footprint, first placement in 58.4 x 22.9 mm
Parts:
- removed Q1, Q2, Q3, Q4: BSC070N10NS5, symbol Device:Q_NMOS
- added Q1, Q2, Q3, Q4: BSC070N10NS5, Package_TO_SOT_SMD:TDSON-8-1, symbol Transistor_FET:BSC070N10NS5
- C1, C2, C20, C21, C22, C23, C3, C4, C5, C6, C7, C8: footprint (none) -> Capacitor_SMD:C_1210_3225Metric
- C10, C12, C13, C14, C15, C16, C17, C18, C19, C26, C27, C28: footprint (none) -> Capacitor_SMD:C_0603_1608Metric
- C11, C9: footprint (none) -> Capacitor_SMD:C_0805_2012Metric
- C24, C25: footprint (none) -> Capacitor_Tantalum_SMD:CP_EIA-7343-31_Kemet-D
- D1, D2, D3: footprint (none) -> Diode_SMD:D_SOD-323
- J1: footprint (none) -> pm:Brick_Eighth_DOSA
- J2: footprint (none) -> Connector_PinHeader_1.27mm:PinHeader_1x05_P1.27mm_Vertical
- L1, L2: footprint (none) -> Inductor_SMD:L_Coilcraft_XAL1010-XXX
- R1, R12, R13, R14, R15, R16, R4, R5, R6, R7, R8, TH1: footprint (none) -> Resistor_SMD:R_0603_1608Metric
- R10, R9: footprint (none) -> Resistor_SMD:R_2512_6332Metric
- R11: footprint (none) -> Resistor_SMD:R_0805_2012Metric
- R3: footprint (none) -> Resistor_SMD:R_1206_3216Metric
- U1: footprint (none) -> Package_QFP:LQFP-48-1EP_7x7mm_P0.5mm_EP3.6x3.6mm
- U2, U3: footprint (none) -> Package_TO_SOT_SMD:SOT-23-6
Connections:
- net BG1: now also Q2.4 (G)
- net BG2: now also Q4.4 (G)
- net GND: now also Q2.1 (S), Q2.2 (S), Q2.3 (S), Q4.1 (S), Q4.2 (S), Q4.3 (S)
- net SW1: now also Q1.1 (S), Q1.2 (S), Q1.3 (S), Q2.5 (D)
- net SW2: now also Q3.1 (S), Q3.2 (S), Q3.3 (S), Q4.5 (D)
- net TG1: now also Q1.4 (G)
- net TG2: now also Q3.4 (G)
- net VIN: now also Q1.5 (D), Q3.5 (D)

Commit message: pm-19v-200w: LCSC numbers on 52 of 58 parts (schematic and board); handoff: open module parts and brick pin research
Parts:
- C1, C2, C3, C4, C5, C6, C7, C8: LCSC (none) -> C5449052
- C10, C15, C18, C19, C27, C28: LCSC (none) -> C14663
- C11: LCSC (none) -> C354262
- C12: LCSC (none) -> C94904
- C13: LCSC (none) -> C374074
- C14: LCSC (none) -> C1635
- C16, C17: LCSC (none) -> C100040
- C20, C21, C22, C23: LCSC (none) -> C778721
- C26: LCSC (none) -> C380328
- C9: LCSC (none) -> C5370002
- D1, D2: LCSC (none) -> C82466
- D3: LCSC (none) -> C107713
- Q1, Q2, Q3, Q4: LCSC (none) -> C534364
- R1: LCSC (none) -> C22859
- R10, R9: LCSC (none) -> C2904240
- R11: LCSC (none) -> C17713
- R12: LCSC (none) -> C22823
- R13, R15, R16, R7: LCSC (none) -> C25804
- R14: LCSC (none) -> C22870
- R3: LCSC (none) -> C247164
- R4: LCSC (none) -> C22865
- R5: LCSC (none) -> C22898
- R6: LCSC (none) -> C22827
- R8: LCSC (none) -> C22809
- TH1: LCSC (none) -> C13564
- U1: LCSC (none) -> C581067
- U2, U3: LCSC (none) -> C116625

Commit message: power: screwed PM module mount footprints (M2 into SMT standoffs, pogo aux) on module, plane and bench carrier; RUN moves to aux pad 8; copper not yet rerouted
Parts:
- J1: value Brick 1/8 (DOSA) -> PM mount M2; footprint pm:Brick_Eighth_DOSA -> pm:PM_Mount_M2; symbol Connector_Generic:Conn_01x08 -> Connector_Generic:Conn_01x04
- J2: value Aux -> Aux pads (pogo); footprint Connector_PinHeader_1.27mm:PinHeader_1x05_P1.27mm_Vertical -> pm:PM_Aux_Pads_2x04; symbol Connector_Generic:Conn_01x05 -> Connector_Generic:Conn_01x08
Connections:
- net GND: now also J1.2 (Pin_2); no longer J1.4 (Pin_4)
- net RUN: now also J2.8 (Pin_8); no longer J1.2 (Pin_2)
- net VOUT: now also J1.4 (Pin_4); no longer J1.8 (Pin_8)
- no-connect marks 4 -> 3
Other:
- note added: "UVLO 38.4 V / OVLO 62.7 V via R3-R5. RUN (J2.8, aux pad) open = on, pulled low = off."
- note removed: "UVLO 38.4 V / OVLO 62.7 V via R3-R5. RUN (J1.2) open = on, pulled low = off."

Commit message: Revert "power: screwed PM module mount footprints (M2 into SMT standoffs, pogo aux) on module, plane and bench carrier; RUN moves to aux pad 8; copper not yet rerouted"
This reverts commit abb9f50ba34d0b63e5425fa3cd376420f2890e7d.
Parts:
- J1: value PM mount M2 -> Brick 1/8 (DOSA); footprint pm:PM_Mount_M2 -> pm:Brick_Eighth_DOSA; symbol Connector_Generic:Conn_01x04 -> Connector_Generic:Conn_01x08
- J2: value Aux pads (pogo) -> Aux; footprint pm:PM_Aux_Pads_2x04 -> Connector_PinHeader_1.27mm:PinHeader_1x05_P1.27mm_Vertical; symbol Connector_Generic:Conn_01x08 -> Connector_Generic:Conn_01x05
Connections:
- net GND: now also J1.4 (Pin_4); no longer J1.2 (Pin_2)
- net RUN: now also J1.2 (Pin_2); no longer J2.8 (Pin_8)
- net VOUT: now also J1.8 (Pin_8); no longer J1.4 (Pin_4)
- no-connect marks 3 -> 4
Other:
- note added: "UVLO 38.4 V / OVLO 62.7 V via R3-R5. RUN (J1.2) open = on, pulled low = off."
- note removed: "UVLO 38.4 V / OVLO 62.7 V via R3-R5. RUN (J2.8, aux pad) open = on, pulled low = off."
