File: power/pp-48/sheets/input.kicad_sch (KiCad schematic)
At the start: 28 parts, among them J1 XT90PW-M, Q2 BSC040N10NS5, Q3 BSC040N10NS5, Q4 2N7002, U7 LM5069MM-1, U8 INA238AIDGSR

Commit message: pp-48: TVS polarity fix (slot clamp SMBJ60A and bus TVS SMDJ60A are unidirectional: cathode pad 1 now on OUT / VIN, symbol Device:D_Zener; they had pad 1 on GND and would have shorted the rail); Input resistors renumbered R33-R38 (collided with the 3V3 buck's R3-R8); handoff notes the same bug in pp-48-2s
Parts:
- removed R3: 143k, Resistor_SMD:R_0805_2012Metric, symbol Device:R
- removed R4, R8: 10k, Resistor_SMD:R_0402_1005Metric, symbol Device:R
- removed R5: 124k, Resistor_SMD:R_0805_2012Metric, symbol Device:R
- removed R6: 4.99k, Resistor_SMD:R_0402_1005Metric, symbol Device:R
- removed R7: 10.2k, Resistor_SMD:R_0402_1005Metric, symbol Device:R
- added R33: 143k, Resistor_SMD:R_0805_2012Metric, symbol Device:R
- added R34, R38: 10k, Resistor_SMD:R_0402_1005Metric, symbol Device:R
- added R35: 124k, Resistor_SMD:R_0805_2012Metric, symbol Device:R
- added R36: 4.99k, Resistor_SMD:R_0402_1005Metric, symbol Device:R
- added R37: 10.2k, Resistor_SMD:R_0402_1005Metric, symbol Device:R
- D1: symbol Device:D_TVS -> Device:D_Zener
Connections:
- net +3V3: now also R38.1
- net GND: now also D1.2 (A), R34.2, R36.2, R37.2; no longer D1.1 (A1)
- net OVLO: now also R35.2, R36.1
- net PWR: now also R37.1
- net TILE_PGD: now also R38.2
- net UVLO: now also R33.2, R34.1
- net VIN: now also D1.1 (K), R33.1, R35.1; no longer D1.2 (A2)
Other:
- moved on the sheet: D1
Changed lines of the file:
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@@
 	)
 	(symbol
-		(lib_id "Device:D_TVS")
-		(at 35.56 68.58 90)
+		(lib_id "Device:D_Zener")
+		(at 35.56 68.58 270)
 		(unit 1)
 		(body_style 1)
@@
 			)
 		)
-		(property "Description" "bus TVS 3 kW: 60 V standoff, breakdown >= 66.7 V, clamp 96.8 V; LCSC code to check"
+		(property "Description" "bus TVS 3 kW, unidirectional: cathode (pad 1) on VIN; 60 V standoff, breakdown >= 66.7 V, clamp 96.8 V; LCSC code to check"
 			(at 35.56 68.58 0)
 			(hide yes)
@@
 		(in_pos_files yes)
 		(dnp no)
-		(property "Reference" "R3"
-			(at 122.666 106.68 0)
+		(property "Reference" "R33"
+			(at 123.166 106.68 0)
 			(show_name no)
 			(do_not_autoplace no)
@@
 			(project "pp-48"
 				(path "/cf0d5c0a-6642-53ea-ac93-0bbad631a43a/e269b960-91e5-5c21-9cb3-23d8112f0bf9"
-					(reference "R3")
+					(reference "R33")
 					(unit 1)
 				)
@@
 		(in_pos_files yes)
 		(dnp no)
-		(property "Reference" "R4"
-			(at 122.666 116.84 0)
+		(property "Reference" "R34"
+			(at 123.166 116.84 0)
 			(show_name no)
 			(do_not_autoplace no)
@@
 			(project "pp-48"
 				(path "/cf0d5c0a-6642-53ea-ac93-0bbad631a43a/e269b960-91e5-5c21-9cb3-23d8112f0bf9"
-					(reference "R4")
+					(reference "R34")
 					(unit 1)
 				)
@@
 		(in_pos_files yes)
 		(dnp no)
-		(property "Reference" "R5"
-			(at 132.826 88.9 0)
+		(property "Reference" "R35"
+			(at 133.326 88.9 0)
 			(show_name no)
 			(do_not_autoplace no)
@@
 			(project "pp-48"
 				(path "/cf0d5c0a-6642-53ea-ac93-0bbad631a43a/e269b960-91e5-5c21-9cb3-23d8112f0bf9"
-					(reference "R5")
+					(reference "R35")
 					(unit 1)
 				)
@@
 		(in_pos_files yes)
 		(dnp no)
-		(property "Reference" "R6"
-			(at 132.826 99.06 0)
+		(property "Reference" "R36"
+			(at 133.326 99.06 0)
 			(show_name no)
 			(do_not_autoplace no)
@@
 			(project "pp-48"
 				(path "/cf0d5c0a-6642-53ea-ac93-0bbad631a43a/e269b960-91e5-5c21-9cb3-23d8112f0bf9"
-					(reference "R6")
+					(reference "R36")
 					(unit 1)
 				)
@@
 		(in_pos_files yes)
 		(dnp no)
-		(property "Reference" "R7"
-			(at 183.626 102.87 0)
+		(property "Reference" "R37"
+			(at 184.126 102.87 0)
 			(show_name no)
 			(do_not_autoplace no)
@@
 			(project "pp-48"
 				(path "/cf0d5c0a-6642-53ea-ac93-0bbad631a43a/e269b960-91e5-5c21-9cb3-23d8112f0bf9"
-					(reference "R7")
+					(reference "R37")
 					(unit 1)
 				)
@@
 		(in_pos_files yes)
 		(dnp no)
-		(property "Reference" "R8"
-			(at 196.326 85.09 0)
+		(property "Reference" "R38"
+			(at 196.826 85.09 0)
 			(show_name no)
 			(do_not_autoplace no)
@@
 			(project "pp-48"
 				(path "/cf0d5c0a-6642-53ea-ac93-0bbad631a43a/e269b960-91e5-5c21-9cb3-23d8112f0bf9"
-					(reference "R8")
-					(unit 1)
-				)
+					(reference "R38")
+					(unit 1)
+				)

Commit message: pp-48: board routed with the core (N = 2, 106 x 72): DRC 0 unconnected / 0 parity / 0 errors, old track_dangling exclusions gone; route_hand.py core(): tile VIN / TSENSE / VBUS copper, Kelvin sense for U7 / U8, In2 channel rows under the VBUS via field to a via ladder and the mux, +3V3 trunk end, CTRL_GND pours with a 2 mm isolation band; tools/netsplit.py renames +3V3 and COLn per column around krt-route (KRT does not count In2 tracks as connections); gndstitch also stitches CTRL_GND; copycol keeps the core routes; placement changes in core.py; J1 retention pegs on GND; core channel limited to N <= 4
Connections:
- net GND: now also J1.MP (MountPin)
- no-connect marks 1 -> 0
