File: power/pp-48/sheets/mux.kicad_sch (KiCad schematic)
At the start: 5 parts, among them Q6 2N7002, U6 TCA9548APWR

Commit message: pp-48: schematic as 2-slot units (ADR 0004 decision 9): sheets/unit.kicad_sch replaces column.kicad_sch, instantiated N/2 times (refs +100 per unit, slot B +50, nets A_* / B_*); TCA6424ARGJR U5 (0x22, LCSC C80692, pp symbol added, VQFN-32 EP3.15) with C9 / C13 / R30 and the segment pull-ups once per unit; slot B straps INA238 A0 and ADC ADR0 to +3V3 (0x41 / 0x52); root nets UNITu_SDA / SCL, mux channel k = unit k+1; ERC 0
Connections:
- net COL1_SCL renamed UNIT1_SCL
- net COL1_SDA renamed UNIT1_SDA
- net COL2_SCL: no longer names the net of U6.7 (SC1)
- net COL2_SDA: no longer names the net of U6.6 (SD1)
- no-connect marks 12 -> 14
Other:
- note added: "I2C SWITCH U6 TCA9548A 0x70, channel k = unit k + 1"
- note removed: "I2C SWITCH U6 TCA9548A 0x70, channel k = column k + 1"
Changed lines of the file:
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@@
+	)
+	(no_connect
+		(at 111.76 78.74)
+	)
+	(no_connect
+		(at 111.76 76.2)
 	)
 	(no_connect
@@
 		)
 	)
-	(hierarchical_label "COL1_SDA"
+	(hierarchical_label "UNIT1_SDA"
 		(shape bidirectional)
 		(at 111.76 73.66 0)
@@
 		)
 	)
-	(hierarchical_label "COL1_SCL"
+	(hierarchical_label "UNIT1_SCL"
 		(shape bidirectional)
 		(at 111.76 71.12 0)
-		(effects
-			(font
-				(size 1.27 1.27)
-			)
-			(justify left)
-		)
-	)
-	(hierarchical_label "COL2_SDA"
-		(shape bidirectional)
-		(at 111.76 78.74 0)
-		(effects
-			(font
-				(size 1.27 1.27)
-			)
-			(justify left)
-		)
-	)
-	(hierarchical_label "COL2_SCL"
-		(shape bidirectional)
-		(at 111.76 76.2 0)
 		(effects
 			(font
@@
 		)
 	)
-	(text "I2C SWITCH  U6 TCA9548A 0x70, channel k = column k + 1"
+	(text "I2C SWITCH  U6 TCA9548A 0x70, channel k = unit k + 1"
 		(exclude_from_sim no)
 		(at 38.1 50.8 0)
@@
 			)
 		)
-		(property "Description" "I2C switch, 0x70; channel k = column k + 1"
+		(property "Description" "I2C switch, 0x70; channel k = unit k + 1"
 			(at 101.6 88.9 0)
 			(hide yes)
