File: power/pp-48/sheets/unit.kicad_sch (KiCad schematic)
At the start: 120 parts, among them J101 NODE 19V, J102 FRONT PANEL, J103 AUX, J151 NODE 19V, J152 FRONT PANEL, J153 AUX, Q101 BSC070N10NS5, Q102 2N7002, Q103 2N7002, Q104 2N7002, Q105 2N7002, Q106 2N7002, Q107 2N7002, Q108 2N7002, Q109 2N7002, Q151 BSC070N10NS5, Q152 2N7002, Q153 2N7002, Q154 2N7002, Q155 2N7002, Q156 2N7002, Q157 2N7002, Q158 2N7002, Q159 2N7002, U101 LM5069MM-2, U102 INA238AIDGSR, U103 74LVC1G74, U104 ADC121C027CIMK, U105 TCA6424ARGJR, U106 TLP176AM, U107 TLP176AM, U108 TLP291, U110 74LVC1G74, U151 LM5069MM-2, U152 INA238AIDGSR, U153 74LVC1G74, U154 ADC121C027CIMK, U156 TLP176AM, U157 TLP176AM, U158 TLP291, U160 74LVC1G74

Commit message: pp-48: board routed as 2-slot units (N = 2, 106 x 72): DRC 0 unconnected / 0 parity / 0 errors (3 silk warnings, core D1); expander U5 in slot B, slot A's 11 lines on an In2 bus between via ladders (pad-via footprints, KRT routes only to pads), In2 no-via band and F rule areas over the SENSE pours (KRT ignores both), U10 PGD escape, J3 GND pins joined, 4 vias in U5's exposed pad; place.py slot table for both slots + unit parts, photoMOS stack 0.6 mm lower; route_hand.py channel / trunk / fences per unit (incl. last unit edge); netsplit.py per unit + slot A expander nets split at the bus; copycol.py unit pitch 50; expander ports reordered to the bus ladder; ADR 0004 decision 9 layout note; handoff
Connections:
- net A_LCLR: now also U105.5 (P04); no longer U105.9 (P10)
- net A_LED: now also U105.9 (P10); no longer U105.7 (P06)
- net A_OVK: now also U105.6 (P05); no longer U105.10 (P11)
- net A_PG: now also U105.7 (P06); no longer U105.11 (P12)
- net A_PWRD: now also U105.10 (P11); no longer U105.5 (P04)
- net A_RSTD: now also U105.11 (P12); no longer U105.6 (P05)
- net A_RUNOFF: now also U105.8 (P07); no longer U105.12 (P13)
- net B_DISARM: now also U105.23 (P26); no longer U105.16 (P17)
- net B_LCLR: now also U105.19 (P22); no longer U105.20 (P23)
- net B_LQ: now also U105.20 (P23); no longer U105.21 (P24)
- net B_OFF: now also U105.22 (P25); no longer U105.23 (P26)
- net B_OVK: now also U105.18 (P21); no longer U105.19 (P22)
- net B_PG: now also U105.17 (P20); no longer U105.18 (P21)
- net B_PGD: now also U105.21 (P24); no longer U105.22 (P25)
- net B_RUNOFF: now also U105.16 (P17); no longer U105.17 (P20)
Changed lines of the file:
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@@
 	)
 	(no_connect
-		(at 114.3 227.33)
+		(at 114.3 240.03)
 	)
 	(no_connect
@@
 		)
 	)
-	(label "A_PWRD"
+	(label "A_LCLR"
 		(at 114.3 219.71 0)
 		(effects
@@
 		)
 	)
-	(label "A_RSTD"
+	(label "A_OVK"
 		(at 114.3 222.25 0)
 		(effects
@@
 		)
 	)
-	(label "A_LED"
+	(label "A_PG"
 		(at 114.3 224.79 0)
 		(effects
@@
 		)
 	)
-	(label "A_LCLR"
-		(at 114.3 232.41 0)
+	(label "A_RUNOFF"
+		(at 114.3 227.33 0)
 		(effects
 			(font
@@
 		)
 	)
-	(label "A_OVK"
-		(at 114.3 234.95 0)
+	(label "A_LED"
+		(at 114.3 232.41 0)
 		(effects
 			(font
@@
 		)
 	)
-	(label "A_PG"
-		(at 114.3 237.49 0)
+	(label "A_PWRD"
+		(at 114.3 234.95 0)
 		(effects
 			(font
@@
 		)
 	)
-	(label "A_RUNOFF"
-		(at 114.3 240.03 0)
+	(label "A_RSTD"
+		(at 114.3 237.49 0)
 		(effects
 			(font
@@
 		)
 	)
-	(label "B_DISARM"
+	(label "B_RUNOFF"
 		(at 114.3 250.19 0)
 		(effects
@@
 		)
 	)
-	(label "B_RUNOFF"
+	(label "B_PG"
 		(at 114.3 255.27 0)
 		(effects
@@
 		)
 	)
-	(label "B_PG"
+	(label "B_OVK"
 		(at 114.3 257.81 0)
 		(effects
@@
 		)
 	)
-	(label "B_OVK"
+	(label "B_LCLR"
 		(at 114.3 260.35 0)
 		(effects
@@
 		)
 	)
-	(label "B_LCLR"
+	(label "B_LQ"
 		(at 114.3 262.89 0)
 		(effects
@@
 		)
 	)
-	(label "B_LQ"
+	(label "B_PGD"
 		(at 114.3 265.43 0)
 		(effects
@@
 		)
 	)
-	(label "B_PGD"
+	(label "B_OFF"
 		(at 114.3 267.97 0)
 		(effects
@@
 		)
 	)
-	(label "B_OFF"
+	(label "B_DISARM"
 		(at 114.3 270.51 0)
 		(effects
@@
 			)
 		)
-		(property "Description" "unit GPIO, address 0x22 (ADDR GND); 11 lines per slot: slot A P00-P07 / P10-P12, slot B P13-P17 / P20-P26 (P0 left, P1 bottom, P2 right side of the package at rot 0); INT unused (polled); all inputs after reset"
+		(property "Description" "unit GPIO in slot B, address 0x22 (ADDR GND); 11 lines per slot: slot A P00-P07 / P10-P12 (to slot A over the In2 bus), slot B P14-P17 / P20-P26; INT unused (polled); all inputs after reset"
 			(at 101.6 241.3 0)
 			(hide yes)
