File: power/pp-48-core/sheets/input.kicad_sch (KiCad schematic)
At the start: 7 parts, among them J1 XT30PW-M

Commit message: pp-48 chained plane: LCSC codes for the input TVS (SMDJ60A C2990209), bulk cap (RVT2A470M1010 C87862) and unit shunts (6 mOhm SMA25A3FR006T C2692028), stock rechecked on JLCPCB's own API (jlcsearch mirror stale: mux, FET, 7 mOhm shunts are in stock); LM5069MM-1 down to 1; handoff
Parts:
- C1: LCSC (none) -> C87862; MPN (none) -> Lelon RVT2A470M1010
- D1: LCSC (none) -> C2990209
Changed lines of the file:
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@@
 			)
 		)
-		(property "Description" "bus TVS 3 kW, unidirectional: cathode (pad 1) on VIN; 60 V standoff, breakdown >= 66.7 V, clamp 96.8 V; LCSC code to check"
+		(property "Description" "bus TVS 3 kW, unidirectional: cathode (pad 1) on VIN; 60 V standoff, breakdown >= 66.7 V, clamp 96.8 V"
 			(at 35.56 68.58 0)
 			(hide yes)
@@
 			)
 		)
-		(property "LCSC" ""
+		(property "LCSC" "C2990209"
 			(at 35.56 68.58 0)
 			(hide yes)
@@
 			)
 		)
-		(property "Description" "input bulk, damps the ringing of a live plug-in; LCSC code to check"
+		(property "Description" "input bulk, damps the ringing of a live plug-in"
 			(at 50.8 68.58 0)
 			(hide yes)
@@
 			)
 		)
-		(property "LCSC" ""
+		(property "LCSC" "C87862"
 			(at 50.8 68.58 0)
 			(hide yes)
+			(show_name no)
+			(do_not_autoplace no)
+			(effects
+				(font
+					(size 1.27 1.27)
+				)
+				(justify left)
+			)
+		)
+		(property "MPN" "Lelon RVT2A470M1010"
+			(at 50.8 68.58 0)
+			(hide yes)

Commit message: pp-48-core: GND stitch (1 via), silk (23 refs placed, 71 small ones hidden), JLC outputs; LCSC codes for the 25 passive values that had none (sch/draw.py BASIC table, JLC parts API: basic where JLC has one), copied onto the routed board; BOM 86 parts, left out only CV1/CV2, holes, J5 / JP1-3 (copper only) and DNP R28 / R29; DRC 0 unconnected, parity clean, isocheck clean
Parts:
- R15: LCSC (none) -> C17556
Changed lines of the file:
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@@
 			)
 		)
-		(property "LCSC" ""
+		(property "LCSC" "C17556"
 			(at 58.42 134.62 0)
 			(hide yes)

Commit message: pp-48-core J1: project footprint pp48:AMASS_XT30PW-M (the stock one points to a STEP KiCad does not ship) with the LCSC / EasyEDA model C431092 (pp48.3dshapes), turned 180 and offset (-2.5, 8.48) to sit on the pins and pegs (checked in a top / bottom render); J1 on the routed board updated in place; ERC 0, DRC unchanged
Parts:
- J1: footprint Connector_AMASS:AMASS_XT30PW-M_1x02_P2.50mm_Horizontal -> pp48:AMASS_XT30PW-M_1x02_P2.50mm_Horizontal
Changed lines of the file:
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@@
 			)
 		)
-		(property "Footprint" "Connector_AMASS:AMASS_XT30PW-M_1x02_P2.50mm_Horizontal"
+		(property "Footprint" "pp48:AMASS_XT30PW-M_1x02_P2.50mm_Horizontal"
 			(at 22.86 58.42 0)
 			(hide yes)
