File: controller/schematic/power.kicad_sch (KiCad schematic)
At the start: 29 parts, among them J3 19V_IN, U2 TLV62569DBV, U8 LMR51430YDDCR

Commit message: controller: rev D schematic - node section (relays sheet: J11-J18, K1-K16, U14-U17 and passives), J8 expansion header network (RN2, U7, F2, D7, R19, EXP_nRESET) and the 19 V input (J3, F3, D1, D8) removed; two 12 V PH 2p inputs J11 / J12 OR-ed by SS34 D10 / D11 with SMAJ15A D12 (C148216), VIN_SENSE divider 68k / 10k; new Plane link sheet: J13 / J14 PH 5p, 2.2k SDA / SCL and 10k EXP_INT pull-ups, 33R series, TPD4E05U06 U19 / U20, TPS2553DBVR load switches U21 / U22 (C55266, R_ILIM 180k, 129-174 mA) with a granite:TPS2553DBV symbol; MCU: plane link on GPIO2/3, TMP1075 and J9 on the local bus GPIO6/7, dry inputs on GPIO10/11/4/15, rev C GPIO4 pull-down gone; title blocks rev D; ERC 0, netlist pin map checked
Parts:
- removed D1: SMAJ22A, Diode_SMD:D_SMA, symbol Device:D_Zener
- removed D8: SS34, Diode_SMD:D_SMA, symbol Device:D_Schottky
- removed F3: PTC 0.75A, Fuse:Fuse_1206_3216Metric, symbol Device:Polyfuse
- removed J3: 19V_IN, Connector_JST:JST_PH_B2B-PH-K_1x02_P2.00mm_Vertical, symbol Connector_Generic:Conn_01x02
- added D10, D11: SS34, Diode_SMD:D_SMA, symbol Device:D_Schottky
- added D12: SMAJ15A, Diode_SMD:D_SMA, symbol Device:D_Zener
- added J11: 12V_IN_A, Connector_JST:JST_PH_B2B-PH-K_1x02_P2.00mm_Vertical, symbol Connector_Generic:Conn_01x02
- added J12: 12V_IN_B, Connector_JST:JST_PH_B2B-PH-K_1x02_P2.00mm_Vertical, symbol Connector_Generic:Conn_01x02
- R63: value 100k -> 68k; LCSC C25741 -> C36871; MPN 0402WGF1003TCE -> 0402WGF6802TCE
Connections:
- net GND: now also D12.2 (A), J11.2 (Pin_2), J12.2 (Pin_2)
- net VIN_19V renamed VIN_12V
- net VIN_12V: now also D10.1 (K), D11.1 (K), D12.1 (K)
- new net 12V_IN_A: D10.2 (A), J11.1 (Pin_1)
- new net 12V_IN_B: D11.2 (A), J12.1 (Pin_1)
Other:
- note added: "12 V input: two plane aux feeds (plane J4: PH 2p, 1 CTRL_12V, 2 CTRL_GND) -> one SS34 each (OR-ing + reverse polarity) -> SMAJ15A -> LMR51430 buck (1.1 MHz) -> 5.2 V. No fuse: the plane iso module limits its own output."
- note added: "5 V: 12 V buck or USB VBUS (bench), Schottky OR-ing"
- note added: "BUCK_5V = 0.6 V x (1 + 100k/12.4k) = 5.44 V, so +5V is ~5.0 V loaded after D2. D9 SMAJ6.0A crowbars BUCK_5V if U8 fails short (the plane module current-limits). SMAJ15A clamps (24.4 V) below the LMR51430 36 V / 38 V abs max."
- note added: "BUCK_5V from the 12 V input stage below"
- note added: "VIN_SENSE = VIN_12V x 10k / 78k (68k/10k) -> ESP32 GPIO5 (ADC1). 12 V -> 1.54 V, 24.4 V clamp -> 3.13 V."
- note removed: "19 V input: redundant 19 V bus, tapped upstream of the per-node hot-swap channels -> PTC, TVS, reverse-polarity Schottky -> LMR51430 buck (1.1 MHz) -> 5.2 V"
- note removed: "5 V: 19 V buck or USB VBUS (bench), Schottky OR-ing"
- note removed: "BUCK_5V = 0.6 V x (1 + 100k/12.4k) = 5.44 V, so +5V is ~5.0 V loaded after D2. D9 SMAJ6.0A crowbars BUCK_5V if U8 fails short (F3 trips). SMAJ22A clamps below the LMR51430 38 V abs max."
- note removed: "BUCK_5V from the 19 V input stage below"
- note removed: "VIN_SENSE = VIN_19V / 11 (100k/10k) -> ESP32 GPIO5 (ADC1). 19 V -> 1.73 V, 36 V clamp -> 3.27 V."
- title: Granite Controller - Power -> Granite controller rev D - Power
