File: controller/granite-controller.kicad_pcb (KiCad board)
At the start: 4 copper layers, 105 x 50 mm, 139 parts, among them J1 HR911105A, J10 DRY_IN, J11 12V_IN_A, J12 12V_IN_B, J13 PLANE_LINK_A, J14 PLANE_LINK_B, J2 TYPE-C-31-M-12, J4 1WIRE, J5 1WIRE, J6 1WIRE, J7 1WIRE, J9 I2C_SENSOR, U1 ESP32-C6-WROOM-1-N8, U18 TPD4E05U06DQA, U19 TPD4E05U06DQA, U2 TLV62569DBV, U20 TPD4E05U06DQA, U21 TPS2553DBVR, U22 TPS2553DBVR, U3 W5500, U4 USBLC6-2SC6, U5 TMP1075D, U6 TPD4E05U06DQA, U8 LMR51430YDDCR, Y2 25MHz 12pF YXC

Commit message: controller rev D: probes J4-J7 respaced, J4 body 6.0 mm clear of the RJ45 body (was ~2 mm); place.py keeps 3D model offsets
J4-J7 moved right by 4.06 / 3.97 / 3.88 / 3.79 mm on the top edge, 1.5 mm
body gaps, J7 2.2 mm from the USB-C shell (bodies = F.Fab outlines, which
match the 3D models); J1 / J2 untouched. OW_DATA re-routed with
krt-reroute --keep; the 3V3 buck output (L1 / C4) now reaches In2
through two vias beside L1 instead of via J4 pin 1. GND pour, stitching,
silk and connector labels redone. place.py copies the block footprints'
3D model offset / rotation / scale by value (the SWIG vector assignment
left them zero, see 67a10e3). DRC 0 errors, 0 unconnected, parity
clean.
Parts:
- moved J4 4.06 mm to (62.1, 30.9)
- moved J5 3.97 mm to (72.0, 30.9)
- moved J6 3.88 mm to (81.9, 30.9)
- moved J7 3.79 mm to (91.8, 30.9)
Routing:
- net +3V3: track 175.2 -> 156.5 mm, vias 22 -> 24
- net GND: track 466.5 -> 460.5 mm
- net /MCU/OW_DATA: track 65.5 -> 65.4 mm, vias 0 -> 2
Other:
- board text added: "J7"
- board text removed: "J7 1-WIRE"
