File: power/pp-48-unit/pp-48-unit.kicad_pcb (KiCad board)
At the start: 4 copper layers, 76 x 72 mm, 152 parts, among them J1 NODE 19V, J2 FRONT PANEL, J201 XT60PW-M, J3 AUX, J301 CHAIN IN, J302 CHAIN OUT, J51 NODE 19V, J52 FRONT PANEL, J53 AUX, Q1 BSC070N10NS5, Q2 2N7002, Q202 BSC040N10NS5, Q203 BSC040N10NS5, Q204 2N7002, Q3 2N7002, Q4 2N7002, Q5 2N7002, Q51 BSC070N10NS5, Q52 2N7002, Q53 2N7002, Q54 2N7002, Q55 2N7002, Q56 2N7002, Q57 2N7002, Q58 2N7002, Q59 2N7002, Q6 2N7002, Q7 2N7002, Q8 2N7002, Q9 2N7002, U1 LM5069MM-2, U10 74LVC1G74, U2 INA238AIDGSR, U207 LM5069MM-1, U208 INA238AIDGSR, U3 74LVC1G74, U4 ADC121C027CIMK, U5 TCA6424ARGJR, U51 LM5069MM-2, U52 INA238AIDGSR, U53 74LVC1G74, U54 ADC121C027CIMK, U56 TLP176AM, U57 TLP176AM, U58 TLP291, U6 TLP176AM, U60 74LVC1G74, U7 TLP176AM, U8 TLP291

Commit message: pp-48 plane boards: press deadline line (docs/press-deadline-line.md decided: option B + A) on a 14-pin chain (S14B-PH-K-S C157938; 13 PRESS_EN, 14 EXP_RSTN, cable n -> 15 - n, pins v 35..61); unit Q10 / R31 switch the photoMOS LED returns (PRESS_RTN), core U301 74LVC1G123 deadline (pp:74LVC1G123 single-unit copy) on PC6 PRESS_TRIG, PC7 EXP_RSTN to the units' /RESET; ERC 0 both; boards rebuilt and placed, unit 78.5 x 72 with the strip power path re-placed top-down; unit routing tools (route_unit.py hand copper + In2 band / +3V3 trunk, unitsplit.py, route_unit.sh flow): DRC 0 errors, ~10 unconnected at expander U5; core placed, not routed; pmmount.py restored from granite_controller; ADR 0005 decision 4; handoff
Parts:
- added BV100: , , F.Cu at (107.5, 134.8)
- added BV101: , , F.Cu at (108.1, 135.3)
- added BV102: , , F.Cu at (108.7, 135.8)
- added BV103: , , F.Cu at (109.3, 136.3)
- added BV104: , , F.Cu at (109.9, 136.8)
- added BV105: , , F.Cu at (110.5, 137.3)
- added BV106: , , F.Cu at (111.1, 137.8)
- added BV107: , , F.Cu at (111.7, 138.3)
- added BV108: , , F.Cu at (112.3, 138.8)
- added BV109: , , F.Cu at (112.9, 139.3)
- added BV110: , , F.Cu at (113.5, 139.8)
- added BV150: , , F.Cu at (126.6, 134.8)
- added BV151: , , F.Cu at (127.2, 135.3)
- added BV152: , , F.Cu at (127.8, 135.8)
- added BV153: , , F.Cu at (128.4, 136.3)
- added BV154: , , F.Cu at (129.0, 136.8)
- added BV155: , , F.Cu at (129.6, 137.3)
- added BV156: , , F.Cu at (130.2, 137.8)
- added BV157: , , F.Cu at (130.8, 138.3)
- added BV158: , , F.Cu at (131.4, 138.8)
- added BV159: , , F.Cu at (132.0, 139.3)
- added BV160: , , F.Cu at (132.6, 139.8)
- added BV900: , , F.Cu at (150.4, 159.3)
- added BV901: , , F.Cu at (151.0, 158.9)
- added BV902: , , F.Cu at (151.6, 158.4)
- added BV903: , , F.Cu at (152.2, 158.0)
- added BV904: , , F.Cu at (152.8, 157.5)
- added BV905: , , F.Cu at (153.4, 157.1)
- added BV906: , , F.Cu at (154.0, 156.7)
- added BV907: , , F.Cu at (154.6, 156.2)
- added GV202: , , F.Cu at (155.7, 170.5)
- added GV203: , , F.Cu at (161.5, 170.5)
- added PV1B3: , , F.Cu at (134.8, 133.6)
- added PV1B4: , , F.Cu at (138.4, 133.4)
- added PV3A: , , F.Cu at (111.6, 164.9)
- added PV3B: , , F.Cu at (136.6, 164.9)
- added Q10: 2N7002, Package_TO_SOT_SMD:SOT-23, F.Cu at (95.5, 130.0)
- added R31: 100k, Resistor_SMD:R_0402_1005Metric, F.Cu at (95.5, 127.2)
- added RV1: , , F.Cu at (136.0, 131.9)
- added SV8: , , F.Cu at (110.8, 163.2)
- added SV9: , , F.Cu at (109.6, 163.2)
- C202: moved to B.Cu
- J301, J302: footprint Connector_JST:JST_PH_S12B-PH-K_1x12_P2.00mm_Horizontal -> Connector_JST:JST_PH_S14B-PH-K_1x14_P2.00mm_Horizontal
- moved R210 14.1 mm to (157.0, 171.0), turned to 180 degrees
- moved R211 12.0 mm to (162.8, 171.0), turned to 0 degrees
- moved R214 9.81 mm to (155.2, 130.4)
- moved Q204 9.60 mm to (152.4, 130.2)
- moved H3 8.63 mm to (166.3, 126.5)
- moved Q202 7.23 mm to (153.8, 166.2), turned to 90 degrees
- moved C202 6.68 mm to (157.6, 127.0)
- moved C214 5.20 mm to (152.6, 164.0)
- moved C215 5.20 mm to (157.4, 164.0)
- moved Q203 5.12 mm to (159.6, 166.2), turned to 90 degrees
- moved J302 4.72 mm to (162.9, 135.0)
- moved R201 4.22 mm to (154.5, 147.7), turned to 0 degrees
- moved D201 3.14 mm to (156.5, 140.5)
- moved H4 3.04 mm to (166.0, 168.5)
- moved C201 2.75 mm to (156.4, 129.3)
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Connections:
- J302 pad 1: unconnected-(J302-Pin_1-Pad1) -> /EXP_RSTN
- J302 pad 10: /Chain/CH1_SCL -> /Chain/CH2_SDA
- J302 pad 11: /Chain/CH1_SDA -> GND
- J302 pad 12: +3V3 -> /Chain/CH1_SCL
- J302 pad 2: unconnected-(J302-Pin_2-Pad2) -> /PRESS_EN
- J302 pad 3: GND -> unconnected-(J302-Pin_3-Pad3)
- J302 pad 4: /Chain/CH3_SCL -> unconnected-(J302-Pin_4-Pad4)
- J302 pad 5: /Chain/CH3_SDA -> GND
- J302 pad 6: GND -> /Chain/CH3_SCL
- J302 pad 7: /Chain/CH2_SCL -> /Chain/CH3_SDA
- J302 pad 8: /Chain/CH2_SDA -> GND
- J302 pad 9: GND -> /Chain/CH2_SCL
- R30 pad 1: /Unit/EXP_RSTN -> /EXP_RSTN
- U5 pad 28: /Unit/EXP_RSTN -> /EXP_RSTN
- U56 pad 3: GND -> /Unit/PRESS_RTN
- U57 pad 3: GND -> /Unit/PRESS_RTN
- U6 pad 3: GND -> /Unit/PRESS_RTN
- U7 pad 3: GND -> /Unit/PRESS_RTN
Routing:
- net +3V3: track 0.00 -> 392.8 mm, vias 0 -> 35
- net /SEG_SCL: track 0.00 -> 283.6 mm, vias 0 -> 18
- net /SEG_SDA: track 0.00 -> 220.9 mm, vias 0 -> 18
- net GND: track 0.00 -> 189.8 mm, vias 0 -> 58
- net /EXP_RSTN: track 0.00 -> 187.6 mm, vias 0 -> 1
- net /PRESS_EN: track 0.00 -> 141.5 mm, vias 0 -> 4
- net /Unit/A_OVK: track 0.00 -> 118.1 mm, vias 0 -> 9
- net /Chain/CH2_SCL: track 0.00 -> 102.3 mm
- net /Chain/CH3_SCL: track 0.00 -> 95.7 mm, vias 0 -> 1
- net /Chain/CH3_SDA: track 0.00 -> 94.1 mm
- net /Chain/CH2_SDA: track 0.00 -> 93.0 mm, vias 0 -> 2
- net VBUS: track 0.00 -> 91.6 mm, vias 0 -> 60
- net /Unit/A_PGD: track 0.00 -> 82.7 mm, vias 0 -> 3
- net /Chain/CH1_SCL: track 0.00 -> 81.8 mm
- net /Chain/CH1_SDA: track 0.00 -> 80.4 mm
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- added copper zone on F.Cu, net /Input/USENSE
- added copper zone on B.Cu, net /Unit/A_NODE
- added copper zone on F.Cu, net /Unit/A_NODE
- added copper zone on B.Cu, net /Unit/A_OUT
- added copper zone on F.Cu, net /Unit/A_OUT
- added copper zone on F.Cu, net /Unit/A_SENSE
- added copper zone on B.Cu, net /Unit/B_NODE
- added copper zone on F.Cu, net /Unit/B_NODE
- added copper zone on B.Cu, net /Unit/B_OUT
- added copper zone on F.Cu, net /Unit/B_OUT
- added copper zone on F.Cu, net /Unit/B_SENSE
- added copper zone on B.Cu, net GND
- added copper zone on F.Cu, net GND
- added copper zone on In1.Cu, net GND
- added copper zone on F.Cu, net VBUS
- added copper zone on In2.Cu, net VBUS
- added copper zone on F.Cu, net VIN
Other:
- board size 76 x 72 mm -> 78.5 x 72 mm

Commit message: pp-48-unit: routing finishes (DRC 0 unconnected, parity clean): bottom-row expander escapes EV13 / EV16 for B_PWRD / B_RUNOFF, placement tweaks; tools/mazefix.py closes the last opens with a grid maze on F / B (IN1=1: hops on In1, here SCL 16 mm and U_OFF 11 mm); tools/mergetracks.py redraws the routers' 45-degree staircases with fewer segments (DRC-checked against its input, 2608 -> 1960 on F / B); route_unit.sh runs both and fills the zones; layer names set
Parts:
- added EV12: , , F.Cu at (136.6, 141.4)
- added EV13: , , F.Cu at (137.1, 142.0)
- added EV16: , , F.Cu at (138.6, 141.0)
- added EV22: , , F.Cu at (141.4, 136.2)
- added EV23: , , F.Cu at (140.6, 135.5)
- added EV24: , , F.Cu at (140.0, 134.9)
- added EV29: , , F.Cu at (136.4, 133.4)
- added EV30: , , F.Cu at (135.6, 133.2)
- added UV1: , , F.Cu at (148.8, 130.8)
- added XV1A1: , , F.Cu at (118.1, 132.9)
- added XV1A2: , , F.Cu at (118.1, 134.1)
- added XV1A3: , , F.Cu at (102.9, 126.2)
- added XV1B1: , , F.Cu at (143.1, 132.9)
- added XV1B2: , , F.Cu at (143.1, 134.1)
- added XV1B3: , , F.Cu at (127.9, 126.2)
- moved C216 12.2 mm to (151.6, 153.0)
- moved C203 12.2 mm to (156.0, 141.0)
- moved U207 6.00 mm to (154.0, 144.0)
- moved U208 6.00 mm to (154.0, 150.0)
- moved R237 5.20 mm to (156.4, 138.5)
- moved R71 1.80 mm to (136.4, 143.4)
- moved R72 1.80 mm to (137.8, 143.4)
- moved R238 1.60 mm to (154.6, 138.5)
Routing:
- net +3V3: track 392.8 -> 513.2 mm, vias 35 -> 43
- net GND: track 189.8 -> 302.2 mm, vias 58 -> 62
- net /U_PGD: track 17.9 -> 71.6 mm, vias 3 -> 4
- net /SEG_SCL: track 283.6 -> 232.0 mm
- net /U_OFF: track 4.84 -> 38.5 mm, vias 0 -> 7
- net /Unit/B_PGD: track 59.7 -> 92.1 mm
- net /Unit/A_PG: track 57.3 -> 89.6 mm, vias 2 -> 5
- net /Unit/B_LED: track 37.3 -> 6.77 mm
- net /Unit/B_ARM: track 51.6 -> 21.3 mm, vias 3 -> 1
- net /Unit/A_RSTD: track 37.1 -> 58.0 mm, vias 0 -> 1
- net /Input/UVLO: track 45.9 -> 25.6 mm, vias 4 -> 2
- net /PRESS_EN: track 141.5 -> 124.0 mm, vias 4 -> 3
- net /Unit/A_ID_F: track 33.5 -> 17.0 mm
- net /EXP_RSTN: track 187.6 -> 199.2 mm, vias 1 -> 4
- net /Unit/B_CLRN: track 19.8 -> 30.5 mm
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
Commit message: 3D models: module aux header J2 on pm-19v-250w (hanxia HX PZ1.27-2x3P TP, C41376035; on B, offset sign follows the flip); unit U5 (stock VQFN-32 footprint points at a STEP KiCad does not ship: pp48 copy with the stock QFN-32 5x5 EP3.3 body), J201 XT60 (C98732), photoMOS U6 / U7 / U56 / U57 TLP176AM (C5370540) and opto U8 / U58 TLP291 (C55144, turned to its pin-1 dot) as pp48 footprint copies (stock models missing), FPIDs moved in uinput.py / unit.py and the board; carrier F1 nano2 fuse (C44479) as a carrier footprint copy; placement = pad fit of the LCSC footprint + the STEP-to-WRL origin shift (EasyEDA STEPs are not on the footprint origin, checked against the XT30 of 020591f), which also corrects today's aux socket (+0.3 mm z) and Degson terminal (-0.1 y, +0.2 z); renders checked; ERC 0 and DRC counts unchanged on unit, carrier, module
Parts:
- J201: footprint Connector_AMASS:AMASS_XT60PW-M_1x02_P7.20mm_Horizontal -> pp48:AMASS_XT60PW-M_1x02_P7.20mm_Horizontal
- U5: footprint Package_DFN_QFN:VQFN-32-1EP_5x5mm_P0.5mm_EP3.15x3.15mm -> pp48:VQFN-32-1EP_5x5mm_P0.5mm_EP3.15x3.15mm
- U56, U57, U6, U7: footprint Package_SO:SOIC-4_4.55x3.7mm_P2.54mm -> pp48:SOIC-4_4.55x3.7mm_P2.54mm
- U58, U8: footprint Package_SO:SOIC-4_4.55x2.6mm_P1.27mm -> pp48:SOIC-4_4.55x2.6mm_P1.27mm
Changed lines of the file:
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@@
 		)
 	)
-	(footprint "Connector_AMASS:AMASS_XT60PW-M_1x02_P7.20mm_Horizontal"
+	(footprint "pp48:AMASS_XT60PW-M_1x02_P7.20mm_Horizontal"
 		(layer "F.Cu")
 		(at 154.9 116.494999)
@@
 		)
 		(embedded_fonts no)
-		(model "${KICAD10_3DMODEL_DIR}/Connector_AMASS.3dshapes/AMASS_XT60PW-M_1x02_P7.20mm_Horizontal.step"
+		(model "${KIPRJMOD}/../pp-48/pp48.3dshapes/AMASS_XT60PW-M.step"
 			(offset
-				(xyz 0 0 0)
+				(xyz 3.6 7.1 0)
 			)
 			(scale
@@
 			)
 			(rotate
-				(xyz 0 0 0)
+				(xyz 0 0 270)
 			)
 		)
@@
 		(embedded_fonts no)
 		(model "${KIPRJMOD}/../pp-48/pp48.3dshapes/TerminalBlock_Degson_DG128-5.0-02P.step"
-			(offset (xyz 2.5 0 0))
-			(scale (xyz 1 1 1))
-			(rotate (xyz 0 0 0))
+			(offset
+				(xyz 2.5 -0.1 0.2)
+			)
+			(scale
+				(xyz 1 1 1)
+			)
+			(rotate
+				(xyz 0 0 0)
+			)
 		)
 	)
@@
 		(model "${KIPRJMOD}/../pp-48/pp48.3dshapes/PM_Aux_Socket_2x03_P1.27.step"
 			(offset
-				(xyz 0 0 0)
+				(xyz 0 0 0.3)
 			)
 			(scale
@@
 		(model "${KIPRJMOD}/../pp-48/pp48.3dshapes/PM_Aux_Socket_2x03_P1.27.step"
 			(offset
-				(xyz 0 0 0)
+				(xyz 0 0 0.3)
 			)
 			(scale
@@
 		)
 	)
-	(footprint "Package_DFN_QFN:VQFN-32-1EP_5x5mm_P0.5mm_EP3.15x3.15mm"
+	(footprint "pp48:VQFN-32-1EP_5x5mm_P0.5mm_EP3.15x3.15mm"
 		(layer "F.Cu")
 		(at 136.8 137.6)
@@
 		)
 		(embedded_fonts no)
-		(model "${KICAD10_3DMODEL_DIR}/Package_DFN_QFN.3dshapes/VQFN-32-1EP_5x5mm_P0.5mm_EP3.15x3.15mm.step"
+		(model "${KICAD10_3DMODEL_DIR}/Package_DFN_QFN.3dshapes/QFN-32-1EP_5x5mm_P0.5mm_EP3.3x3.3mm.step"
 			(offset
 				(xyz 0 0 0)
@@
 		(embedded_fonts no)
 		(model "${KIPRJMOD}/../pp-48/pp48.3dshapes/TerminalBlock_Degson_DG128-5.0-02P.step"
-			(offset (xyz 2.5 0 0))
-			(scale (xyz 1 1 1))
-			(rotate (xyz 0 0 0))
+			(offset
+				(xyz 2.5 -0.1 0.2)
+			)
+			(scale
+				(xyz 1 1 1)
+			)
+			(rotate
+				(xyz 0 0 0)
+			)
 		)
 	)
@@
 		)
 	)
-	(footprint "Package_SO:SOIC-4_4.55x3.7mm_P2.54mm"
+	(footprint "pp48:SOIC-4_4.55x3.7mm_P2.54mm"
 		(layer "B.Cu")
 		(at 106 150.8)
@@
 		)
 		(embedded_fonts no)
-		(model "${KICAD10_3DMODEL_DIR}/Package_SO.3dshapes/SOIC-4_4.55x3.7mm_P2.54mm.step"
+		(model "${KIPRJMOD}/../pp-48/pp48.3dshapes/TLP176AM_SO4.step"
 			(offset
-				(xyz 0 0 0)
+				(xyz 0 0 0.07)
 			)
 			(scale
@@
 		)
 	)
-	(footprint "Package_SO:SOIC-4_4.55x3.7mm_P2.54mm"
+	(footprint "pp48:SOIC-4_4.55x3.7mm_P2.54mm"
 		(layer "B.Cu")
 		(at 131 146.2)
@@
 		)
 		(embedded_fonts no)
-		(model "${KICAD10_3DMODEL_DIR}/Package_SO.3dshapes/SOIC-4_4.55x3.7mm_P2.54mm.step"
+		(model "${KIPRJMOD}/../pp-48/pp48.3dshapes/TLP176AM_SO4.step"
 			(offset
-				(xyz 0 0 0)
+				(xyz 0 0 0.07)
 			)
 			(scale
@@
 		)
 	)
-	(footprint "Package_SO:SOIC-4_4.55x2.6mm_P1.27mm"
+	(footprint "pp48:SOIC-4_4.55x2.6mm_P1.27mm"
 		(layer "B.Cu")
 		(at 131 141.6)
@@
 		)
 		(embedded_fonts no)
-		(model "${KICAD10_3DMODEL_DIR}/Package_SO.3dshapes/SOIC-4_4.55x2.6mm_P1.27mm.step"
+		(model "${KIPRJMOD}/../pp-48/pp48.3dshapes/TLP291_SO4.step"
 			(offset
-				(xyz 0 0 0)
+				(xyz 0 0 0.02)
 			)
 			(scale
@@
 		)
 	)
-	(footprint "Package_SO:SOIC-4_4.55x2.6mm_P1.27mm"
+	(footprint "pp48:SOIC-4_4.55x2.6mm_P1.27mm"
 		(layer "B.Cu")
 		(at 106 141.6)
@@
 		)
 		(embedded_fonts no)
-		(model "${KICAD10_3DMODEL_DIR}/Package_SO.3dshapes/SOIC-4_4.55x2.6mm_P1.27mm.step"
+		(model "${KIPRJMOD}/../pp-48/pp48.3dshapes/TLP291_SO4.step"
 			(offset
-				(xyz 0 0 0)
+				(xyz 0 0 0.02)
 			)
 			(scale
@@
 		)
 	)
-	(footprint "Package_SO:SOIC-4_4.55x3.7mm_P2.54mm"
+	(footprint "pp48:SOIC-4_4.55x3.7mm_P2.54mm"
 		(layer "B.Cu")
 		(at 106 146.2)
@@
 		)
 		(embedded_fonts no)
-		(model "${KICAD10_3DMODEL_DIR}/Package_SO.3dshapes/SOIC-4_4.55x3.7mm_P2.54mm.step"
+		(model "${KIPRJMOD}/../pp-48/pp48.3dshapes/TLP176AM_SO4.step"
 			(offset
-				(xyz 0 0 0)
+				(xyz 0 0 0.07)
 			)
 			(scale
@@
 		)
 	)
-	(footprint "Package_SO:SOIC-4_4.55x3.7mm_P2.54mm"
+	(footprint "pp48:SOIC-4_4.55x3.7mm_P2.54mm"
 		(layer "B.Cu")
 		(at 131 150.8)
@@
 		)
 		(embedded_fonts no)
-		(model "${KICAD10_3DMODEL_DIR}/Package_SO.3dshapes/SOIC-4_4.55x3.7mm_P2.54mm.step"
+		(model "${KIPRJMOD}/../pp-48/pp48.3dshapes/TLP176AM_SO4.step"
 			(offset
-				(xyz 0 0 0)
+				(xyz 0 0 0.07)
 			)
 			(scale
