File: power/pm-19v-250w/pm-19v-250w.kicad_pcb (KiCad board)
At the start: 4 copper layers, 58.4 x 22.9 mm, 57 parts, among them J1 Screw pads S1-S4, J2 Aux header 2x3 1.27, Q1 BSC070N10NS5, Q2 BSC070N10NS5, Q3 BSC070N10NS5, Q4 BSC070N10NS5, U1 LTC7810, U2 MCP65R46-1.21, U3 MCP65R46-1.21

Commit message: stock replacements: unit INA238 (0 at JLC) -> INA237AIDGSR C2864837 on U2 / U52 / U208 (pin- and register-compatible for the plane-logic driver: SHUNT_CAL, LSBs, DIETEMP, MANUFACTURER_ID; gain error 0.3 %); module U2 / U3 MCP65R46-1.21 (0) -> MCP65R46T-2402E/CHY C623510 (2.4 V ref, same hysteresis, open drain, pinout) with R12 84.5k / R14 61.9k (OV_KILL 22.68 V, PGOOD 17.26 V, were 22.75 / 17.30), C13 -> C2980802 (100 V, same family); LM5069-1 left open for the user; boards synced from the netlists; ERC unchanged, DRC unchanged, parity clean; handoff
Parts:
- R12: value 178k -> 84.5k
- R14: value 133k -> 61.9k
- U2, U3: value MCP65R46-1.21 -> MCP65R46-2.4
Changed lines of the file:
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@@
 			)
 		)
-		(property "Value" "MCP65R46-1.21"
+		(property "Value" "MCP65R46-2.4"
 			(at 0 2.4 0)
 			(layer "F.Fab")
@@
 			)
 		)
-		(property "LCSC" "C116625"
+		(property "LCSC" "C623510"
 			(at 0 0 0)
 			(layer "F.Fab")
@@
 			)
 		)
-		(property "LCSC" "C77025"
+		(property "LCSC" "C2980802"
 			(at 0 0 180)
 			(layer "F.Fab")
@@
 			)
 		)
-		(property "Value" "MCP65R46-1.21"
+		(property "Value" "MCP65R46-2.4"
 			(at 0 2.4 180)
 			(layer "F.Fab")
@@
 			)
 		)
-		(property "LCSC" "C116625"
+		(property "LCSC" "C623510"
 			(at 0 0 180)
 			(layer "F.Fab")
@@
 			)
 		)
-		(property "Value" "133k"
+		(property "Value" "61.9k"
 			(at 0 -1.17 270)
 			(layer "B.Fab")
@@
 			)
 		)
-		(property "LCSC" "C25753"
+		(property "LCSC" "C2933106"
 			(at 0 0 270)
 			(layer "B.Fab")
@@
 			)
 		)
-		(property "Value" "178k"
+		(property "Value" "84.5k"
 			(at 0 -1.17 90)
 			(layer "B.Fab")
@@
 			)
 		)
-		(property "LCSC" "C26995"
+		(property "LCSC" "C185390"
 			(at 0 0 90)
 			(layer "B.Fab")
