File: power/pm-19v-250w/pm-19v-250w.kicad_sch (KiCad schematic)
At the start: 57 parts, among them J1 Screw pads S1-S4, J2 Aux pads 2x3, Q1 BSC070N10NS5, Q2 BSC070N10NS5, Q3 BSC070N10NS5, Q4 BSC070N10NS5, U1 LTC7810, U2 MCP65R46-1.21, U3 MCP65R46-1.21

Commit message: pm-19v-250w: sense R9/R10 8 -> 7 mOhm (YLRY12-2-7F C20608751; limit ~16-21 A total), R8 15k -> 13k (same crossover with the lower sense resistance); LTC7810 typ/max sense threshold still to confirm
Parts:
- R10, R9: value 8m 2512 -> 7m 2512; LCSC C2904240 -> C20608751
- R8: value 15k -> 13k; LCSC C22809 -> C22797
Changed lines of the file:
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@@
 	(symbol (lib_id "Device:R") (at 295.91 86.36 90) (unit 1) (body_style 1) (exclude_from_sim no) (in_bom yes) (on_board yes) (in_pos_files yes) (dnp no)
 		(property "Reference" "R10" (at 295.91 82.55 90) (show_name no) (do_not_autoplace no) (effects (font (size 1.27 1.27))))
-		(property "Value" "8m 2512" (at 295.91 90.17 90) (show_name no) (do_not_autoplace no) (effects (font (size 1.27 1.27))))
+		(property "Value" "7m 2512" (at 295.91 90.17 90) (show_name no) (do_not_autoplace no) (effects (font (size 1.27 1.27))))
 		(property "Footprint" "Resistor_SMD:R_2512_6332Metric" (at 295.91 86.36 0) (hide yes) (show_name no) (do_not_autoplace no) (effects (font (size 1.27 1.27))))
 		(property "Datasheet" "" (at 295.91 86.36 0) (hide yes) (show_name no) (do_not_autoplace no) (effects (font (size 1.27 1.27))))
 		(property "Description" "" (at 295.91 86.36 0) (hide yes) (show_name no) (do_not_autoplace no) (effects (font (size 1.27 1.27))))
-		(property "LCSC" "C2904240" (at 295.91 86.36 0) (hide yes) (show_name no) (do_not_autoplace no) (effects (font (size 1.27 1.27))))
+		(property "LCSC" "C20608751" (at 295.91 86.36 0) (hide yes) (show_name no) (do_not_autoplace no) (effects (font (size 1.27 1.27))))
 		(pin "1")
 		(pin "2")
@@
 	(symbol (lib_id "Device:R") (at 172.72 177.8 0) (unit 1) (body_style 1) (exclude_from_sim no) (in_bom yes) (on_board yes) (in_pos_files yes) (dnp no)
 		(property "Reference" "R8" (at 171.45 176.53 0) (show_name no) (do_not_autoplace no) (effects (font (size 1.27 1.27)) (justify right)))
-		(property "Value" "15k" (at 171.45 179.07 0) (show_name no) (do_not_autoplace no) (effects (font (size 1.27 1.27)) (justify right)))
+		(property "Value" "13k" (at 171.45 179.07 0) (show_name no) (do_not_autoplace no) (effects (font (size 1.27 1.27)) (justify right)))
 		(property "Footprint" "Resistor_SMD:R_0603_1608Metric" (at 172.72 177.8 0) (hide yes) (show_name no) (do_not_autoplace no) (effects (font (size 1.27 1.27))))
 		(property "Datasheet" "" (at 172.72 177.8 0) (hide yes) (show_name no) (do_not_autoplace no) (effects (font (size 1.27 1.27))))
 		(property "Description" "" (at 172.72 177.8 0) (hide yes) (show_name no) (do_not_autoplace no) (effects (font (size 1.27 1.27))))
-		(property "LCSC" "C22809" (at 172.72 177.8 0) (hide yes) (show_name no) (do_not_autoplace no) (effects (font (size 1.27 1.27))))
+		(property "LCSC" "C22797" (at 172.72 177.8 0) (hide yes) (show_name no) (do_not_autoplace no) (effects (font (size 1.27 1.27))))
 		(pin "1")
 		(pin "2")
@@
 	(symbol (lib_id "Device:R") (at 125.73 86.36 270) (unit 1) (body_style 1) (exclude_from_sim no) (in_bom yes) (on_board yes) (in_pos_files yes) (dnp no)
 		(property "Reference" "R9" (at 125.73 82.55 90) (show_name no) (do_not_autoplace no) (effects (font (size 1.27 1.27))))
-		(property "Value" "8m 2512" (at 125.73 90.17 90) (show_name no) (do_not_autoplace no) (effects (font (size 1.27 1.27))))
+		(property "Value" "7m 2512" (at 125.73 90.17 90) (show_name no) (do_not_autoplace no) (effects (font (size 1.27 1.27))))
 		(property "Footprint" "Resistor_SMD:R_2512_6332Metric" (at 125.73 86.36 0) (hide yes) (show_name no) (do_not_autoplace no) (effects (font (size 1.27 1.27))))
 		(property "Datasheet" "" (at 125.73 86.36 0) (hide yes) (show_name no) (do_not_autoplace no) (effects (font (size 1.27 1.27))))
 		(property "Description" "" (at 125.73 86.36 0) (hide yes) (show_name no) (do_not_autoplace no) (effects (font (size 1.27 1.27))))
-		(property "LCSC" "C2904240" (at 125.73 86.36 0) (hide yes) (show_name no) (do_not_autoplace no) (effects (font (size 1.27 1.27))))
+		(property "LCSC" "C20608751" (at 125.73 86.36 0) (hide yes) (show_name no) (do_not_autoplace no) (effects (font (size 1.27 1.27))))
 		(pin "1")
 		(pin "2")

Commit message: pm-19v-250w: L1/L2 Coilcraft XAL1510-223 (18.7 A Isat, 16 mOhm, consigned), C24/C25 KEMET T523H 100u 35V polymer 7360-20 (C2158991, 2.0 mm high, goes on B)
Parts:
- C24, C25: value 100u -> 100u 35V polymer 7360-20; footprint Capacitor_Tantalum_SMD:CP_EIA-7343-31_Kemet-D -> Capacitor_Tantalum_SMD:CP_EIA-7360-38_Kemet-E; LCSC (none) -> C2158991
- L1, L2: value 22u Isat>=12A -> 22u XAL1510-223; footprint Inductor_SMD:L_Coilcraft_XAL1010-XXX -> Inductor_SMD:L_Coilcraft_XAL1510-223
Changed lines of the file:
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@@
 	(symbol (lib_id "Device:C_Polarized") (at 210.82 261.62 0) (unit 1) (body_style 1) (exclude_from_sim no) (in_bom yes) (on_board yes) (in_pos_files yes) (dnp no)
 		(property "Reference" "C24" (at 212.09 260.35 0) (show_name no) (do_not_autoplace no) (effects (font (size 1.27 1.27)) (justify left)))
-		(property "Value" "100u" (at 212.09 262.89 0) (show_name no) (do_not_autoplace no) (effects (font (size 1.27 1.27)) (justify left)))
-		(property "Footprint" "Capacitor_Tantalum_SMD:CP_EIA-7343-31_Kemet-D" (at 210.82 261.62 0) (hide yes) (show_name no) (do_not_autoplace no) (effects (font (size 1.27 1.27))))
+		(property "Value" "100u 35V polymer 7360-20" (at 212.09 262.89 0) (show_name no) (do_not_autoplace no) (effects (font (size 1.27 1.27)) (justify left)))
+		(property "Footprint" "Capacitor_Tantalum_SMD:CP_EIA-7360-38_Kemet-E" (at 210.82 261.62 0) (hide yes) (show_name no) (do_not_autoplace no) (effects (font (size 1.27 1.27))))
+		(property "LCSC" "C2158991" (at 210.82 261.62 0) (hide yes) (show_name no) (do_not_autoplace no) (effects (font (size 1.27 1.27))))
 		(property "Datasheet" "" (at 210.82 261.62 0) (hide yes) (show_name no) (do_not_autoplace no) (effects (font (size 1.27 1.27))))
 		(property "Description" "" (at 210.82 261.62 0) (hide yes) (show_name no) (do_not_autoplace no) (effects (font (size 1.27 1.27))))
@@
 	(symbol (lib_id "Device:C_Polarized") (at 223.52 261.62 0) (unit 1) (body_style 1) (exclude_from_sim no) (in_bom yes) (on_board yes) (in_pos_files yes) (dnp no)
 		(property "Reference" "C25" (at 224.79000000000002 260.35 0) (show_name no) (do_not_autoplace no) (effects (font (size 1.27 1.27)) (justify left)))
-		(property "Value" "100u" (at 224.79000000000002 262.89 0) (show_name no) (do_not_autoplace no) (effects (font (size 1.27 1.27)) (justify left)))
-		(property "Footprint" "Capacitor_Tantalum_SMD:CP_EIA-7343-31_Kemet-D" (at 223.52 261.62 0) (hide yes) (show_name no) (do_not_autoplace no) (effects (font (size 1.27 1.27))))
+		(property "Value" "100u 35V polymer 7360-20" (at 224.79000000000002 262.89 0) (show_name no) (do_not_autoplace no) (effects (font (size 1.27 1.27)) (justify left)))
+		(property "Footprint" "Capacitor_Tantalum_SMD:CP_EIA-7360-38_Kemet-E" (at 223.52 261.62 0) (hide yes) (show_name no) (do_not_autoplace no) (effects (font (size 1.27 1.27))))
+		(property "LCSC" "C2158991" (at 223.52 261.62 0) (hide yes) (show_name no) (do_not_autoplace no) (effects (font (size 1.27 1.27))))
 		(property "Datasheet" "" (at 223.52 261.62 0) (hide yes) (show_name no) (do_not_autoplace no) (effects (font (size 1.27 1.27))))
 		(property "Description" "" (at 223.52 261.62 0) (hide yes) (show_name no) (do_not_autoplace no) (effects (font (size 1.27 1.27))))
@@
 	(symbol (lib_id "Device:L") (at 143.51 86.36 270) (unit 1) (body_style 1) (exclude_from_sim no) (in_bom yes) (on_board yes) (in_pos_files yes) (dnp no)
 		(property "Reference" "L1" (at 143.51 82.55 90) (show_name no) (do_not_autoplace no) (effects (font (size 1.27 1.27))))
-		(property "Value" "22u Isat>=12A" (at 143.51 90.17 90) (show_name no) (do_not_autoplace no) (effects (font (size 1.27 1.27))))
-		(property "Footprint" "Inductor_SMD:L_Coilcraft_XAL1010-XXX" (at 143.51 86.36 0) (hide yes) (show_name no) (do_not_autoplace no) (effects (font (size 1.27 1.27))))
+		(property "Value" "22u XAL1510-223" (at 143.51 90.17 90) (show_name no) (do_not_autoplace no) (effects (font (size 1.27 1.27))))
+		(property "Footprint" "Inductor_SMD:L_Coilcraft_XAL1510-223" (at 143.51 86.36 0) (hide yes) (show_name no) (do_not_autoplace no) (effects (font (size 1.27 1.27))))
 		(property "Datasheet" "" (at 143.51 86.36 0) (hide yes) (show_name no) (do_not_autoplace no) (effects (font (size 1.27 1.27))))
 		(property "Description" "" (at 143.51 86.36 0) (hide yes) (show_name no) (do_not_autoplace no) (effects (font (size 1.27 1.27))))
@@
 	(symbol (lib_id "Device:L") (at 278.13 86.36 90) (unit 1) (body_style 1) (exclude_from_sim no) (in_bom yes) (on_board yes) (in_pos_files yes) (dnp no)
 		(property "Reference" "L2" (at 278.13 82.55 90) (show_name no) (do_not_autoplace no) (effects (font (size 1.27 1.27))))
-		(property "Value" "22u Isat>=12A" (at 278.13 90.17 90) (show_name no) (do_not_autoplace no) (effects (font (size 1.27 1.27))))
-		(property "Footprint" "Inductor_SMD:L_Coilcraft_XAL1010-XXX" (at 278.13 86.36 0) (hide yes) (show_name no) (do_not_autoplace no) (effects (font (size 1.27 1.27))))
+		(property "Value" "22u XAL1510-223" (at 278.13 90.17 90) (show_name no) (do_not_autoplace no) (effects (font (size 1.27 1.27))))
+		(property "Footprint" "Inductor_SMD:L_Coilcraft_XAL1510-223" (at 278.13 86.36 0) (hide yes) (show_name no) (do_not_autoplace no) (effects (font (size 1.27 1.27))))
 		(property "Datasheet" "" (at 278.13 86.36 0) (hide yes) (show_name no) (do_not_autoplace no) (effects (font (size 1.27 1.27))))
 		(property "Description" "" (at 278.13 86.36 0) (hide yes) (show_name no) (do_not_autoplace no) (effects (font (size 1.27 1.27))))

Commit message: pm-19v-250w: U1 neighbourhood reorganised for hand-routing the gate drive: U1 small-signal passives to 0402 (C10 C12-C19 R5-R8, JLC parts), VFB/ITH1 network in a pocket above pins 45-47, corridor above the phase 1 drive pins and a TG1 lane kept free, bootstraps C18/C19 beside their switch nodes; VIN band under C1-C4 narrowed to 108.2; packer step 0.05, gap 0.2; unrouted
Parts:
- C10, C15, C18, C19: footprint Capacitor_SMD:C_0603_1608Metric -> Capacitor_SMD:C_0402_1005Metric; LCSC C14663 -> C307331
- C12: footprint Capacitor_SMD:C_0603_1608Metric -> Capacitor_SMD:C_0402_1005Metric; LCSC C94904 -> C1567
- C13: footprint Capacitor_SMD:C_0603_1608Metric -> Capacitor_SMD:C_0402_1005Metric; LCSC C374074 -> C77025
- C14: footprint Capacitor_SMD:C_0603_1608Metric -> Capacitor_SMD:C_0402_1005Metric; LCSC C1635 -> C1546
- C16, C17: footprint Capacitor_SMD:C_0603_1608Metric -> Capacitor_SMD:C_0402_1005Metric; LCSC C100040 -> C1523
- R5: footprint Resistor_SMD:R_0603_1608Metric -> Resistor_SMD:R_0402_1005Metric; LCSC C22892 -> C25859
- R6: footprint Resistor_SMD:R_0603_1608Metric -> Resistor_SMD:R_0402_1005Metric; LCSC C22827 -> C25760
- R7: footprint Resistor_SMD:R_0603_1608Metric -> Resistor_SMD:R_0402_1005Metric; LCSC C25804 -> C25744
- R8: footprint Resistor_SMD:R_0603_1608Metric -> Resistor_SMD:R_0402_1005Metric; LCSC C22797 -> C25754

Commit message: pm-19v-250w: supervision block grouped at the input end (dividers and VAUX caps to 0402), RUN/OVLO divider on B at the input end, R16 by J2; hand drive routes kept (group 'hand', krt keep_groups); KRT routed the rest: 14 opens left (VOUT, OVLO, ITH1, INTVCC, DRVCC/NDRV, U2-, U3+, GND taps), 0 clearance errors
Parts:
- C26: footprint Capacitor_SMD:C_0603_1608Metric -> Capacitor_SMD:C_0402_1005Metric; LCSC C380328 -> C52923
- C27, C28: footprint Capacitor_SMD:C_0603_1608Metric -> Capacitor_SMD:C_0402_1005Metric; LCSC C14663 -> C307331
- R12: footprint Resistor_SMD:R_0603_1608Metric -> Resistor_SMD:R_0402_1005Metric; LCSC C22823 -> C26995
- R13, R15: footprint Resistor_SMD:R_0603_1608Metric -> Resistor_SMD:R_0402_1005Metric; LCSC C25804 -> C25744
- R14: footprint Resistor_SMD:R_0603_1608Metric -> Resistor_SMD:R_0402_1005Metric; LCSC C22870 -> C25753
Changed lines of the file:
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@@
 		(property "Reference" "C26" (at 62.230000000000004 205.74 0) (show_name no) (do_not_autoplace no) (effects (font (size 1.27 1.27)) (justify left)))
 		(property "Value" "1u" (at 62.230000000000004 208.28 0) (show_name no) (do_not_autoplace no) (effects (font (size 1.27 1.27)) (justify left)))
-		(property "Footprint" "Capacitor_SMD:C_0603_1608Metric" (at 60.96 207.01 0) (hide yes) (show_name no) (do_not_autoplace no) (effects (font (size 1.27 1.27))))
+		(property "Footprint" "Capacitor_SMD:C_0402_1005Metric" (at 60.96 207.01 0) (hide yes) (show_name no) (do_not_autoplace no) (effects (font (size 1.27 1.27))))
 		(property "Datasheet" "" (at 60.96 207.01 0) (hide yes) (show_name no) (do_not_autoplace no) (effects (font (size 1.27 1.27))))
 		(property "Description" "" (at 60.96 207.01 0) (hide yes) (show_name no) (do_not_autoplace no) (effects (font (size 1.27 1.27))))
-		(property "LCSC" "C380328" (at 60.96 207.01 0) (hide yes) (show_name no) (do_not_autoplace no) (effects (font (size 1.27 1.27))))
+		(property "LCSC" "C52923" (at 60.96 207.01 0) (hide yes) (show_name no) (do_not_autoplace no) (effects (font (size 1.27 1.27))))
 		(pin "1")
 		(pin "2")
@@
 		(property "Reference" "C27" (at 90.17 205.74 0) (show_name no) (do_not_autoplace no) (effects (font (size 1.27 1.27)) (justify left)))
 		(property "Value" "0.1u" (at 90.17 208.28 0) (show_name no) (do_not_autoplace no) (effects (font (size 1.27 1.27)) (justify left)))
-		(property "Footprint" "Capacitor_SMD:C_0603_1608Metric" (at 88.9 207.01 0) (hide yes) (show_name no) (do_not_autoplace no) (effects (font (size 1.27 1.27))))
+		(property "Footprint" "Capacitor_SMD:C_0402_1005Metric" (at 88.9 207.01 0) (hide yes) (show_name no) (do_not_autoplace no) (effects (font (size 1.27 1.27))))
 		(property "Datasheet" "" (at 88.9 207.01 0) (hide yes) (show_name no) (do_not_autoplace no) (effects (font (size 1.27 1.27))))
 		(property "Description" "" (at 88.9 207.01 0) (hide yes) (show_name no) (do_not_autoplace no) (effects (font (size 1.27 1.27))))
-		(property "LCSC" "C14663" (at 88.9 207.01 0) (hide yes) (show_name no) (do_not_autoplace no) (effects (font (size 1.27 1.27))))
+		(property "LCSC" "C307331" (at 88.9 207.01 0) (hide yes) (show_name no) (do_not_autoplace no) (effects (font (size 1.27 1.27))))
 		(pin "1")
 		(pin "2")
@@
 		(property "Reference" "C28" (at 151.13000000000002 205.74 0) (show_name no) (do_not_autoplace no) (effects (font (size 1.27 1.27)) (justify left)))
 		(property "Value" "0.1u" (at 151.13000000000002 208.28 0) (show_name no) (do_not_autoplace no) (effects (font (size 1.27 1.27)) (justify left)))
-		(property "Footprint" "Capacitor_SMD:C_0603_1608Metric" (at 149.86 207.01 0) (hide yes) (show_name no) (do_not_autoplace no) (effects (font (size 1.27 1.27))))
+		(property "Footprint" "Capacitor_SMD:C_0402_1005Metric" (at 149.86 207.01 0) (hide yes) (show_name no) (do_not_autoplace no) (effects (font (size 1.27 1.27))))
 		(property "Datasheet" "" (at 149.86 207.01 0) (hide yes) (show_name no) (do_not_autoplace no) (effects (font (size 1.27 1.27))))
 		(property "Description" "" (at 149.86 207.01 0) (hide yes) (show_name no) (do_not_autoplace no) (effects (font (size 1.27 1.27))))
-		(property "LCSC" "C14663" (at 149.86 207.01 0) (hide yes) (show_name no) (do_not_autoplace no) (effects (font (size 1.27 1.27))))
+		(property "LCSC" "C307331" (at 149.86 207.01 0) (hide yes) (show_name no) (do_not_autoplace no) (effects (font (size 1.27 1.27))))
 		(pin "1")
 		(pin "2")
@@
 		(property "Reference" "R12" (at 69.85000000000001 220.98 0) (show_name no) (do_not_autoplace no) (effects (font (size 1.27 1.27)) (justify right)))
 		(property "Value" "178k" (at 69.85000000000001 223.52 0) (show_name no) (do_not_autoplace no) (effects (font (size 1.27 1.27)) (justify right)))
-		(property "Footprint" "Resistor_SMD:R_0603_1608Metric" (at 71.12 222.25 0) (hide yes) (show_name no) (do_not_autoplace no) (effects (font (size 1.27 1.27))))
+		(property "Footprint" "Resistor_SMD:R_0402_1005Metric" (at 71.12 222.25 0) (hide yes) (show_name no) (do_not_autoplace no) (effects (font (size 1.27 1.27))))
 		(property "Datasheet" "" (at 71.12 222.25 0) (hide yes) (show_name no) (do_not_autoplace no) (effects (font (size 1.27 1.27))))
 		(property "Description" "" (at 71.12 222.25 0) (hide yes) (show_name no) (do_not_autoplace no) (effects (font (size 1.27 1.27))))
-		(property "LCSC" "C22823" (at 71.12 222.25 0) (hide yes) (show_name no) (do_not_autoplace no) (effects (font (size 1.27 1.27))))
+		(property "LCSC" "C26995" (at 71.12 222.25 0) (hide yes) (show_name no) (do_not_autoplace no) (effects (font (size 1.27 1.27))))
 		(pin "1")
 		(pin "2")
@@
 		(property "Reference" "R13" (at 69.85000000000001 237.49 0) (show_name no) (do_not_autoplace no) (effects (font (size 1.27 1.27)) (justify right)))
 		(property "Value" "10k" (at 69.85000000000001 240.03 0) (show_name no) (do_not_autoplace no) (effects (font (size 1.27 1.27)) (justify right)))
-		(property "Footprint" "Resistor_SMD:R_0603_1608Metric" (at 71.12 238.76 0) (hide yes) (show_name no) (do_not_autoplace no) (effects (font (size 1.27 1.27))))
+		(property "Footprint" "Resistor_SMD:R_0402_1005Metric" (at 71.12 238.76 0) (hide yes) (show_name no) (do_not_autoplace no) (effects (font (size 1.27 1.27))))
 		(property "Datasheet" "" (at 71.12 238.76 0) (hide yes) (show_name no) (do_not_autoplace no) (effects (font (size 1.27 1.27))))
 		(property "Description" "" (at 71.12 238.76 0) (hide yes) (show_name no) (do_not_autoplace no) (effects (font (size 1.27 1.27))))
-		(property "LCSC" "C25804" (at 71.12 238.76 0) (hide yes) (show_name no) (do_not_autoplace no) (effects (font (size 1.27 1.27))))
+		(property "LCSC" "C25744" (at 71.12 238.76 0) (hide yes) (show_name no) (do_not_autoplace no) (effects (font (size 1.27 1.27))))
 		(pin "1")
 		(pin "2")
@@
 		(property "Reference" "R14" (at 133.35 220.98 0) (show_name no) (do_not_autoplace no) (effects (font (size 1.27 1.27)) (justify right)))
 		(property "Value" "133k" (at 133.35 223.52 0) (show_name no) (do_not_autoplace no) (effects (font (size 1.27 1.27)) (justify right)))
-		(property "Footprint" "Resistor_SMD:R_0603_1608Metric" (at 134.62 222.25 0) (hide yes) (show_name no) (do_not_autoplace no) (effects (font (size 1.27 1.27))))
+		(property "Footprint" "Resistor_SMD:R_0402_1005Metric" (at 134.62 222.25 0) (hide yes) (show_name no) (do_not_autoplace no) (effects (font (size 1.27 1.27))))
 		(property "Datasheet" "" (at 134.62 222.25 0) (hide yes) (show_name no) (do_not_autoplace no) (effects (font (size 1.27 1.27))))
 		(property "Description" "" (at 134.62 222.25 0) (hide yes) (show_name no) (do_not_autoplace no) (effects (font (size 1.27 1.27))))
-		(property "LCSC" "C22870" (at 134.62 222.25 0) (hide yes) (show_name no) (do_not_autoplace no) (effects (font (size 1.27 1.27))))
+		(property "LCSC" "C25753" (at 134.62 222.25 0) (hide yes) (show_name no) (do_not_autoplace no) (effects (font (size 1.27 1.27))))
 		(pin "1")
 		(pin "2")
@@
 		(property "Reference" "R15" (at 133.35 237.49 0) (show_name no) (do_not_autoplace no) (effects (font (size 1.27 1.27)) (justify right)))
 		(property "Value" "10k" (at 133.35 240.03 0) (show_name no) (do_not_autoplace no) (effects (font (size 1.27 1.27)) (justify right)))
-		(property "Footprint" "Resistor_SMD:R_0603_1608Metric" (at 134.62 238.76 0) (hide yes) (show_name no) (do_not_autoplace no) (effects (font (size 1.27 1.27))))
+		(property "Footprint" "Resistor_SMD:R_0402_1005Metric" (at 134.62 238.76 0) (hide yes) (show_name no) (do_not_autoplace no) (effects (font (size 1.27 1.27))))
 		(property "Datasheet" "" (at 134.62 238.76 0) (hide yes) (show_name no) (do_not_autoplace no) (effects (font (size 1.27 1.27))))
 		(property "Description" "" (at 134.62 238.76 0) (hide yes) (show_name no) (do_not_autoplace no) (effects (font (size 1.27 1.27))))
-		(property "LCSC" "C25804" (at 134.62 238.76 0) (hide yes) (show_name no) (do_not_autoplace no) (effects (font (size 1.27 1.27))))
-		(pin "1")
-		(pin "2")
+		(property "LCSC" "C25744" (at 134.62 238.76 0) (hide yes) (show_name no) (do_not_autoplace no) (effects (font (size 1.27 1.27))))
+		(pin "1")
+		(pin "2")

Commit message: pm-19v-250w: L1/L2 COILANK APS1510M220F (C49261404, JLC stock) on the XAL1510 footprint (terminals match the pads, body inside the courtyard)
Parts:
- L1, L2: value 22u XAL1510-223 -> 22u APS1510M220F; LCSC (none) -> C49261404
Changed lines of the file:
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@@
 	(symbol (lib_id "Device:L") (at 143.51 86.36 270) (unit 1) (body_style 1) (exclude_from_sim no) (in_bom yes) (on_board yes) (in_pos_files yes) (dnp no)
 		(property "Reference" "L1" (at 143.51 82.55 90) (show_name no) (do_not_autoplace no) (effects (font (size 1.27 1.27))))
-		(property "Value" "22u XAL1510-223" (at 143.51 90.17 90) (show_name no) (do_not_autoplace no) (effects (font (size 1.27 1.27))))
+		(property "Value" "22u APS1510M220F" (at 143.51 90.17 90) (show_name no) (do_not_autoplace no) (effects (font (size 1.27 1.27))))
 		(property "Footprint" "Inductor_SMD:L_Coilcraft_XAL1510-223" (at 143.51 86.36 0) (hide yes) (show_name no) (do_not_autoplace no) (effects (font (size 1.27 1.27))))
+		(property "LCSC" "C49261404" (at 143.51 86.36 0) (hide yes) (show_name no) (do_not_autoplace no) (effects (font (size 1.27 1.27))))
 		(property "Datasheet" "" (at 143.51 86.36 0) (hide yes) (show_name no) (do_not_autoplace no) (effects (font (size 1.27 1.27))))
 		(property "Description" "" (at 143.51 86.36 0) (hide yes) (show_name no) (do_not_autoplace no) (effects (font (size 1.27 1.27))))
@@
 	(symbol (lib_id "Device:L") (at 278.13 86.36 90) (unit 1) (body_style 1) (exclude_from_sim no) (in_bom yes) (on_board yes) (in_pos_files yes) (dnp no)
 		(property "Reference" "L2" (at 278.13 82.55 90) (show_name no) (do_not_autoplace no) (effects (font (size 1.27 1.27))))
-		(property "Value" "22u XAL1510-223" (at 278.13 90.17 90) (show_name no) (do_not_autoplace no) (effects (font (size 1.27 1.27))))
+		(property "Value" "22u APS1510M220F" (at 278.13 90.17 90) (show_name no) (do_not_autoplace no) (effects (font (size 1.27 1.27))))
 		(property "Footprint" "Inductor_SMD:L_Coilcraft_XAL1510-223" (at 278.13 86.36 0) (hide yes) (show_name no) (do_not_autoplace no) (effects (font (size 1.27 1.27))))
+		(property "LCSC" "C49261404" (at 278.13 86.36 0) (hide yes) (show_name no) (do_not_autoplace no) (effects (font (size 1.27 1.27))))
 		(property "Datasheet" "" (at 278.13 86.36 0) (hide yes) (show_name no) (do_not_autoplace no) (effects (font (size 1.27 1.27))))
 		(property "Description" "" (at 278.13 86.36 0) (hide yes) (show_name no) (do_not_autoplace no) (effects (font (size 1.27 1.27))))
