File: power/pm-19v-250w/pm-19v-250w.kicad_sch (KiCad schematic)
At the start: 57 parts, among them J1 Screw pads S1-S4, J2 Aux pads 2x3, Q1 BSC070N10NS5, Q2 BSC070N10NS5, Q3 BSC070N10NS5, Q4 BSC070N10NS5, U1 LTC7810, U2 MCP65R46-1.21, U3 MCP65R46-1.21

Commit message: PM aux contacts: 2x3 1.27 mm SMT header (module J2, C41376035) into SMT socket (carrier J3, C41397112) replaces flat pads + pogos; standoffs M2 x 7 (C2916355), gap 7.0 mm. pmmount.py generates the new footprints; module J2 swapped in place, tools/route_aux.py moves PGOOD's via and adds a GND via between the columns (DRC as before, 0 unconnected, parity clean); carrier PG1-PG6 -> J3 and rebuilt by its flow (DRC 0 errors, 0 unconnected, parity clean); spec, ADR 0003 (6, 7), power-board.md and handoff updated; ID open = slot fault rule
Parts:
- J2: value Aux pads 2x3 -> Aux header 2x3 1.27; footprint pm:PM_Aux_Pads_2x03 -> pm:PM_Aux_Header_2x03_P1.27; LCSC (none) -> C41376035; now in the parts list
Changed lines of the file:
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@@
 		(instances (project "" (path "/89669c12-5e74-4100-98d5-4c6ec3ae2f8e" (reference "J1") (unit 1))))
 	)
-	(symbol (lib_id "Connector_Generic:Conn_01x06") (at 304.8 213.36 0) (unit 1) (body_style 1) (exclude_from_sim no) (in_bom no) (on_board yes) (in_pos_files no) (dnp no)
+	(symbol (lib_id "Connector_Generic:Conn_01x06") (at 304.8 213.36 0) (unit 1) (body_style 1) (exclude_from_sim no) (in_bom yes) (on_board yes) (in_pos_files yes) (dnp no)
 		(property "Reference" "J2" (at 304.8 204.47 0) (show_name no) (do_not_autoplace no) (effects (font (size 1.27 1.27))))
-		(property "Value" "Aux pads 2x3" (at 304.8 226.06 0) (show_name no) (do_not_autoplace no) (effects (font (size 1.27 1.27))))
-		(property "Footprint" "pm:PM_Aux_Pads_2x03" (at 304.8 213.36 0) (hide yes) (show_name no) (do_not_autoplace no) (effects (font (size 1.27 1.27))))
+		(property "Value" "Aux header 2x3 1.27" (at 304.8 226.06 0) (show_name no) (do_not_autoplace no) (effects (font (size 1.27 1.27))))
+		(property "Footprint" "pm:PM_Aux_Header_2x03_P1.27" (at 304.8 213.36 0) (hide yes) (show_name no) (do_not_autoplace no) (effects (font (size 1.27 1.27))))
+		(property "LCSC" "C41376035" (at 304.8 213.36 0) (hide yes) (show_name no) (do_not_autoplace no) (effects (font (size 1.27 1.27))))
 		(property "Datasheet" "" (at 304.8 213.36 0) (hide yes) (show_name no) (do_not_autoplace no) (effects (font (size 1.27 1.27))))
 		(property "Description" "" (at 304.8 213.36 0) (hide yes) (show_name no) (do_not_autoplace no) (effects (font (size 1.27 1.27))))

Commit message: stock replacements: unit INA238 (0 at JLC) -> INA237AIDGSR C2864837 on U2 / U52 / U208 (pin- and register-compatible for the plane-logic driver: SHUNT_CAL, LSBs, DIETEMP, MANUFACTURER_ID; gain error 0.3 %); module U2 / U3 MCP65R46-1.21 (0) -> MCP65R46T-2402E/CHY C623510 (2.4 V ref, same hysteresis, open drain, pinout) with R12 84.5k / R14 61.9k (OV_KILL 22.68 V, PGOOD 17.26 V, were 22.75 / 17.30), C13 -> C2980802 (100 V, same family); LM5069-1 left open for the user; boards synced from the netlists; ERC unchanged, DRC unchanged, parity clean; handoff
Parts:
- C13: LCSC C77025 -> C2980802
- R12: value 178k -> 84.5k; LCSC C26995 -> C185390
- R14: value 133k -> 61.9k; LCSC C25753 -> C2933106
- U2, U3: value MCP65R46-1.21 -> MCP65R46-2.4; LCSC C116625 -> C623510
Changed lines of the file:
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@@
 		(property "Datasheet" "" (at 172.72 189.23 0) (hide yes) (show_name no) (do_not_autoplace no) (effects (font (size 1.27 1.27))))
 		(property "Description" "" (at 172.72 189.23 0) (hide yes) (show_name no) (do_not_autoplace no) (effects (font (size 1.27 1.27))))
-		(property "LCSC" "C77025" (at 172.72 189.23 0) (hide yes) (show_name no) (do_not_autoplace no) (effects (font (size 1.27 1.27))))
+		(property "LCSC" "C2980802" (at 172.72 189.23 0) (hide yes) (show_name no) (do_not_autoplace no) (effects (font (size 1.27 1.27))))
 		(pin "1")
 		(pin "2")
@@
 	(symbol (lib_id "Device:R") (at 71.12 222.25 0) (unit 1) (body_style 1) (exclude_from_sim no) (in_bom yes) (on_board yes) (in_pos_files yes) (dnp no)
 		(property "Reference" "R12" (at 69.85000000000001 220.98 0) (show_name no) (do_not_autoplace no) (effects (font (size 1.27 1.27)) (justify right)))
-		(property "Value" "178k" (at 69.85000000000001 223.52 0) (show_name no) (do_not_autoplace no) (effects (font (size 1.27 1.27)) (justify right)))
+		(property "Value" "84.5k" (at 69.85000000000001 223.52 0) (show_name no) (do_not_autoplace no) (effects (font (size 1.27 1.27)) (justify right)))
 		(property "Footprint" "Resistor_SMD:R_0402_1005Metric" (at 71.12 222.25 0) (hide yes) (show_name no) (do_not_autoplace no) (effects (font (size 1.27 1.27))))
 		(property "Datasheet" "" (at 71.12 222.25 0) (hide yes) (show_name no) (do_not_autoplace no) (effects (font (size 1.27 1.27))))
 		(property "Description" "" (at 71.12 222.25 0) (hide yes) (show_name no) (do_not_autoplace no) (effects (font (size 1.27 1.27))))
-		(property "LCSC" "C26995" (at 71.12 222.25 0) (hide yes) (show_name no) (do_not_autoplace no) (effects (font (size 1.27 1.27))))
+		(property "LCSC" "C185390" (at 71.12 222.25 0) (hide yes) (show_name no) (do_not_autoplace no) (effects (font (size 1.27 1.27))))
 		(pin "1")
 		(pin "2")
@@
 	(symbol (lib_id "Device:R") (at 134.62 222.25 0) (unit 1) (body_style 1) (exclude_from_sim no) (in_bom yes) (on_board yes) (in_pos_files yes) (dnp no)
 		(property "Reference" "R14" (at 133.35 220.98 0) (show_name no) (do_not_autoplace no) (effects (font (size 1.27 1.27)) (justify right)))
-		(property "Value" "133k" (at 133.35 223.52 0) (show_name no) (do_not_autoplace no) (effects (font (size 1.27 1.27)) (justify right)))
+		(property "Value" "61.9k" (at 133.35 223.52 0) (show_name no) (do_not_autoplace no) (effects (font (size 1.27 1.27)) (justify right)))
 		(property "Footprint" "Resistor_SMD:R_0402_1005Metric" (at 134.62 222.25 0) (hide yes) (show_name no) (do_not_autoplace no) (effects (font (size 1.27 1.27))))
 		(property "Datasheet" "" (at 134.62 222.25 0) (hide yes) (show_name no) (do_not_autoplace no) (effects (font (size 1.27 1.27))))
 		(property "Description" "" (at 134.62 222.25 0) (hide yes) (show_name no) (do_not_autoplace no) (effects (font (size 1.27 1.27))))
-		(property "LCSC" "C25753" (at 134.62 222.25 0) (hide yes) (show_name no) (do_not_autoplace no) (effects (font (size 1.27 1.27))))
+		(property "LCSC" "C2933106" (at 134.62 222.25 0) (hide yes) (show_name no) (do_not_autoplace no) (effects (font (size 1.27 1.27))))
 		(pin "1")
 		(pin "2")
@@
 	(symbol (lib_id "Comparator:MCP65R46") (at 99.06 228.6 0) (unit 1) (body_style 1) (exclude_from_sim no) (in_bom yes) (on_board yes) (in_pos_files yes) (dnp no)
 		(property "Reference" "U2" (at 101.60000000000001 236.22 0) (show_name no) (do_not_autoplace no) (effects (font (size 1.27 1.27)) (justify left)))
-		(property "Value" "MCP65R46-1.21" (at 101.60000000000001 238.76 0) (show_name no) (do_not_autoplace no) (effects (font (size 1.27 1.27)) (justify left)))
+		(property "Value" "MCP65R46-2.4" (at 101.60000000000001 238.76 0) (show_name no) (do_not_autoplace no) (effects (font (size 1.27 1.27)) (justify left)))
 		(property "Footprint" "Package_TO_SOT_SMD:SOT-23-6" (at 99.06 228.6 0) (hide yes) (show_name no) (do_not_autoplace no) (effects (font (size 1.27 1.27))))
 		(property "Datasheet" "" (at 99.06 228.6 0) (hide yes) (show_name no) (do_not_autoplace no) (effects (font (size 1.27 1.27))))
 		(property "Description" "" (at 99.06 228.6 0) (hide yes) (show_name no) (do_not_autoplace no) (effects (font (size 1.27 1.27))))
-		(property "LCSC" "C116625" (at 99.06 228.6 0) (hide yes) (show_name no) (do_not_autoplace no) (effects (font (size 1.27 1.27))))
+		(property "LCSC" "C623510" (at 99.06 228.6 0) (hide yes) (show_name no) (do_not_autoplace no) (effects (font (size 1.27 1.27))))
 		(pin "1")
 		(pin "2")
@@
 	(symbol (lib_id "Comparator:MCP65R46") (at 160.02 228.6 0) (unit 1) (body_style 1) (exclude_from_sim no) (in_bom yes) (on_board yes) (in_pos_files yes) (dnp no)
 		(property "Reference" "U3" (at 162.56 236.22 0) (show_name no) (do_not_autoplace no) (effects (font (size 1.27 1.27)) (justify left)))
-		(property "Value" "MCP65R46-1.21" (at 162.56 238.76 0) (show_name no) (do_not_autoplace no) (effects (font (size 1.27 1.27)) (justify left)))
+		(property "Value" "MCP65R46-2.4" (at 162.56 238.76 0) (show_name no) (do_not_autoplace no) (effects (font (size 1.27 1.27)) (justify left)))
 		(property "Footprint" "Package_TO_SOT_SMD:SOT-23-6" (at 160.02 228.6 0) (hide yes) (show_name no) (do_not_autoplace no) (effects (font (size 1.27 1.27))))
 		(property "Datasheet" "" (at 160.02 228.6 0) (hide yes) (show_name no) (do_not_autoplace no) (effects (font (size 1.27 1.27))))
 		(property "Description" "" (at 160.02 228.6 0) (hide yes) (show_name no) (do_not_autoplace no) (effects (font (size 1.27 1.27))))
-		(property "LCSC" "C116625" (at 160.02 228.6 0) (hide yes) (show_name no) (do_not_autoplace no) (effects (font (size 1.27 1.27))))
-		(pin "1")
-		(pin "2")
+		(property "LCSC" "C623510" (at 160.02 228.6 0) (hide yes) (show_name no) (do_not_autoplace no) (effects (font (size 1.27 1.27))))
+		(pin "1")
+		(pin "2")
