File: power/pp-48-unit/sheets/unit.kicad_sch (KiCad schematic)
At the start: 120 parts, among them J1 NODE 19V, J2 FRONT PANEL, J3 AUX, J51 NODE 19V, J52 FRONT PANEL, J53 AUX, Q1 BSC070N10NS5, Q2 2N7002, Q3 2N7002, Q4 2N7002, Q5 2N7002, Q51 BSC070N10NS5, Q52 2N7002, Q53 2N7002, Q54 2N7002, Q55 2N7002, Q56 2N7002, Q57 2N7002, Q58 2N7002, Q59 2N7002, Q6 2N7002, Q7 2N7002, Q8 2N7002, Q9 2N7002, U1 LM5069MM-2, U10 74LVC1G74, U2 INA238AIDGSR, U3 74LVC1G74, U4 ADC121C027CIMK, U5 TCA6424ARGJR, U51 LM5069MM-2, U52 INA238AIDGSR, U53 74LVC1G74, U54 ADC121C027CIMK, U56 TLP176AM, U57 TLP176AM, U58 TLP291, U6 TLP176AM, U60 74LVC1G74, U7 TLP176AM, U8 TLP291

Commit message: pp-48 plane boards: press deadline line (docs/press-deadline-line.md decided: option B + A) on a 14-pin chain (S14B-PH-K-S C157938; 13 PRESS_EN, 14 EXP_RSTN, cable n -> 15 - n, pins v 35..61); unit Q10 / R31 switch the photoMOS LED returns (PRESS_RTN), core U301 74LVC1G123 deadline (pp:74LVC1G123 single-unit copy) on PC6 PRESS_TRIG, PC7 EXP_RSTN to the units' /RESET; ERC 0 both; boards rebuilt and placed, unit 78.5 x 72 with the strip power path re-placed top-down; unit routing tools (route_unit.py hand copper + In2 band / +3V3 trunk, unitsplit.py, route_unit.sh flow): DRC 0 errors, ~10 unconnected at expander U5; core placed, not routed; pmmount.py restored from granite_controller; ADR 0005 decision 4; handoff
Parts:
- added Q10: 2N7002, Package_TO_SOT_SMD:SOT-23, symbol Transistor_FET:2N7002
- added R31: 100k, Resistor_SMD:R_0402_1005Metric, symbol Device:R
Connections:
- net GND: now also Q10.2 (S), R31.2; no longer U56.3, U57.3, U6.3, U7.3
- new net PRESS_EN: Q10.1 (G), R31.1
- new net PRESS_RTN: Q10.3 (D), U56.3, U57.3, U6.3, U7.3

Commit message: 3D models: module aux header J2 on pm-19v-250w (hanxia HX PZ1.27-2x3P TP, C41376035; on B, offset sign follows the flip); unit U5 (stock VQFN-32 footprint points at a STEP KiCad does not ship: pp48 copy with the stock QFN-32 5x5 EP3.3 body), J201 XT60 (C98732), photoMOS U6 / U7 / U56 / U57 TLP176AM (C5370540) and opto U8 / U58 TLP291 (C55144, turned to its pin-1 dot) as pp48 footprint copies (stock models missing), FPIDs moved in uinput.py / unit.py and the board; carrier F1 nano2 fuse (C44479) as a carrier footprint copy; placement = pad fit of the LCSC footprint + the STEP-to-WRL origin shift (EasyEDA STEPs are not on the footprint origin, checked against the XT30 of 020591f), which also corrects today's aux socket (+0.3 mm z) and Degson terminal (-0.1 y, +0.2 z); renders checked; ERC 0 and DRC counts unchanged on unit, carrier, module
Parts:
- U5: footprint Package_DFN_QFN:VQFN-32-1EP_5x5mm_P0.5mm_EP3.15x3.15mm -> pp48:VQFN-32-1EP_5x5mm_P0.5mm_EP3.15x3.15mm
- U56, U57, U6, U7: footprint Package_SO:SOIC-4_4.55x3.7mm_P2.54mm -> pp48:SOIC-4_4.55x3.7mm_P2.54mm
- U58, U8: footprint Package_SO:SOIC-4_4.55x2.6mm_P1.27mm -> pp48:SOIC-4_4.55x2.6mm_P1.27mm
Changed lines of the file:
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@@
 			)
 		)
-		(property "Footprint" "Package_SO:SOIC-4_4.55x3.7mm_P2.54mm"
+		(property "Footprint" "pp48:SOIC-4_4.55x3.7mm_P2.54mm"
 			(at 264.16 73.66 0)
 			(hide yes)
@@
 			)
 		)
-		(property "Footprint" "Package_SO:SOIC-4_4.55x3.7mm_P2.54mm"
+		(property "Footprint" "pp48:SOIC-4_4.55x3.7mm_P2.54mm"
 			(at 312.42 58.42 0)
 			(hide yes)
@@
 			)
 		)
-		(property "Footprint" "Package_SO:SOIC-4_4.55x2.6mm_P1.27mm"
+		(property "Footprint" "pp48:SOIC-4_4.55x2.6mm_P1.27mm"
 			(at 287.02 78.74 0)
 			(hide yes)
@@
 			)
 		)
-		(property "Footprint" "Package_SO:SOIC-4_4.55x3.7mm_P2.54mm"
+		(property "Footprint" "pp48:SOIC-4_4.55x3.7mm_P2.54mm"
 			(at 645.16 73.66 0)
 			(hide yes)
@@
 			)
 		)
-		(property "Footprint" "Package_SO:SOIC-4_4.55x3.7mm_P2.54mm"
+		(property "Footprint" "pp48:SOIC-4_4.55x3.7mm_P2.54mm"
 			(at 693.42 58.42 0)
 			(hide yes)
@@
 			)
 		)
-		(property "Footprint" "Package_SO:SOIC-4_4.55x2.6mm_P1.27mm"
+		(property "Footprint" "pp48:SOIC-4_4.55x2.6mm_P1.27mm"
 			(at 668.02 78.74 0)
 			(hide yes)
@@
 			)
 		)
-		(property "Footprint" "Package_DFN_QFN:VQFN-32-1EP_5x5mm_P0.5mm_EP3.15x3.15mm"
+		(property "Footprint" "pp48:VQFN-32-1EP_5x5mm_P0.5mm_EP3.15x3.15mm"
 			(at 101.6 241.3 0)
 			(hide yes)

Commit message: pp-48-unit: LCSC codes on the 22 parts that had none (JLC parts API 2026-10-30): BASIC table gains the hot-swap passives (143k / 124k 0805, 4.99k / 13.7k 0402 extended, best stocked; 20.0k, 10R 0402 and 220n 0603 25 V basic); Q1 / Q51 BSC070N10NS5 C534364 (the module's code); U2 / U52 / U208 INA238AIDGSR C2868250 (JLC stock 0: global sourcing or consigned); schematic regenerated, fields set on the routed board from the netlist; ERC 0, DRC unchanged (171, 0 unconnected, parity clean)
Parts:
- C1, C51: LCSC (none) -> C21120
- Q1, Q51: LCSC (none) -> C534364
- R3, R53: LCSC (none) -> C2930167
- R5, R55: LCSC (none) -> C2933298
- R56, R6: LCSC (none) -> C137965
- R57, R7: LCSC (none) -> C2933072
- U2, U52: LCSC (none) -> C2868250; MPN (none) -> TI INA238AIDGSR
Changed lines of the file:
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@@
 			)
 		)
-		(property "LCSC" ""
+		(property "LCSC" "C534364"
 			(at 124.46 43.18 0)
 			(hide yes)
@@
 			)
 		)
-		(property "LCSC" ""
+		(property "LCSC" "C2930167"
 			(at 86.36 87.63 0)
 			(hide yes)
@@
 			)
 		)
-		(property "LCSC" ""
+		(property "LCSC" "C2933298"
 			(at 96.52 69.85 0)
 			(hide yes)
@@
 			)
 		)
-		(property "LCSC" ""
+		(property "LCSC" "C137965"
 			(at 96.52 80.01 0)
 			(hide yes)
@@
 			)
 		)
-		(property "LCSC" ""
+		(property "LCSC" "C2933072"
 			(at 147.32 83.82 0)
 			(hide yes)
@@
 			)
 		)
-		(property "LCSC" ""
+		(property "LCSC" "C21120"
 			(at 137.16 86.36 0)
 			(hide yes)
@@
 			)
 		)
-		(property "LCSC" ""
+		(property "LCSC" "C2868250"
+			(at 55.88 76.2 0)
+			(hide yes)
+			(show_name no)
+			(do_not_autoplace no)
+			(effects
+				(font
+					(size 1.27 1.27)
+				)
+				(justify left)
+			)
+		)
+		(property "MPN" "TI INA238AIDGSR"
 			(at 55.88 76.2 0)
 			(hide yes)
@@
 			)
 		)
-		(property "LCSC" ""
+		(property "LCSC" "C534364"
 			(at 505.46 43.18 0)
 			(hide yes)
@@
 			)
 		)
-		(property "LCSC" ""
+		(property "LCSC" "C2930167"
 			(at 467.36 87.63 0)
 			(hide yes)
@@
 			)
 		)
-		(property "LCSC" ""
+		(property "LCSC" "C2933298"
 			(at 477.52 69.85 0)
 			(hide yes)
@@
 			)
 		)
-		(property "LCSC" ""
+		(property "LCSC" "C137965"
 			(at 477.52 80.01 0)
 			(hide yes)
@@
 			)
 		)
-		(property "LCSC" ""
+		(property "LCSC" "C2933072"
 			(at 528.32 83.82 0)
 			(hide yes)
@@
 			)
 		)
-		(property "LCSC" ""
+		(property "LCSC" "C21120"
 			(at 518.16 86.36 0)
 			(hide yes)
@@
 			)
 		)
-		(property "LCSC" ""
+		(property "LCSC" "C2868250"
+			(at 436.88 76.2 0)
+			(hide yes)
+			(show_name no)
+			(do_not_autoplace no)
+			(effects
+				(font
+					(size 1.27 1.27)
+				)
+				(justify left)
+			)
+		)
+		(property "MPN" "TI INA238AIDGSR"
 			(at 436.88 76.2 0)
 			(hide yes)

Commit message: stock replacements: unit INA238 (0 at JLC) -> INA237AIDGSR C2864837 on U2 / U52 / U208 (pin- and register-compatible for the plane-logic driver: SHUNT_CAL, LSBs, DIETEMP, MANUFACTURER_ID; gain error 0.3 %); module U2 / U3 MCP65R46-1.21 (0) -> MCP65R46T-2402E/CHY C623510 (2.4 V ref, same hysteresis, open drain, pinout) with R12 84.5k / R14 61.9k (OV_KILL 22.68 V, PGOOD 17.26 V, were 22.75 / 17.30), C13 -> C2980802 (100 V, same family); LM5069-1 left open for the user; boards synced from the netlists; ERC unchanged, DRC unchanged, parity clean; handoff
Parts:
- U2, U52: value INA238AIDGSR -> INA237AIDGSR; symbol Sensor_Energy:INA238 -> Sensor_Energy:INA237; LCSC C2868250 -> C2864837; MPN TI INA238AIDGSR -> TI INA237AIDGSR
Other:
- note added: "I2C SEGMENT: INA237 0x40 / 0x41, ADC121C027 0x51 / 0x52 (slot A / B), TCA6424A 0x22"
- note added: "SLOT A: 48 V HOT-SWAP, INA237, OV LATCH, MODULE MOUNT, ID ADC, NODE TERMINAL"
- note added: "SLOT B: 48 V HOT-SWAP, INA237, OV LATCH, MODULE MOUNT, ID ADC, NODE TERMINAL"
- note removed: "I2C SEGMENT: INA238 0x40 / 0x41, ADC121C027 0x51 / 0x52 (slot A / B), TCA6424A 0x22"
- note removed: "SLOT A: 48 V HOT-SWAP, INA238, OV LATCH, MODULE MOUNT, ID ADC, NODE TERMINAL"
- note removed: "SLOT B: 48 V HOT-SWAP, INA238, OV LATCH, MODULE MOUNT, ID ADC, NODE TERMINAL"
Changed lines of the file:
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@@
 		)
 	)
-	(text "SLOT A: 48 V HOT-SWAP, INA238, OV LATCH, MODULE MOUNT, ID ADC, NODE TERMINAL"
+	(text "SLOT A: 48 V HOT-SWAP, INA237, OV LATCH, MODULE MOUNT, ID ADC, NODE TERMINAL"
 		(exclude_from_sim no)
 		(at 15.24 25.4 0)
@@
 		)
 	)
-	(text "SLOT B: 48 V HOT-SWAP, INA238, OV LATCH, MODULE MOUNT, ID ADC, NODE TERMINAL"
+	(text "SLOT B: 48 V HOT-SWAP, INA237, OV LATCH, MODULE MOUNT, ID ADC, NODE TERMINAL"
 		(exclude_from_sim no)
 		(at 396.24 25.4 0)
@@
 		)
 	)
-	(text "I2C SEGMENT: INA238 0x40 / 0x41, ADC121C027 0x51 / 0x52 (slot A / B), TCA6424A 0x22"
+	(text "I2C SEGMENT: INA237 0x40 / 0x41, ADC121C027 0x51 / 0x52 (slot A / B), TCA6424A 0x22"
 		(exclude_from_sim no)
 		(at 15.24 190.5 0)
@@
 	)
 	(symbol
-		(lib_id "Sensor_Energy:INA238")
+		(lib_id "Sensor_Energy:INA237")
 		(at 55.88 76.2 270)
 		(unit 1)
@@
 			)
 		)
-		(property "Value" "INA238AIDGSR"
+		(property "Value" "INA237AIDGSR"
 			(at 75.85 64.77 90)
 			(show_name no)
@@
 			)
 		)
-		(property "LCSC" "C2868250"
+		(property "LCSC" "C2864837"
 			(at 55.88 76.2 0)
 			(hide yes)
@@
 			)
 		)
-		(property "MPN" "TI INA238AIDGSR"
+		(property "MPN" "TI INA237AIDGSR"
 			(at 55.88 76.2 0)
 			(hide yes)
@@
 			)
 		)
-		(property "Description" "INA238 VS"
+		(property "Description" "INA237 VS"
 			(at 73.66 80.01 0)
 			(hide yes)
@@
 	)
 	(symbol
-		(lib_id "Sensor_Energy:INA238")
+		(lib_id "Sensor_Energy:INA237")
 		(at 436.88 76.2 270)
 		(unit 1)
@@
 			)
 		)
-		(property "Value" "INA238AIDGSR"
+		(property "Value" "INA237AIDGSR"
 			(at 456.85 64.77 90)
 			(show_name no)
@@
 			)
 		)
-		(property "LCSC" "C2868250"
+		(property "LCSC" "C2864837"
 			(at 436.88 76.2 0)
 			(hide yes)
@@
 			)
 		)
-		(property "MPN" "TI INA238AIDGSR"
+		(property "MPN" "TI INA237AIDGSR"
 			(at 436.88 76.2 0)
 			(hide yes)
@@
 			)
 		)
-		(property "Description" "INA238 VS"
+		(property "Description" "INA237 VS"
 			(at 454.66 80.01 0)
 			(hide yes)
