File: power/pp-48-unit/sheets/input.kicad_sch (KiCad schematic)
At the start: 24 parts, among them J201 XT60PW-M, Q202 BSC040N10NS5, Q203 BSC040N10NS5, Q204 2N7002, U207 LM5069MM-1, U208 INA238AIDGSR

Commit message: pp-48 chained plane: LCSC codes for the input TVS (SMDJ60A C2990209), bulk cap (RVT2A470M1010 C87862) and unit shunts (6 mOhm SMA25A3FR006T C2692028), stock rechecked on JLCPCB's own API (jlcsearch mirror stale: mux, FET, 7 mOhm shunts are in stock); LM5069MM-1 down to 1; handoff
Parts:
- C201: LCSC (none) -> C87862; MPN (none) -> Lelon RVT2A470M1010
- D201: LCSC (none) -> C2990209
- R201, R202: LCSC (none) -> C2692028
Changed lines of the file:
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@@
 			)
 		)
-		(property "Description" "bus TVS 3 kW, unidirectional: cathode (pad 1) on VIN; 60 V standoff, breakdown >= 66.7 V, clamp 96.8 V; LCSC code to check"
+		(property "Description" "bus TVS 3 kW, unidirectional: cathode (pad 1) on VIN; 60 V standoff, breakdown >= 66.7 V, clamp 96.8 V"
 			(at 35.56 68.58 0)
 			(hide yes)
@@
 			)
 		)
-		(property "LCSC" ""
+		(property "LCSC" "C2990209"
 			(at 35.56 68.58 0)
 			(hide yes)
@@
 			)
 		)
-		(property "Description" "input bulk, damps cable ringing when the hot-swap opens; LCSC code to check"
+		(property "Description" "input bulk, damps cable ringing when the hot-swap opens"
 			(at 50.8 68.58 0)
 			(hide yes)
@@
 			)
 		)
-		(property "LCSC" ""
+		(property "LCSC" "C87862"
+			(at 50.8 68.58 0)
+			(hide yes)
+			(show_name no)
+			(do_not_autoplace no)
+			(effects
+				(font
+					(size 1.27 1.27)
+				)
+				(justify left)
+			)
+		)
+		(property "MPN" "Lelon RVT2A470M1010"
 			(at 50.8 68.58 0)
 			(hide yes)
@@
 			)
 		)
-		(property "Description" "shunt, two 6 mOhm in parallel = 3 mOhm: limit 18.3 A, breaker 35 A; LCSC code to check"
+		(property "Description" "shunt, two 6 mOhm in parallel = 3 mOhm: limit 18.3 A, breaker 35 A"
 			(at 77.47 60.96 0)
 			(hide yes)
@@
 			)
 		)
-		(property "LCSC" ""
+		(property "LCSC" "C2692028"
 			(at 77.47 60.96 0)
 			(hide yes)
@@
 			)
 		)
-		(property "LCSC" ""
+		(property "LCSC" "C2692028"
 			(at 77.47 68.58 0)
 			(hide yes)
@@
 			)
 		)
-		(property "Description" "100 V 4 mOhm pass FET; carries the start-up SOA alone (power limit 75 W, 10 ms); LCSC stock to check"
+		(property "Description" "100 V 4 mOhm pass FET; carries the start-up SOA alone (power limit 75 W, 10 ms)"
 			(at 157.48 63.5 0)
 			(hide yes)
@@
 			)
 		)
-		(property "Description" "unit hot-swap, 55 mV current limit, power limit, LATCH-OFF (-1); LCSC stock low (5 in a 2026-10-29 snapshot)"
+		(property "Description" "unit hot-swap, 55 mV current limit, power limit, LATCH-OFF (-1); LCSC stock 1 on 2026-10-29 (LM5069MM-2 C111822 has 7k)"
 			(at 154.94 91.44 0)
 			(hide yes)

Commit message: 3D models: module aux header J2 on pm-19v-250w (hanxia HX PZ1.27-2x3P TP, C41376035; on B, offset sign follows the flip); unit U5 (stock VQFN-32 footprint points at a STEP KiCad does not ship: pp48 copy with the stock QFN-32 5x5 EP3.3 body), J201 XT60 (C98732), photoMOS U6 / U7 / U56 / U57 TLP176AM (C5370540) and opto U8 / U58 TLP291 (C55144, turned to its pin-1 dot) as pp48 footprint copies (stock models missing), FPIDs moved in uinput.py / unit.py and the board; carrier F1 nano2 fuse (C44479) as a carrier footprint copy; placement = pad fit of the LCSC footprint + the STEP-to-WRL origin shift (EasyEDA STEPs are not on the footprint origin, checked against the XT30 of 020591f), which also corrects today's aux socket (+0.3 mm z) and Degson terminal (-0.1 y, +0.2 z); renders checked; ERC 0 and DRC counts unchanged on unit, carrier, module
Parts:
- J201: footprint Connector_AMASS:AMASS_XT60PW-M_1x02_P7.20mm_Horizontal -> pp48:AMASS_XT60PW-M_1x02_P7.20mm_Horizontal
Changed lines of the file:
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@@
 			)
 		)
-		(property "Footprint" "Connector_AMASS:AMASS_XT60PW-M_1x02_P7.20mm_Horizontal"
+		(property "Footprint" "pp48:AMASS_XT60PW-M_1x02_P7.20mm_Horizontal"
 			(at 22.86 58.42 0)
 			(hide yes)

Commit message: pp-48-unit: LCSC codes on the 22 parts that had none (JLC parts API 2026-10-30): BASIC table gains the hot-swap passives (143k / 124k 0805, 4.99k / 13.7k 0402 extended, best stocked; 20.0k, 10R 0402 and 220n 0603 25 V basic); Q1 / Q51 BSC070N10NS5 C534364 (the module's code); U2 / U52 / U208 INA238AIDGSR C2868250 (JLC stock 0: global sourcing or consigned); schematic regenerated, fields set on the routed board from the netlist; ERC 0, DRC unchanged (171, 0 unconnected, parity clean)
Parts:
- C203: LCSC (none) -> C21120
- R210, R211: LCSC (none) -> C25077
- R233: LCSC (none) -> C2930167
- R235: LCSC (none) -> C2933298
- R236: LCSC (none) -> C137965
- R237: LCSC (none) -> C25765
- U208: LCSC (none) -> C2868250; MPN (none) -> TI INA238AIDGSR
Changed lines of the file:
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@@
 			)
 		)
-		(property "LCSC" ""
+		(property "LCSC" "C25077"
 			(at 147.32 72.39 0)
 			(hide yes)
@@
 			)
 		)
-		(property "LCSC" ""
+		(property "LCSC" "C25077"
 			(at 157.48 41.91 0)
 			(hide yes)
@@
 			)
 		)
-		(property "LCSC" ""
+		(property "LCSC" "C2930167"
 			(at 119.38 107.95 0)
 			(hide yes)
@@
 			)
 		)
-		(property "LCSC" ""
+		(property "LCSC" "C2933298"
 			(at 129.54 90.17 0)
 			(hide yes)
@@
 			)
 		)
-		(property "LCSC" ""
+		(property "LCSC" "C137965"
 			(at 129.54 100.33 0)
 			(hide yes)
@@
 			)
 		)
-		(property "LCSC" ""
+		(property "LCSC" "C25765"
 			(at 180.34 104.14 0)
 			(hide yes)
@@
 			)
 		)
-		(property "LCSC" ""
+		(property "LCSC" "C21120"
 			(at 170.18 106.68 0)
 			(hide yes)
@@
 			)
 		)
-		(property "LCSC" ""
+		(property "LCSC" "C2868250"
 			(at 88.9 96.52 0)
 			(hide yes)
+			(show_name no)
+			(do_not_autoplace no)
+			(effects
+				(font
+					(size 1.27 1.27)
+				)
+				(justify left)
+			)
+		)
+		(property "MPN" "TI INA238AIDGSR"
+			(at 88.9 96.52 0)
+			(hide yes)

Commit message: stock replacements: unit INA238 (0 at JLC) -> INA237AIDGSR C2864837 on U2 / U52 / U208 (pin- and register-compatible for the plane-logic driver: SHUNT_CAL, LSBs, DIETEMP, MANUFACTURER_ID; gain error 0.3 %); module U2 / U3 MCP65R46-1.21 (0) -> MCP65R46T-2402E/CHY C623510 (2.4 V ref, same hysteresis, open drain, pinout) with R12 84.5k / R14 61.9k (OV_KILL 22.68 V, PGOOD 17.26 V, were 22.75 / 17.30), C13 -> C2980802 (100 V, same family); LM5069-1 left open for the user; boards synced from the netlists; ERC unchanged, DRC unchanged, parity clean; handoff
Parts:
- U208: value INA238AIDGSR -> INA237AIDGSR; symbol Sensor_Energy:INA238 -> Sensor_Energy:INA237; LCSC C2868250 -> C2864837; MPN TI INA238AIDGSR -> TI INA237AIDGSR
Other:
- note added: "UNIT INPUT J201 XT60 -> TVS -> U207 LM5069-1 (3 mOhm, Q202 || Q203) -> VBUS; U208 INA237 0x44"
- note removed: "UNIT INPUT J201 XT60 -> TVS -> U207 LM5069-1 (3 mOhm, Q202 || Q203) -> VBUS; U208 INA238 0x44"
Changed lines of the file:
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@@
 		)
 	)
-	(text "UNIT INPUT  J201 XT60 -> TVS -> U207 LM5069-1 (3 mOhm, Q202 || Q203) -> VBUS; U208 INA238 0x44"
+	(text "UNIT INPUT  J201 XT60 -> TVS -> U207 LM5069-1 (3 mOhm, Q202 || Q203) -> VBUS; U208 INA237 0x44"
 		(exclude_from_sim no)
 		(at 15.24 15.24 0)
@@
 	)
 	(symbol
-		(lib_id "Sensor_Energy:INA238")
+		(lib_id "Sensor_Energy:INA237")
 		(at 88.9 96.52 270)
 		(unit 1)
@@
 			)
 		)
-		(property "Value" "INA238AIDGSR"
+		(property "Value" "INA237AIDGSR"
 			(at 108.87 85.09 90)
 			(show_name no)
@@
 			)
 		)
-		(property "LCSC" "C2868250"
+		(property "LCSC" "C2864837"
 			(at 88.9 96.52 0)
 			(hide yes)
@@
 			)
 		)
-		(property "MPN" "TI INA238AIDGSR"
+		(property "MPN" "TI INA237AIDGSR"
 			(at 88.9 96.52 0)
 			(hide yes)
@@
 			)
 		)
-		(property "Description" "INA238 VS"
+		(property "Description" "INA237 VS"
 			(at 106.68 100.33 0)
 			(hide yes)

Commit message: pp-48-unit: unit hot-swap U207 LM5069MM-1 (latch-off, 1 at JLC) -> LM5069MM-2 C111822 (auto-retry, as the slots; user 2026-10-30); the latch moves into the core firmware: ADR 0005 decision 3 (U_PGD falling with the unit input in range -> core holds U_OFF high until unit_reset; no latch on a bus dip; no core = retry forever, unit ON), uinput.py notes, Q204 / U207 descriptions, title comment; schematic regenerated, board synced; ERC 0, DRC unchanged, parity clean; handoff
Parts:
- U207: value LM5069MM-1 -> LM5069MM-2; symbol Power_Management:LM5069MM-1 -> Power_Management:LM5069MM-2; LCSC C486026 -> C111822
Other:
- note added: "UNIT INPUT J201 XT60 -> TVS -> U207 LM5069-2 (3 mOhm, Q202 || Q203) -> VBUS; U208 INA237 0x44"
- note removed: "UNIT INPUT J201 XT60 -> TVS -> U207 LM5069-1 (3 mOhm, Q202 || Q203) -> VBUS; U208 INA237 0x44"
Changed lines of the file:
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@@
 		)
 	)
-	(text "UNIT INPUT  J201 XT60 -> TVS -> U207 LM5069-1 (3 mOhm, Q202 || Q203) -> VBUS; U208 INA237 0x44"
+	(text "UNIT INPUT  J201 XT60 -> TVS -> U207 LM5069-2 (3 mOhm, Q202 || Q203) -> VBUS; U208 INA237 0x44"
 		(exclude_from_sim no)
 		(at 15.24 15.24 0)
@@
 	)
 	(symbol
-		(lib_id "Power_Management:LM5069MM-1")
+		(lib_id "Power_Management:LM5069MM-2")
 		(at 154.94 91.44 0)
 		(unit 1)
@@
 			)
 		)
-		(property "Value" "LM5069MM-1"
+		(property "Value" "LM5069MM-2"
 			(at 173.91 80.01 0)
 			(show_name no)
@@
 			)
 		)
-		(property "Description" "unit hot-swap, 55 mV current limit, power limit, LATCH-OFF (-1); LCSC stock 1 on 2026-10-29 (LM5069MM-2 C111822 has 7k)"
+		(property "Description" "unit hot-swap, 55 mV current limit, power limit, auto-retry 0.5 % (-2); the latch is the firmware's, over U_OFF"
 			(at 154.94 91.44 0)
 			(hide yes)
@@
 			)
 		)
-		(property "LCSC" "C486026"
+		(property "LCSC" "C111822"
 			(at 154.94 91.44 0)
 			(hide yes)
@@
 			)
 		)
-		(property "Description" "expander U_OFF (P13) high = unit off (and resets the latched LM5069-1)"
+		(property "Description" "expander U_OFF (P13) high = unit off: the firmware latch after a unit fault"
 			(at 137.16 134.62 0)
 			(hide yes)
