File: power/pm-19v-250w-b/pm-19v-250w-b.kicad_sch (KiCad schematic)
At the start: 64 parts, among them J1 Screw pads S1-S4, J2 Aux header 2x3 1.27, Q1 BSC098N10NS5, Q2 BSC070N10NS5, Q3 BCX56-16, U1 LM5116MHX, U2 MCP65R46-2.4, U3 MCP65R46-2.4, U4 TPS3701DDCR

Commit message: PM-19V-250W-B schematic: second Kelvin net tie NT2 for CS, snubber dropped; ERC 0
Parts:
- removed C8: 470p 100V DNP, Capacitor_SMD:C_0805_2012Metric, symbol Device:C
- removed R5: 2.2R DNP, Resistor_SMD:R_0805_2012Metric, symbol Device:R
- added NT2: NetTie, NetTie:NetTie-2_SMD_Pad0.5mm, symbol Device:NetTie_2
Connections:
- net LSS: now also NT2.1; no longer U1.12 (CS)
- new net CS: NT2.2, U1.12 (CS)
Other:
- note added: "CS / CSG: Kelvin from R4's two pads through NT2 / NT1"
- note removed: "CSG: Kelvin from R4's GND pad through NT1; CS (LSS): Kelvin from R4's top pad"
